File: HC4_KiCad/HC4_KiCad.kicad_pcb (KiCad board)
At the start: 2 copper layers, 150 x 150 mm, 152 parts, among them IC1 RAM, IC10 74HC4002, IC11 74HC161, IC12 74HC377, IC13 74HC161, IC14 74HC161, IC15 74HC161, IC16 74HC257, IC17 74HC257, IC18 74HC00, IC19 74HC74, IC2 ROM, IC20 74HC4053, IC21 74HC04, IC22 74HC151, IC23 74HC32, IC24 74HC14, IC3 74HC153, IC4 74HC153, IC5 74HC153, IC6 74HC153, IC7 74HC283, IC8 74HC244, IC9 74HC244, J1 Power, J2 CE, J3 Expantion_Connector, SW1 SW_SPDT, SW2 Bus_Open, SW3 SW_Push, SW4 SW_Push, SW5 SW_SPDT

Commit message: ALU基板の製作途中
Parts:
- moved CP5 131.6 mm to (215.9, 35.6), turned to 90 degrees
- moved CP4 118.6 mm to (215.9, 48.3), turned to 90 degrees
- moved CP3 114.5 mm to (191.8, 35.5), turned to 90 degrees
- moved CP6 110.9 mm to (194.2, 142.4)
- moved CP7 110.9 mm to (197.3, 142.4)
- moved LD5 107.9 mm to (209.5, 147.3)
- moved LD4 106.9 mm to (212.1, 147.3)
- moved LD3 106.3 mm to (214.6, 147.3)
- moved LD2 106.1 mm to (217.2, 147.3)
- moved CP2 100.3 mm to (191.8, 48.2), turned to 90 degrees
- moved RN2 94.4 mm to (208.3, 128.3), turned to 180 degrees
- moved IC9 94.3 mm to (221.0, 130.8)
- moved J3 92.7 mm to (198.1, 152.4)
- moved IC10 92.2 mm to (227.3, 144.8)
- moved CP1 88.7 mm to (191.8, 58.5), turned to -90 degrees
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Routing:
- net /ALU/I3a: track 0.00 -> 53.5 mm
- net /Instruction Decoder/ALU_~{Eb}: track 0.00 -> 53.5 mm, vias 0 -> 1

Commit message: フットプリントの割り当て修正
Parts:
- added CP23: 0.1u, Capacitor_THT:C_Disc_D3.0mm_W1.6mm_P2.50mm, F.Cu at (169.5, 35.0)
- added CP24: 0.1u, Capacitor_THT:C_Disc_D3.0mm_W1.6mm_P2.50mm, F.Cu at (169.5, 38.2)
- added IC8: 74HC257, Package_DIP:DIP-16_W7.62mm_Socket, F.Cu at (156.2, 35.6)
- renumbered D14 to D10, D15 to D11, D16 to D12, D17 to D13, D18 to D14, D19 to D15, D20 to D16, D21 to D17, D22 to D18, D23 to D19, D6 to D2, D24 to D20, D25 to D21, D26 to D22, D27 to D23, D28 to D24, D29 to D25, D30 to D26, D31 to D27, D32 to D28, D33 to D29, D7 to D3, D34 to D30, D35 to D31, D36 to D32, D37 to D33, D38 to D34, D39 to D35, D40 to D36, D41 to D37, D42 to D38, D43 to D39, D8 to D4, D44 to D40, D45 to D41, D9 to D5, D10 to D6, D11 to D7, D12 to D8, D13 to D9, IC23 to IC19, IC19 to IC20, IC20 to IC21, IC21 to IC22, IC22 to IC23, LD8 to LD10, LD9 to LD11, LD10 to LD12, LD11 to LD13, LD12 to LD14, LD13 to LD15, LD14 to LD16, LD15 to LD17, LD16 to LD18, LD17 to LD19, LD26 to LD2, LD18 to LD20, LD19 to LD21, LD20 to LD22, LD21 to LD23, LD22 to LD24, LD23 to LD25, LD24 to LD26, LD25 to LD27, LD27 to LD3, LD2 to LD4, LD3 to LD5, LD4 to LD6, LD5 to LD7, LD6 to LD8, LD7 to LD9, R9 to R10, R10 to R11, R11 to R12, R12 to R13, R13 to R2, R14 to R3, R2 to R4, R4 to R5, R5 to R6, R6 to R7, R7 to R8, R8 to R9
Connections:
- D11 pad 2: Net-(D15-A) -> Net-(D11-A)
- D12 pad 2: Net-(D16-A) -> Net-(D12-A)
- D16 pad 2: Net-(D16-A) -> Net-(D12-A)
- D19 pad 2: Net-(D15-A) -> Net-(D11-A)
- D2 pad 1: Net-(D6-K) (its old number) -> Net-(D2-K)
- D27 pad 2: Net-(D15-A) -> Net-(D11-A)
- D3 pad 1: Net-(D6-K) (its old number) -> Net-(D2-K)
- D3 pad 2: Net-(D15-A) -> Net-(D11-A)
- D30 pad 1: Net-(D34-K) -> Net-(D30-K)
- D31 pad 1: Net-(D34-K) -> Net-(D30-K)
- D32 pad 1: Net-(D34-K) -> Net-(D30-K)
- D33 pad 1: Net-(D34-K) -> Net-(D30-K)
- D35 pad 2: Net-(D15-A) -> Net-(D11-A)
- D36 pad 2: Net-(D16-A) -> Net-(D12-A)
- D38 pad 1: Net-(D42-K) -> /Data BUS/Level_C_OE
- D38 pad 2: Net-(D42-A) -> unconnected-(D38-A-Pad2)
- D39 pad 1: Net-(D42-K) -> /Data BUS/Level_C_OE
- D39 pad 2: Net-(D15-A) -> Net-(D11-A)
- D4 pad 1: Net-(D6-K) (its old number) -> Net-(D2-K)
- D40 pad 1: Net-(D42-K) -> /Data BUS/Level_C_OE
- D40 pad 2: Net-(D16-A) -> Net-(D12-A)
- D41 pad 1: Net-(D42-K) -> /Data BUS/Level_C_OE
- D5 pad 1: Net-(D6-K) (its old number) -> Net-(D2-K)
- D5 pad 2: unconnected-(D9-A-Pad2) (its old number) -> unconnected-(D5-A-Pad2)
- IC18 pad 10: Net-(D42-K) -> VCC
- IC18 pad 13: Net-(D15-A) -> Net-(D11-A)
- IC18 pad 8: /Data BUS/~{Level_C_OE} -> unconnected-(IC18-Pad8)
- IC18 pad 9: Net-(D42-K) -> VCC
- IC19 pad 1: /Address BUS/Instruction_7 -> VCC
- IC19 pad 13: Net-(D34-K) -> Net-(D30-K)
- IC19 pad 2: Net-(D2-K) -> VCC
- IC19 pad 3: /Data BUS/~{ALU_OE} -> unconnected-(IC19-Pad3)
- IC19 pad 4: Net-(D42-A) -> Net-(IC19-Pad4)
- IC19 pad 9: Net-(D16-A) -> Net-(D12-A)
- IC22 pad 12: Net-(D15-A) -> Net-(D11-A)
- IC22 pad 2: Net-(D42-A) -> Net-(IC19-Pad4)
- IC22 pad 4: Net-(D16-A) -> Net-(D12-A)
- IC22 pad 9: Net-(D6-K) (its old number) -> Net-(D2-K)
- IC23 pad 11: /Address BUS/Instruction_2 -> /Address BUS/Instruction_0
- IC23 pad 9: /Address BUS/Instruction_0 -> /Address BUS/Instruction_2
- IC9 pad 2: /Address BUS/Instruction_4 -> /Address BUS/Instruction_0
- IC9 pad 4: /Address BUS/Instruction_5 -> /Address BUS/Instruction_1
- IC9 pad 6: /Address BUS/Instruction_6 -> /Address BUS/Instruction_2
- IC9 pad 8: /Address BUS/Instruction_7 -> /Address BUS/Instruction_3
- R6 pad 2: Net-(D42-K) -> /Data BUS/Level_C_OE
- RN6 pad 2: Net-(D2-K) -> Net-(D30-K)
- RN6 pad 3: Net-(D6-K) (its old number) -> Net-(D2-K)

Commit message: ALU単体の配線完了(芸術点Up)
Parts:
- moved IC8 68.2 mm to (218.4, 63.5), turned to 90 degrees
- moved CP23 52.0 mm to (215.9, 58.4), turned to -90 degrees
- moved CP4 2.54 mm to (215.9, 45.7), turned to -90 degrees
- moved CP5 2.54 mm to (215.9, 33.0), turned to -90 degrees
- moved CP2 2.46 mm to (191.8, 45.8), turned to -90 degrees
- moved CP3 2.46 mm to (191.8, 33.1), turned to -90 degrees
Routing:
- net GND: track 0.00 -> 207.9 mm, vias 0 -> 4
- net VCC: track 0.00 -> 173.2 mm
- net /ALU/I1a: track 0.00 -> 99.5 mm, vias 0 -> 4
- net /ALU/ALU_OUT1: track 0.00 -> 56.9 mm, vias 0 -> 1
- net /ALU/I0a: track 0.00 -> 56.6 mm
- net /ALU/ALU_OUT2: track 0.00 -> 56.5 mm
- net /ALU/Internal_A3: track 0.00 -> 54.7 mm
- net /ALU/I2a: track 0.00 -> 53.5 mm, vias 0 -> 2
- net /ALU/ALU_OUT0: track 0.00 -> 41.5 mm, vias 0 -> 1
- net /ALU/Internal_B3: track 0.00 -> 39.0 mm
- net /ALU/ALU_OUT3: track 0.00 -> 37.4 mm, vias 0 -> 1
- net /ALU/Internal_A2: track 0.00 -> 31.1 mm
- net /ALU/Internal_B2: track 0.00 -> 20.4 mm
- net /ALU/Internal_A0: track 0.00 -> 17.4 mm, vias 0 -> 1
- net /ALU/Internal_A1: track 0.00 -> 15.0 mm
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
Commit message: Adress Busを若干配線
Parts:
- moved IC18 109.0 mm to (197.6, 89.8), turned to 90 degrees
- moved LD20 106.1 mm to (172.3, 103.8), turned to 90 degrees
- moved LD21 102.4 mm to (175.3, 103.8), turned to 90 degrees
- moved LD22 98.9 mm to (178.3, 103.8), turned to 90 degrees
- moved LD23 95.4 mm to (181.3, 103.8), turned to 90 degrees
- moved LD24 92.1 mm to (184.3, 103.8), turned to 90 degrees
- moved CP15 91.0 mm to (195.1, 84.8), turned to -90 degrees
- moved LD25 88.9 mm to (187.3, 103.8), turned to 90 degrees
- moved R4 86.8 mm to (202.3, 122.9)
- moved RN5 86.8 mm to (203.0, 118.7)
- moved SW2 86.8 mm to (217.3, 122.9)
- moved LD26 85.9 mm to (190.3, 103.8), turned to 90 degrees
- moved LD27 82.8 mm to (193.3, 103.8), turned to 90 degrees
- moved IC17 79.2 mm to (218.4, 103.9), turned to 90 degrees
- moved CP13 69.3 mm to (215.8, 84.8), turned to -90 degrees
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Routing:
- net GND: track 207.9 -> 296.0 mm, vias 4 -> 5
- net VCC: track 173.2 -> 249.2 mm
- net /Address BUS/RAM_A1: track 0.00 -> 0.62 mm

Commit message: Adress Bus完成(芸術点Up)
Parts:
- IC19: footprint Package_DIP:DIP-16_W7.62mm_Socket -> Package_DIP:DIP-14_W7.62mm_Socket
- moved LD20 21.9 mm to (193.0, 96.5)
- moved LD21 21.5 mm to (195.6, 96.5)
- moved LD22 21.1 mm to (198.1, 96.5)
- moved LD23 20.6 mm to (200.7, 96.5)
- moved LD24 20.2 mm to (203.2, 96.5)
- moved LD25 19.8 mm to (205.7, 96.5)
- moved LD26 19.4 mm to (208.3, 96.5)
- moved LD27 18.9 mm to (210.8, 96.5)
- moved RN5 18.2 mm to (193.0, 103.5)
- moved R4 16.1 mm to (210.8, 109.2), turned to 180 degrees
- moved SW2 14.3 mm to (221.6, 109.2)
- moved CP4 12.7 mm to (215.9, 33.0)
- moved CP5 12.7 mm to (215.9, 45.7)
- moved IC6 12.7 mm to (218.4, 38.1)
- moved IC7 12.7 mm to (218.4, 50.8)
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Routing:
- net /ALU/ALU_in_A2: track 0.00 -> 135.3 mm, vias 0 -> 1
- net /ALU/ALU_in_A1: track 0.00 -> 115.6 mm, vias 0 -> 2
- net /ALU/ALU_in_A0: track 0.00 -> 88.1 mm
- net /ALU/ALU_in_A3: track 0.00 -> 82.8 mm, vias 0 -> 1
- net /Address BUS/RAM_A4: track 0.00 -> 75.6 mm
- net /ALU/ALU_in_B1: track 0.00 -> 74.9 mm, vias 0 -> 2
- net /Address BUS/RAM_A5: track 0.00 -> 67.5 mm, vias 0 -> 1
- net /ALU/ALU_in_B2: track 0.00 -> 58.0 mm, vias 0 -> 2
- net /ALU/ALU_in_B0: track 0.00 -> 56.2 mm, vias 0 -> 3
- net GND: track 296.0 -> 346.3 mm, vias 5 -> 4
- net /ALU/ALU_in_B3: track 0.00 -> 43.8 mm, vias 0 -> 1
- net /Address BUS/RAM_A6: track 0.00 -> 43.3 mm, vias 0 -> 1
- net /ALU/ALU_OUT2: track 56.5 -> 13.8 mm
- net /Address BUS/Instruction_7: track 0.00 -> 42.4 mm, vias 0 -> 4
- net /Address BUS/RAM_A2: track 0.00 -> 42.3 mm, vias 0 -> 2
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Other:
- board text added: "Adress Bus"
- board text removed: "adress bus"

Commit message: DataBus製作途中
Parts:
- moved SW4 124.4 mm to (117.5, 142.7)
- moved SW5 110.1 mm to (112.8, 154.0)
- moved SW3 106.6 mm to (121.7, 158.0)
- moved CP24 99.1 mm to (210.8, 128.3), turned to -90 degrees
- moved CP22 81.3 mm to (102.3, 158.1)
- moved IC24 81.3 mm to (98.8, 135.0)
- moved C2 81.3 mm to (92.2, 136.1)
- moved C3 81.3 mm to (92.2, 142.7)
- moved C4 81.3 mm to (92.2, 149.2)
- moved R10 81.3 mm to (80.9, 147.0)
- moved R11 81.3 mm to (80.9, 151.1)
- moved R12 81.3 mm to (80.9, 155.1)
- moved R13 81.3 mm to (80.9, 159.2)
- moved R7 81.3 mm to (80.9, 134.9)
- moved R8 81.3 mm to (80.9, 138.9)
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Routing:
- net /Data BUS/Stack0: track 0.00 -> 124.9 mm, vias 0 -> 4
- net GND: track 346.3 -> 447.3 mm, vias 4 -> 5
- net VCC: track 280.4 -> 380.0 mm
- net /ALU/I1a: track 97.4 -> 173.2 mm, vias 4 -> 6
- net /Data BUS/Stack1: track 0.00 -> 58.3 mm, vias 0 -> 1
- net /Data BUS/Stack2: track 0.00 -> 58.0 mm
- net /Data BUS/Stack3: track 0.00 -> 57.4 mm
- net (no net): track 0.00 -> 8.67 mm
- net Net-(D22-K): track 0.00 -> 2.54 mm
- net Net-(D18-K): track 0.00 -> 2.54 mm

Commit message: 電源周りが詰みそう
Parts:
- moved C3 17.9 mm to (82.3, 157.6)
- moved R10 17.9 mm to (71.0, 161.9)
- moved R11 17.9 mm to (71.0, 166.0)
- moved R13 17.9 mm to (71.0, 174.1)
- moved R8 17.9 mm to (71.0, 153.8)
- moved SW3 17.9 mm to (111.8, 172.9)
- moved SW4 17.9 mm to (107.6, 157.6)
- moved C2 17.9 mm to (82.3, 151.0)
- moved C4 17.9 mm to (82.3, 164.1)
- moved CP22 17.9 mm to (92.3, 173.0)
- moved IC24 17.9 mm to (88.9, 149.9)
- moved R12 17.9 mm to (71.0, 170.0)
- moved R7 17.9 mm to (71.0, 149.8)
- moved R9 17.9 mm to (71.0, 157.9)
- moved SW5 17.9 mm to (102.9, 168.9)
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Routing:
- net /ALU/ALU_OUT1: track 27.5 -> 179.8 mm, vias 0 -> 4
- net /Data BUS/Stack3: track 57.4 -> 200.0 mm, vias 0 -> 4
- net /ALU/ALU_OUT2: track 13.8 -> 150.4 mm, vias 0 -> 7
- net /Data BUS/Stack2: track 58.0 -> 189.4 mm, vias 0 -> 5
- net /Data BUS/Level_C0: track 0.00 -> 131.1 mm, vias 0 -> 4
- net /Address BUS/~{RAM_RD}: track 0.00 -> 112.4 mm, vias 0 -> 7
- net /ALU/ALU_OUT3: track 13.8 -> 114.8 mm, vias 0 -> 4
- net GND: track 447.3 -> 531.7 mm, vias 5 -> 9
- net /ALU/ALU_OUT0: track 14.8 -> 99.2 mm, vias 0 -> 7
- net /Data BUS/Level_C1: track 0.00 -> 79.0 mm, vias 0 -> 10
- net /Data BUS/Level_C3: track 0.00 -> 77.3 mm, vias 0 -> 1
- net VCC: track 380.0 -> 456.6 mm, vias 0 -> 2
- net /Data BUS/Stack1: track 58.3 -> 123.1 mm, vias 1 -> 3
- net /Address BUS/Instruction_1: track 0.00 -> 61.7 mm, vias 0 -> 4
- net /Address BUS/Instruction_0: track 0.00 -> 61.7 mm, vias 0 -> 4
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
Commit message: 更地になった。
Parts:
- moved IC1 91.5 mm to (82.5, 53.4)
- moved D1 88.2 mm to (99.6, 99.0)
- moved J1 88.2 mm to (125.7, 57.8)
- moved LD2 88.2 mm to (126.9, 86.5)
- moved LD3 88.2 mm to (126.9, 90.3)
- moved R1 88.2 mm to (121.8, 74.5)
- moved R3 88.2 mm to (121.8, 82.6)
- moved SW1 88.2 mm to (89.2, 99.3)
- moved C1 88.2 mm to (126.9, 95.4)
- moved F1 88.2 mm to (101.2, 94.6)
- moved IC2 88.2 mm to (101.5, 53.4)
- moved J2 88.2 mm to (122.5, 96.7)
- moved JP1 88.2 mm to (122.5, 87.0)
- moved LD1 88.2 mm to (112.0, 96.7)
- moved R2 88.2 mm to (121.8, 78.6)
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Routing:
- net /Data BUS/Stack3: track 200.0 -> 10.2 mm, vias 4 -> 0
- net /ALU/ALU_OUT1: track 179.8 -> 0.00 mm, vias 4 -> 0
- net /Data BUS/Stack2: track 189.4 -> 10.2 mm, vias 5 -> 0
- net /ALU/I1a: track 179.0 -> 0.57 mm, vias 5 -> 0
- net /ALU/ALU_OUT2: track 150.4 -> 0.00 mm, vias 7 -> 0
- net /ALU/ALU_in_A2: track 135.3 -> 0.00 mm, vias 1 -> 0
- net /Data BUS/Level_C0: track 131.1 -> 0.00 mm, vias 4 -> 0
- net /Data BUS/Stack0: track 129.7 -> 10.2 mm, vias 4 -> 0
- net /ALU/ALU_in_A1: track 115.6 -> 0.00 mm, vias 2 -> 0
- net /ALU/ALU_OUT3: track 114.8 -> 0.00 mm, vias 4 -> 0
- net /Data BUS/Stack1: track 123.1 -> 10.2 mm, vias 3 -> 0
- net /Address BUS/~{RAM_RD}: track 112.4 -> 0.00 mm, vias 7 -> 0
- net /Address BUS/RAM_A4: track 109.3 -> 0.00 mm, vias 1 -> 0
- net /Address BUS/RAM_A5: track 105.1 -> 0.00 mm, vias 2 -> 0
- net /Address BUS/RAM_A6: track 99.3 -> 0.00 mm, vias 2 -> 0
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