File: HC4_KiCad/HC4_KiCad.kicad_pcb (KiCad board)
At the start: 2 copper layers, 100 x 100 mm, 173 parts, among them IC1 KM62256CLP, IC10 74HC4002, IC11 74HC161, IC12 74HC377, IC13 74HC161, IC14 74HC161, IC15 74HC161, IC16 74HC257, IC17 74HC257, IC18 74HC74, IC19 74HC32, IC2 ROM, IC20 74HC04, IC21 74HC00, IC22 74HC4053, IC23 74HC151, IC24 74HC14, IC3 74HC153, IC4 74HC153, IC5 74HC153, IC6 74HC153, IC7 74HC283, IC8 74HC257, IC9 74HC244, J1 Power, J2 ~{CE}_EXT, J3 Expantion_Connector, SW1 SW_SPDT_312, SW2 Bus_Open, SW3 SW_Push, SW4 SW_Push, SW5 SW_SPDT

Commit message: さようなら、爺さん
Parts:
- moved IC8 135.5 mm to (68.6, 79.4), turned to 90 degrees
- moved IC14 0.64 mm to (129.5, 94.0)
- moved IC15 0.64 mm to (143.5, 94.0)
- moved IC13 0.64 mm to (115.6, 94.0)
Changed lines of the file:
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@@
 	(footprint "Package_SO:SO-16_5.3x10.2mm_P1.27mm"
 		(layer "F.Cu")
-		(at 130.175 93.98 90)
+		(at 129.54 93.98 90)
 		(descr "SO, 16 Pin (https://www.ti.com/lit/ml/msop002a/msop002a.pdf), generated with kicad-footprint-generator ipc_gullwing_generator.py")
 		(tags "SO SO")
@@
 	(footprint "Package_SO:SO-16_5.3x10.2mm_P1.27mm"
 		(layer "F.Cu")
-		(at 116.205 93.98 90)
+		(at 115.57 93.98 90)
 		(descr "SO, 16 Pin (https://www.ti.com/lit/ml/msop002a/msop002a.pdf), generated with kicad-footprint-generator ipc_gullwing_generator.py")
 		(tags "SO SO")
@@
 		(tags "LED")
 		(property "Reference" "LD4"
-			(at 1.27 -2.06 360)
+			(at 1.27 -2.06 0)
 			(layer "F.SilkS")
 			(effects
@@
 		)
 		(property "Value" "LED"
-			(at 1.27 2.06 360)
+			(at 1.27 2.06 0)
 			(layer "F.Fab")
 			(effects
@@
 		)
 		(property "Footprint" "LED_THT:LED_Rectangular_W5.0mm_H2.0mm"
-			(at 0 0 360)
+			(at 0 0 0)
 			(layer "F.Fab")
 			(hide yes)
@@
 		)
 		(property "Datasheet" ""
-			(at 0 0 360)
+			(at 0 0 0)
 			(layer "F.Fab")
 			(hide yes)
@@
 		)
 		(property "Description" "Light emitting diode"
-			(at 0 0 360)
+			(at 0 0 0)
 			(layer "F.Fab")
 			(hide yes)
@@
 		)
 		(fp_text user "${REFERENCE}"
-			(at 1.27 0 360)
+			(at 1.27 0 0)
 			(layer "F.Fab")
 			(effects
@@
 		(tags "Diode DO-34_SOD68 series Axial Horizontal pin pitch 7.62mm  length 3.04mm diameter 1.6mm")
 		(property "Reference" "D1"
-			(at 10.16 0 360)
+			(at 10.16 0 0)
 			(layer "F.SilkS")
 			(effects
@@
 		)
 		(property "Value" "5.6V"
-			(at 3.81 1.92 360)
+			(at 3.81 1.92 0)
 			(layer "F.Fab")
 			(effects
@@
 		)
 		(fp_text user "K"
-			(at -1.905 0 360)
+			(at -1.905 0 0)
 			(layer "F.SilkS")
 			(effects
@@
 		)
 		(fp_text user "K"
-			(at 0 -1.75 360)
+			(at 0 -1.75 0)
 			(layer "F.Fab")
 			(effects
@@
 		)
 		(fp_text user "${REFERENCE}"
-			(at 4.038 0 360)
+			(at 4.038 0 0)
 			(layer "F.Fab")
 			(effects
@@
 		(tags "LED")
 		(property "Reference" "LD32"
-			(at -3.81 0 360)
+			(at -3.81 0 0)
 			(layer "F.SilkS")
 			(effects
@@
 	(footprint "Package_SO:SO-16_5.3x10.2mm_P1.27mm"
 		(layer "F.Cu")
-		(at 191.56 136.27)
+		(at 68.58 79.375 90)
 		(descr "SO, 16 Pin (https://www.ti.com/lit/ml/msop002a/msop002a.pdf), generated with kicad-footprint-generator ipc_gullwing_generator.py")
 		(tags "SO SO")
 		(property "Reference" "IC8"
-			(at 0 -6.05 0)
+			(at 0 6.35 90)
 			(layer "F.SilkS")
 			(effects
@@
 		)
 		(property "Value" "74HC257"
-			(at 0 6.05 0)
+			(at 0 6.05 90)
 			(layer "F.Fab")
 			(effects
@@
 		)
 		(property "Footprint" "Package_SO:SO-16_5.3x10.2mm_P1.27mm"
-			(at 0 0 0)
+			(at 0 0 90)
 			(layer "F.Fab")
 			(hide yes)
@@
 		)
 		(property "Datasheet" "http://www.ti.com/lit/gpn/sn74LS257"
-			(at 0 0 0)
+			(at 0 0 90)
 			(layer "F.Fab")
 			(hide yes)
@@
 		)
 		(property "Description" "Quad 2 to 1 Multiplexer"
-			(at 0 0 0)
+			(at 0 0 90)
 			(layer "F.Fab")
 			(hide yes)
@@
 		(attr smd)
 		(fp_line
-			(start -2.76 -5.21)
-			(end -2.76 -5.005)
+			(start 2.76 -5.21)
+			(end 2.76 -5.005)
 			(stroke
 				(width 0.12)
@@
 		)
 		(fp_line
-			(start -2.76 5.21)
-			(end -2.76 5.005)
+			(start 0 -5.21)
+			(end 2.76 -5.21)
 			(stroke
 				(width 0.12)
@@
 		)
 		(fp_line
-			(start 0 -5.21)
-			(end 2.76 -5.21)
+			(start -2.76 -5.21)
+			(end -2.76 -5.005)
 			(stroke
 				(width 0.12)
@@
 		)
 		(fp_line
-			(start 0 5.21)
-			(end -2.76 5.21)
+			(start 2.76 5.21)
+			(end 2.76 5.005)
 			(stroke
 				(width 0.12)
@@
 		)
 		(fp_line
-			(start 2.76 -5.21)
-			(end 2.76 -5.005)
+			(start 0 5.21)
+			(end -2.76 5.21)
 			(stroke
 				(width 0.12)
@@
 		)
 		(fp_line
-			(start 2.76 5.21)
-			(end 2.76 5.005)
+			(start -2.76 5.21)
+			(end -2.76 5.005)
 			(stroke
 				(width 0.12)
@@
 		)
 		(fp_line
-			(start -4.7 -5.35)
-			(end -4.7 5.35)
+			(start 4.7 -5.35)
+			(end -4.7 -5.35)
 			(stroke
 				(width 0.05)
@@
 		)
 		(fp_line
-			(start -4.7 5.35)
-			(end 4.7 5.35)
+			(start -4.7 -5.35)
+			(end -4.7 5.35)
 			(stroke
 				(width 0.05)
@@
 		)
 		(fp_line
-			(start 4.7 -5.35)
-			(end -4.7 -5.35)
+			(start 4.7 5.35)
+			(end 4.7 -5.35)
 			(stroke
 				(width 0.05)
@@
 		)
 		(fp_line
-			(start 4.7 5.35)
-			(end 4.7 -5.35)
+			(start -4.7 5.35)
+			(end 4.7 5.35)
 			(stroke
 				(width 0.05)
@@
 		)
 		(fp_line
-			(start -2.65 -4.1)
-			(end -1.65 -5.1)
+			(start 2.65 -5.1)
+			(end 2.65 5.1)
 			(stroke
 				(width 0.1)
@@
 		)
 		(fp_line
-			(start -2.65 5.1)
-			(end -2.65 -4.1)
+			(start -1.65 -5.1)
+			(end 2.65 -5.1)
 			(stroke
 				(width 0.1)
@@
 		)
 		(fp_line
-			(start -1.65 -5.1)
-			(end 2.65 -5.1)
+			(start -2.65 -4.1)
+			(end -1.65 -5.1)
 			(stroke
 				(width 0.1)
@@
 		)
 		(fp_line
-			(start 2.65 -5.1)
-			(end 2.65 5.1)
+			(start 2.65 5.1)
+			(end -2.65 5.1)
 			(stroke
 				(width 0.1)
@@
 		)
 		(fp_line
-			(start 2.65 5.1)
-			(end -2.65 5.1)
+			(start -2.65 5.1)
+			(end -2.65 -4.1)
 			(stroke
 				(width 0.1)
@@
 		)
 		(fp_text user "${REFERENCE}"
-			(at 0 0 0)
+			(at 0 0 90)
 			(layer "F.Fab")
 			(effects
@@
 		)
 		(pad "1" smd roundrect
-			(at -3.4625 -4.445)
+			(at -3.4625 -4.445 90)
 			(size 1.975 0.6)
 			(layers "F.Cu" "F.Paste" "F.Mask")
@@
 		)
 		(pad "2" smd roundrect
-			(at -3.4625 -3.175)
+			(at -3.4625 -3.175 90)
 			(size 1.975 0.6)
 			(layers "F.Cu" "F.Paste" "F.Mask")
@@
 		)
 		(pad "3" smd roundrect
-			(at -3.4625 -1.905)
+			(at -3.4625 -1.905 90)
 			(size 1.975 0.6)
 			(layers "F.Cu" "F.Paste" "F.Mask")
@@
 		)
 		(pad "4" smd roundrect
-			(at -3.4625 -0.635)
+			(at -3.4625 -0.635 90)
 			(size 1.975 0.6)
 			(layers "F.Cu" "F.Paste" "F.Mask")
@@
 		)
 		(pad "5" smd roundrect
-			(at -3.4625 0.635)
+			(at -3.4625 0.635 90)
 			(size 1.975 0.6)
 			(layers "F.Cu" "F.Paste" "F.Mask")
@@
 		)
 		(pad "6" smd roundrect
-			(at -3.4625 1.905)
+			(at -3.4625 1.905 90)
 			(size 1.975 0.6)
 			(layers "F.Cu" "F.Paste" "F.Mask")
@@
 		)
 		(pad "7" smd roundrect
-			(at -3.4625 3.175)
+			(at -3.4625 3.175 90)
 			(size 1.975 0.6)
 			(layers "F.Cu" "F.Paste" "F.Mask")
@@
 		)
 		(pad "8" smd roundrect
-			(at -3.4625 4.445)
+			(at -3.4625 4.445 90)
 			(size 1.975 0.6)
 			(layers "F.Cu" "F.Paste" "F.Mask")
@@
 		)
 		(pad "9" smd roundrect
-			(at 3.4625 4.445)
+			(at 3.4625 4.445 90)
 			(size 1.975 0.6)
 			(layers "F.Cu" "F.Paste" "F.Mask")
@@
 		)
 		(pad "10" smd roundrect
-			(at 3.4625 3.175)
+			(at 3.4625 3.175 90)
 			(size 1.975 0.6)
 			(layers "F.Cu" "F.Paste" "F.Mask")
@@
 		)
 		(pad "11" smd roundrect
-			(at 3.4625 1.905)
+			(at 3.4625 1.905 90)
 			(size 1.975 0.6)
 			(layers "F.Cu" "F.Paste" "F.Mask")
@@
 		)
 		(pad "12" smd roundrect
-			(at 3.4625 0.635)
+			(at 3.4625 0.635 90)
 			(size 1.975 0.6)
 			(layers "F.Cu" "F.Paste" "F.Mask")
@@
 		)
 		(pad "13" smd roundrect
-			(at 3.4625 -0.635)
+			(at 3.4625 -0.635 90)
 			(size 1.975 0.6)
 			(layers "F.Cu" "F.Paste" "F.Mask")
@@
 		)
 		(pad "14" smd roundrect
-			(at 3.4625 -1.905)
+			(at 3.4625 -1.905 90)
 			(size 1.975 0.6)
 			(layers "F.Cu" "F.Paste" "F.Mask")
@@
 		)
 		(pad "15" smd roundrect
-			(at 3.4625 -3.175)
+			(at 3.4625 -3.175 90)
 			(size 1.975 0.6)
 			(layers "F.Cu" "F.Paste" "F.Mask")
@@
 		)
 		(pad "16" smd roundrect
-			(at 3.4625 -4.445)
+			(at 3.4625 -4.445 90)
 			(size 1.975 0.6)
 			(layers "F.Cu" "F.Paste" "F.Mask")
@@
 		(tags "ptc resettable fuse polyfuse THT")
 		(property "Reference" "F1"
-			(at 2.54 -1.905 360)
+			(at 2.54 -1.905 0)
 			(layer "F.SilkS")
 			(effects
@@
 		)
 		(property "Value" "Polyfuse"
-			(at 2.55 3.1 360)
+			(at 2.55 3.1 0)
 			(layer "F.Fab")
 			(effects
@@
 		)
 		(fp_text user "${REFERENCE}"
-			(at 2.55 0.6 360)
+			(at 2.55 0.6 0)
 			(layer "F.Fab")
 			(effects
@@
 	(footprint "Package_SO:SO-16_5.3x10.2mm_P1.27mm"
 		(layer "F.Cu")
-		(at 144.145 93.98 90)
+		(at 143.51 93.98 90)
 		(descr "SO, 16 Pin (https://www.ti.com/lit/ml/msop002a/msop002a.pdf), generated with kicad-footprint-generator ipc_gullwing_generator.py")
 		(tags "SO SO")
@@
 		(tags "THT DIP DIL ZIF 15.24mm 600mil Socket")
 		(property "Reference" "IC2"
-			(at -5.08 -10.16 360)
+			(at -5.08 -10.16 0)
 			(layer "F.SilkS")
 			(effects

Commit message: Added output port for blink
Parts:
- removed the IC1 at (64.8, 97.2)
- added IC10: 74HC374, Package_SO:SOP-20_7.5x12.8mm_P1.27mm, F.Cu at (83.2, 118.7)
- added JP1: Blink_EN, Connector_PinSocket_2.54mm:PinSocket_1x02_P2.54mm_Vertical, F.Cu at (188.8, 72.5)
- added LD10: LED, LED_THT:LED_Rectangular_W5.0mm_H2.0mm, F.Cu at (104.8, 144.1)
- added LD11: LED, LED_THT:LED_Rectangular_W5.0mm_H2.0mm, F.Cu at (107.3, 144.1)
- added LD8: LED, LED_THT:LED_Rectangular_W5.0mm_H2.0mm, F.Cu at (99.7, 144.1)
- added LD9: LED, LED_THT:LED_Rectangular_W5.0mm_H2.0mm, F.Cu at (102.2, 144.1)
- RN1: footprint Resistor_THT:R_Array_SIP5 -> Resistor_THT:R_Array_SIP9
- moved IC6 201.5 mm to (67.3, 89.5), turned to 90 degrees
- moved IC2 156.8 mm to (67.3, 67.9), turned to 90 degrees
- moved IC3 155.5 mm to (79.0, 33.7)
- moved IC4 155.5 mm to (89.5, 33.7)
- moved IC5 155.5 mm to (99.9, 33.7)
- moved IC8 114.9 mm to (66.7, 118.7), turned to 90 degrees
- moved RN1 97.8 mm to (89.5, 148.0)
- moved LD4 90.4 mm to (89.5, 144.1), turned to 90 degrees
- moved LD5 86.8 mm to (92.1, 144.1), turned to 90 degrees
- moved LD6 83.4 mm to (94.6, 144.1), turned to 90 degrees
- moved LD7 80.1 mm to (97.2, 144.1), turned to 90 degrees
- moved IC7 22.9 mm to (67.3, 102.2)
- moved CP16 21.0 mm to (83.2, 67.9)
- moved IC16 21.0 mm to (89.5, 67.9)
- moved IC17 12.3 mm to (89.5, 78.1)
- renumbered IC2 to IC1, IC3 to IC2, IC4 to IC3, IC5 to IC4, IC6 to IC5, IC7 to IC6, IC8 to IC7, IC9 to IC8, IC10 to IC9, J3 to J2, LD8 to LD12, LD9 to LD13, LD10 to LD14, LD11 to LD15, LD12 to LD16, LD13 to LD17, LD14 to LD18, LD15 to LD19, LD16 to LD20, LD17 to LD21, LD18 to LD22, LD19 to LD23, LD20 to LD24, LD21 to LD25, LD22 to LD26, LD23 to LD27, LD24 to LD28, LD25 to LD29, LD26 to LD30, LD27 to LD31, LD28 to LD32, LD29 to LD33, LD30 to LD34, LD31 to LD35, LD32 to LD36, LD33 to LD37, LD34 to LD38, LD35 to LD39, LD36 to LD40, LD37 to LD41, LD38 to LD42, LD39 to LD43, LD40 to LD44, LD41 to LD45, SW2 to SW1, SW3 to SW2, SW4 to SW3, SW5 to SW4
Connections:
- J2 pad 31: unconnected-(J3-Pin_31-Pad31) -> /Data BUS/PA0
- J2 pad 32: unconnected-(J3-Pin_32-Pad32) -> /Data BUS/PA1
- J2 pad 33: unconnected-(J3-Pin_33-Pad33) -> /Data BUS/PA2
- J2 pad 34: unconnected-(J3-Pin_34-Pad34) -> /Data BUS/PA3

Commit message: 部品配置完了
Parts:
- removed the J2 at (213.4, 104.0)
- removed the JP1 at (213.6, 46.9)
- removed REF** (x3): MountingHole_3.2mm_M3, MountingHole:MountingHole_3.2mm_M3
- removed the SW1 at (198.7, 100.5)
- added G***: LOGO, LOGO, F.Cu at (134.5, 143.0)
- added H1: MountingHole, MountingHole:MountingHole_3.2mm_M3, F.Cu at (146.5, 57.5)
- added H2: MountingHole, MountingHole:MountingHole_3.2mm_M3, F.Cu at (53.5, 57.5)
- added H3: MountingHole, MountingHole:MountingHole_3.2mm_M3, F.Cu at (146.5, 146.5)
- added H4: MountingHole, MountingHole:MountingHole_3.2mm_M3, F.Cu at (53.5, 146.5)
- added TP1: TestPoint, Library:TestPoint_THTPad_1.0x1.0mm_Drill0.5mm, F.Cu at (130.2, 100.3)
- added TP10: TestPoint, Library:TestPoint_THTPad_1.0x1.0mm_Drill0.5mm, F.Cu at (144.8, 114.3)
- added TP11: TestPoint, Library:TestPoint_THTPad_1.0x1.0mm_Drill0.5mm, F.Cu at (144.8, 116.8)
- added TP12: TestPoint, Library:TestPoint_THTPad_1.0x1.0mm_Drill0.5mm, F.Cu at (144.8, 119.4)
- added TP13: TestPoint, Library:TestPoint_THTPad_1.0x1.0mm_Drill0.5mm, F.Cu at (144.8, 121.9)
- added TP14: TestPoint, Library:TestPoint_THTPad_1.0x1.0mm_Drill0.5mm, F.Cu at (144.8, 124.5)
- added TP15: TestPoint, Library:TestPoint_THTPad_1.0x1.0mm_Drill0.5mm, F.Cu at (144.8, 127.0)
- added TP16: TestPoint, Library:TestPoint_THTPad_1.0x1.0mm_Drill0.5mm, F.Cu at (85.7, 77.5)
- added TP17: TestPoint, Library:TestPoint_THTPad_1.0x1.0mm_Drill0.5mm, F.Cu at (78.7, 132.7)
- added TP18: TestPoint, Library:TestPoint_THTPad_1.0x1.0mm_Drill0.5mm, F.Cu at (109.9, 113.7)
- added TP19: TestPoint, Library:TestPoint_THTPad_1.0x1.0mm_Drill0.5mm, F.Cu at (76.8, 104.8)
- added TP2: TestPoint, Library:TestPoint_THTPad_1.0x1.0mm_Drill0.5mm, F.Cu at (130.2, 97.2)
- added TP20: TestPoint, Library:TestPoint_THTPad_1.0x1.0mm_Drill0.5mm, F.Cu at (70.5, 91.4)
- added TP21: TestPoint, Library:TestPoint_THTPad_1.0x1.0mm_Drill0.5mm, F.Cu at (66.7, 91.4)
- added TP22: TestPoint, Library:TestPoint_THTPad_1.0x1.0mm_Drill0.5mm, F.Cu at (62.9, 91.4)
- added TP23: TestPoint, Library:TestPoint_THTPad_1.0x1.0mm_Drill0.5mm, F.Cu at (109.9, 92.1)
- added TP3: TestPoint, Library:TestPoint_THTPad_1.0x1.0mm_Drill0.5mm, F.Cu at (130.2, 94.0)
- added TP4: TestPoint, Library:TestPoint_THTPad_1.0x1.0mm_Drill0.5mm, F.Cu at (130.2, 90.8)
- added TP5: TestPoint, Library:TestPoint_THTPad_1.0x1.0mm_Drill0.5mm, F.Cu at (74.3, 91.4)
- added TP6: TestPoint, Library:TestPoint_THTPad_1.0x1.0mm_Drill0.5mm, F.Cu at (144.8, 104.1)
- added TP7: TestPoint, Library:TestPoint_THTPad_1.0x1.0mm_Drill0.5mm, F.Cu at (144.8, 106.7)
- added TP8: TestPoint, Library:TestPoint_THTPad_1.0x1.0mm_Drill0.5mm, F.Cu at (144.8, 109.2)
- added TP9: TestPoint, Library:TestPoint_THTPad_1.0x1.0mm_Drill0.5mm, F.Cu at (144.8, 111.8)
- moved CP24 206.6 mm to (83.8, 116.8), turned to -90 degrees
- moved C4 205.2 mm to (88.3, 129.5)
- moved CP12 202.9 mm to (77.5, 92.7), turned to -90 degrees
- moved SW4 201.8 mm to (84.5, 132.7), turned to 90 degrees
- moved R15 191.4 mm to (104.8, 137.8), turned to 90 degrees
- moved R17 190.3 mm to (94.0, 137.2), turned to 90 degrees
- moved C3 190.2 mm to (97.2, 136.5)
- moved C2 189.9 mm to (97.2, 128.9)
- moved R16 187.6 mm to (108.0, 137.8), turned to 90 degrees
- moved CP17 185.4 mm to (60.3, 107.3), turned to -90 degrees
- moved LD44 184.2 mm to (119.5, 143.5), turned to 90 degrees
- moved IC24 183.2 mm to (90.2, 120.0), turned to 90 degrees
- moved CP13 182.6 mm to (96.5, 104.8), turned to -90 degrees
- moved LD45 180.5 mm to (122.0, 143.5), turned to 90 degrees
- moved R19 180.4 mm to (113.7, 137.2), turned to 90 degrees
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Routing:
- net /ALU/I1a: track 0.00 -> 26.4 mm
- net /ALU/I2a: track 0.00 -> 26.4 mm
- net /ALU/Carry_IN: track 0.00 -> 26.4 mm
- net /ALU/I3a: track 0.00 -> 26.4 mm
- net /Data BUS/Dummy6: track 0.00 -> 14.9 mm
- net /Data BUS/Dummy7: track 0.00 -> 13.0 mm
- net /Data BUS/Dummy4: track 0.00 -> 12.5 mm
- net /Data BUS/Dummy5: track 0.00 -> 10.5 mm
- net /Data BUS/Databus2: track 0.00 -> 9.83 mm
- net /Data BUS/Databus3: track 0.00 -> 7.93 mm
- net /Data BUS/Databus0: track 0.00 -> 7.83 mm
- net /Data BUS/Databus1: track 0.00 -> 5.84 mm
Other:
- board text added: "0"
- board text added: "2025 DGK"
- board text added: "3 LevelA 0"
- board text added: "3 LevelB 0"
- board text added: "3 LevelC 0"
- board text added: "HC4_CPU Rev 2.0"
- board text added: "LSB"
- board text added: "MSB"
- board text added: "RAM_Address"

Commit message: 配線完了とみられる
Parts:
- moved IC11 1.91 mm to (86.4, 108.0)
- moved CP11 1.77 mm to (80.0, 104.9)
- moved TP20 0.18 mm to (70.3, 91.4)
Routing:
- net GND: track 9.00 -> 879.1 mm, vias 0 -> 78
- net VCC: track 4.52 -> 620.2 mm, vias 0 -> 20
- net /Address BUS/Instruction_7: track 0.00 -> 179.1 mm, vias 0 -> 6
- net /ALU/ALU_in_B1: track 0.00 -> 178.1 mm, vias 0 -> 9
- net /Data BUS/Databus3: track 7.93 -> 175.9 mm, vias 0 -> 8
- net /Data BUS/Databus2: track 9.83 -> 176.5 mm, vias 0 -> 6
- net /Instruction Decoder/~{Carry_EN}: track 0.00 -> 162.3 mm, vias 0 -> 9
- net /ALU/I2a: track 26.4 -> 184.0 mm, vias 0 -> 8
- net /Address BUS/Instruction_0: track 0.00 -> 157.5 mm, vias 0 -> 4
- net ~{RESET}: track 0.00 -> 155.6 mm, vias 0 -> 14
- net /Data BUS/Databus0: track 7.83 -> 158.9 mm, vias 0 -> 9
- net /ALU/I3a: track 26.4 -> 174.0 mm, vias 0 -> 7
- net /Data BUS/Databus1: track 5.84 -> 152.8 mm, vias 0 -> 9
- net /ALU/Carry_IN: track 26.4 -> 171.7 mm, vias 0 -> 5
- net CLK: track 0.00 -> 143.8 mm, vias 0 -> 9
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- added copper zone on B.Cu, net GND
- added copper zone on F.Cu, net GND
