File: HC4_KiCad/alu.kicad_sch (KiCad schematic)
At the start: 5 parts, among them U1 74HC153, U2 74HC153, U3 74HC153, U4 74HC153, U5 74HC283

Commit message: 進捗コミット
Parts:
- added CP1, CP2, CP3, CP4, CP5: C_Byp, symbol Device2:C_Bypass
- renumbered U1 to IC3, U2 to IC4, U3 to IC5, U4 to IC6, U5 to IC7
Connections:
- net GND: now also IC3.1 (Ea), IC3.6 (I0a), IC4.1 (Ea), IC4.6 (I0a), IC5.1 (Ea), IC5.6 (I0a), IC6.1 (Ea), IC6.6 (I0a), CP1.2, CP2.2, CP3.2, CP4.2, CP5.2
- net VCC: now also CP1.1, CP2.1, CP3.1, CP4.1, CP5.1
- net Sub: now reaches IC6.10 (I0b)
- net Sub: now also IC3.10 (I0b), IC3.12 (I2b), IC4.10 (I0b), IC4.12 (I2b), IC5.10 (I0b), IC5.12 (I2b), IC6.12 (I2b)
- net ~{Sub}: now reaches IC6.11 (I1b)
- net ~{Sub}: now also IC3.11 (I1b), IC3.13 (I3b), IC4.11 (I1b), IC4.13 (I3b), IC5.11 (I1b), IC5.13 (I3b), IC6.13 (I3b)
- net ALU_~{Eb}: now reaches IC6.15 (Eb)
- net ALU_~{Eb}: now also IC3.15 (Eb), IC4.15 (Eb), IC5.15 (Eb)
- net I3a: now reaches IC6.3 (I3a)
- net I3a: now also IC3.3 (I3a), IC4.3 (I3a), IC5.3 (I3a)
- net I2a: now reaches IC6.4 (I2a)
- net I2a: now also IC3.4 (I2a), IC4.4 (I2a), IC5.4 (I2a)
- net I1a: now reaches IC6.5 (I1a)
- net I1a: now also IC3.5 (I1a), IC4.5 (I1a), IC5.5 (I1a)

Commit message: 進捗コミット2
Connections:
- net Sub is gone; now on net GND: IC3.10 (I0b), IC3.12 (I2b), IC4.10 (I0b), IC4.12 (I2b), IC5.10 (I0b), IC5.12 (I2b), IC6.10 (I0b), IC6.12 (I2b)
- net ~{Sub} is gone; now on net VCC: IC3.11 (I1b), IC3.13 (I3b), IC4.11 (I1b), IC4.13 (I3b), IC5.11 (I1b), IC5.13 (I3b), IC6.11 (I1b), IC6.13 (I3b)
- net GND: no longer IC3.6 (I0a), IC4.6 (I0a), IC5.6 (I0a), IC6.6 (I0a)
- new net I0a: IC3.6 (I0a), IC4.6 (I0a), IC5.6 (I0a), IC6.6 (I0a)

Commit message: I'm tired. あとは任せた　頑張りたまえ
Parts:
- CP1, CP2, CP3, CP4, CP5: value C_Byp -> 0.1u; footprint (none) -> Capacitor_THT:C_Disc_D3.0mm_W1.6mm_P2.50mm
Other:
- title: (none) -> CPU
Changed lines of the file:
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@@
 	(generator_version "8.0")
 	(paper "A4")
+	(title_block
+		(title "CPU")
+		(date "2025-02-09")
+		(rev "1.0")
+	)
 	(junction
 		(at 55.88 44.45)
@@
 		(dnp no)
 		(fields_autoplaced yes)
-		(property "Reference" "#PWR022"
+		(property "Reference" "#PWR025"
 			(at 191.77 73.66 0)
 			(effects
@@
 			(project "HC4_KiCad"
 				(path "/33731ded-38c0-4297-bdd8-92b082f46ff8/51fb15b9-2319-4d69-a07a-a04158a23ae2"
-					(reference "#PWR022")
+					(reference "#PWR025")
 					(unit 1)
 				)
@@
 			)
 		)
-		(property "Value" "C_Byp"
+		(property "Value" "0.1u"
 			(at 80.01 172.7199 0)
 			(effects
@@
 			)
 		)
-		(property "Footprint" ""
+		(property "Footprint" "Capacitor_THT:C_Disc_D3.0mm_W1.6mm_P2.50mm"
 			(at 77.1652 175.26 0)
 			(effects
@@
 			)
 		)
-		(property "Value" "C_Byp"
+		(property "Value" "0.1u"
 			(at 92.71 172.7199 0)
 			(effects
@@
 			)
 		)
-		(property "Footprint" ""
+		(property "Footprint" "Capacitor_THT:C_Disc_D3.0mm_W1.6mm_P2.50mm"
 			(at 89.8652 175.26 0)
 			(effects
@@
 		(dnp no)
 		(fields_autoplaced yes)
-		(property "Reference" "#PWR013"
+		(property "Reference" "#PWR016"
 			(at 50.8 170.18 0)
 			(effects
@@
 			(project "HC4_KiCad"
 				(path "/33731ded-38c0-4297-bdd8-92b082f46ff8/51fb15b9-2319-4d69-a07a-a04158a23ae2"
-					(reference "#PWR013")
+					(reference "#PWR016")
 					(unit 1)
 				)
@@
 		(dnp no)
 		(fields_autoplaced yes)
-		(property "Reference" "#PWR015"
+		(property "Reference" "#PWR018"
 			(at 55.88 46.99 0)
 			(effects
@@
 			(project ""
 				(path "/33731ded-38c0-4297-bdd8-92b082f46ff8/51fb15b9-2319-4d69-a07a-a04158a23ae2"
-					(reference "#PWR015")
+					(reference "#PWR018")
 					(unit 1)
 				)
@@
 		(dnp no)
 		(fields_autoplaced yes)
-		(property "Reference" "#PWR021"
+		(property "Reference" "#PWR024"
 			(at 187.96 80.01 0)
 			(effects
@@
 			(project "HC4_KiCad"
 				(path "/33731ded-38c0-4297-bdd8-92b082f46ff8/51fb15b9-2319-4d69-a07a-a04158a23ae2"
-					(reference "#PWR021")
+					(reference "#PWR024")
 					(unit 1)
 				)
@@
 		(on_board yes)
 		(dnp no)
-		(property "Reference" "#PWR014"
+		(property "Reference" "#PWR017"
 			(at 50.8 182.88 0)
 			(effects
@@
 			(project "HC4_KiCad"
 				(path "/33731ded-38c0-4297-bdd8-92b082f46ff8/51fb15b9-2319-4d69-a07a-a04158a23ae2"
-					(reference "#PWR014")
+					(reference "#PWR017")
 					(unit 1)
 				)
@@
 			)
 		)
-		(property "Value" "C_Byp"
+		(property "Value" "0.1u"
 			(at 54.61 172.7199 0)
 			(effects
@@
 			)
 		)
-		(property "Footprint" ""
+		(property "Footprint" "Capacitor_THT:C_Disc_D3.0mm_W1.6mm_P2.50mm"
 			(at 51.7652 175.26 0)
 			(effects
@@
 		(dnp no)
 		(fields_autoplaced yes)
-		(property "Reference" "#PWR016"
+		(property "Reference" "#PWR019"
 			(at 55.88 135.89 0)
 			(effects
@@
 			(project ""
 				(path "/33731ded-38c0-4297-bdd8-92b082f46ff8/51fb15b9-2319-4d69-a07a-a04158a23ae2"
-					(reference "#PWR016")
+					(reference "#PWR019")
 					(unit 1)
 				)
@@
 		(dnp no)
 		(fields_autoplaced yes)
-		(property "Reference" "#PWR019"
+		(property "Reference" "#PWR022"
 			(at 137.16 80.01 0)
 			(effects
@@
 			(project "HC4_KiCad"
 				(path "/33731ded-38c0-4297-bdd8-92b082f46ff8/51fb15b9-2319-4d69-a07a-a04158a23ae2"
-					(reference "#PWR019")
+					(reference "#PWR022")
 					(unit 1)
 				)
@@
 			)
 		)
-		(property "Value" "C_Byp"
+		(property "Value" "0.1u"
 			(at 105.41 172.7199 0)
 			(effects
@@
 			)
 		)
-		(property "Footprint" ""
+		(property "Footprint" "Capacitor_THT:C_Disc_D3.0mm_W1.6mm_P2.50mm"
 			(at 102.5652 175.26 0)
 			(effects
@@
 			)
 		)
-		(property "Value" "C_Byp"
+		(property "Value" "0.1u"
 			(at 67.31 172.7199 0)
 			(effects
@@
 			)
 		)
-		(property "Footprint" ""
+		(property "Footprint" "Capacitor_THT:C_Disc_D3.0mm_W1.6mm_P2.50mm"
 			(at 64.4652 175.26 0)
 			(effects
@@
 		(dnp no)
 		(fields_autoplaced yes)
-		(property "Reference" "#PWR011"
+		(property "Reference" "#PWR014"
 			(at 35.56 80.01 0)
 			(effects
@@
 			(project "HC4_KiCad"
 				(path "/33731ded-38c0-4297-bdd8-92b082f46ff8/51fb15b9-2319-4d69-a07a-a04158a23ae2"
-					(reference "#PWR011")
+					(reference "#PWR014")
 					(unit 1)
 				)
@@
 		(dnp no)
 		(fields_autoplaced yes)
-		(property "Reference" "#PWR020"
+		(property "Reference" "#PWR023"
 			(at 140.97 73.66 0)
 			(effects
@@
 			(project "HC4_KiCad"
 				(path "/33731ded-38c0-4297-bdd8-92b082f46ff8/51fb15b9-2319-4d69-a07a-a04158a23ae2"
-					(reference "#PWR020")
+					(reference "#PWR023")
 					(unit 1)
 				)
@@
 		(dnp no)
 		(fields_autoplaced yes)
-		(property "Reference" "#PWR017"
+		(property "Reference" "#PWR020"
 			(at 86.36 80.01 0)
 			(effects
@@
 			(project ""
 				(path "/33731ded-38c0-4297-bdd8-92b082f46ff8/51fb15b9-2319-4d69-a07a-a04158a23ae2"
-					(reference "#PWR017")
+					(reference "#PWR020")
 					(unit 1)
 				)
@@
 		(dnp no)
 		(fields_autoplaced yes)
-		(property "Reference" "#PWR012"
+		(property "Reference" "#PWR015"
 			(at 39.37 73.66 0)
 			(effects
@@
 			(project "HC4_KiCad"
 				(path "/33731ded-38c0-4297-bdd8-92b082f46ff8/51fb15b9-2319-4d69-a07a-a04158a23ae2"
-					(reference "#PWR012")
+					(reference "#PWR015")
 					(unit 1)
 				)
@@
 		(dnp no)
 		(fields_autoplaced yes)
-		(property "Reference" "#PWR018"
+		(property "Reference" "#PWR021"
 			(at 90.17 73.66 0)
 			(effects
@@
 			(project ""
 				(path "/33731ded-38c0-4297-bdd8-92b082f46ff8/51fb15b9-2319-4d69-a07a-a04158a23ae2"
-					(reference "#PWR018")
+					(reference "#PWR021")
 					(unit 1)
 				)

Commit message: フットプリントの割り当て修正
Parts:
- IC3, IC4, IC5, IC6, IC7: footprint (none) -> Package_DIP:DIP-16_W7.62mm_Socket
Changed lines of the file:
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@@
 	(label "Internal_A1"
 		(at 234.95 60.96 0)
+		(fields_autoplaced yes)
 		(effects
 			(font
@@
 	(label "Internal_A2"
 		(at 130.81 53.34 180)
+		(fields_autoplaced yes)
 		(effects
 			(font
@@
 	(label "ALU_OUT1"
 		(at 280.67 55.88 180)
+		(fields_autoplaced yes)
 		(effects
 			(font
@@
 	(label "Internal_B3"
 		(at 80.01 71.12 180)
+		(fields_autoplaced yes)
 		(effects
 			(font
@@
 	(label "Internal_A0"
 		(at 234.95 58.42 0)
+		(fields_autoplaced yes)
 		(effects
 			(font
@@
 	(label "Internal_B3"
 		(at 234.95 78.74 0)
+		(fields_autoplaced yes)
 		(effects
 			(font
@@
 	(label "Internal_A2"
 		(at 234.95 63.5 0)
+		(fields_autoplaced yes)
 		(effects
 			(font
@@
 	(label "ALU_in_A1"
 		(at 135.89 88.9 0)
+		(fields_autoplaced yes)
 		(effects
 			(font
@@
 	(label "Internal_B2"
 		(at 234.95 76.2 0)
+		(fields_autoplaced yes)
 		(effects
 			(font
@@
 	(label "ALU_in_A2"
 		(at 85.09 88.9 0)
+		(fields_autoplaced yes)
 		(effects
 			(font
@@
 	(label "ALU_in_A3"
 		(at 34.29 88.9 0)
+		(fields_autoplaced yes)
 		(effects
 			(font
@@
 	(label "ALU_in_B2"
 		(at 85.09 91.44 0)
+		(fields_autoplaced yes)
 		(effects
 			(font
@@
 	(label "ALU_in_B0"
 		(at 186.69 91.44 0)
+		(fields_autoplaced yes)
 		(effects
 			(font
@@
 	(label "Internal_B2"
 		(at 130.81 71.12 180)
+		(fields_autoplaced yes)
 		(effects
 			(font
@@
 	(label "ALU_in_B3"
 		(at 34.29 91.44 0)
+		(fields_autoplaced yes)
 		(effects
 			(font
@@
 	(label "Internal_A1"
 		(at 181.61 53.34 180)
+		(fields_autoplaced yes)
 		(effects
 			(font
@@
 	(label "Internal_B0"
 		(at 232.41 71.12 180)
+		(fields_autoplaced yes)
 		(effects
 			(font
@@
 	(label "ALU_OUT0"
 		(at 280.67 53.34 180)
+		(fields_autoplaced yes)
 		(effects
 			(font
@@
 	(label "Internal_B0"
 		(at 234.95 71.12 0)
+		(fields_autoplaced yes)
 		(effects
 			(font
@@
 	(label "Internal_A3"
 		(at 80.01 53.34 180)
+		(fields_autoplaced yes)
 		(effects
 			(font
@@
 	(label "Internal_B1"
 		(at 181.61 71.12 180)
+		(fields_autoplaced yes)
 		(effects
 			(font
@@
 	(label "Internal_B1"
 		(at 234.95 73.66 0)
+		(fields_autoplaced yes)
 		(effects
 			(font
@@
 	(label "Internal_A3"
 		(at 234.95 66.04 0)
+		(fields_autoplaced yes)
 		(effects
 			(font
@@
 	(label "ALU_in_A0"
 		(at 186.69 88.9 0)
+		(fields_autoplaced yes)
 		(effects
 			(font
@@
 	(label "Internal_A0"
 		(at 232.41 53.34 180)
+		(fields_autoplaced yes)
 		(effects
 			(font
@@
 	(label "ALU_in_B1"
 		(at 135.89 91.44 0)
+		(fields_autoplaced yes)
 		(effects
 			(font
@@
 	(label "ALU_OUT3"
 		(at 280.67 60.96 180)
+		(fields_autoplaced yes)
 		(effects
 			(font
@@
 	(label "ALU_OUT2"
 		(at 280.67 58.42 180)
+		(fields_autoplaced yes)
 		(effects
 			(font
@@
 		(shape input)
 		(at 191.77 55.88 180)
+		(fields_autoplaced yes)
 		(effects
 			(font
@@
 		(shape input)
 		(at 191.77 53.34 180)
+		(fields_autoplaced yes)
 		(effects
 			(font
@@
 		(shape input)
 		(at 90.17 53.34 180)
+		(fields_autoplaced yes)
 		(effects
 			(font
@@
 		(shape input)
 		(at 191.77 58.42 180)
+		(fields_autoplaced yes)
 		(effects
 			(font
@@
 		(shape input)
 		(at 90.17 60.96 180)
+		(fields_autoplaced yes)
 		(effects
 			(font
@@
 		(shape input)
 		(at 140.97 55.88 180)
+		(fields_autoplaced yes)
 		(effects
 			(font
@@
 		(shape input)
 		(at 194.31 83.82 180)
+		(fields_autoplaced yes)
 		(effects
 			(font
@@
 		(shape input)
 		(at 194.31 83.82 180)
+		(fields_autoplaced yes)
 		(effects
 			(font
@@
 		(shape input)
 		(at 143.51 83.82 180)
+		(fields_autoplaced yes)
 		(effects
 			(font
@@
 		(shape output)
 		(at 275.59 69.85 270)
+		(fields_autoplaced yes)
 		(effects
 			(font
@@
 		(shape input)
 		(at 39.37 60.96 180)
+		(fields_autoplaced yes)
 		(effects
 			(font
@@
 		(shape input)
 		(at 140.97 58.42 180)
+		(fields_autoplaced yes)
 		(effects
 			(font
@@
 		(shape input)
 		(at 92.71 83.82 180)
+		(fields_autoplaced yes)
 		(effects
 			(font
@@
 		(shape output)
 		(at 283.21 69.85 270)
+		(fields_autoplaced yes)
 		(effects
 			(font
@@
 		(shape input)
 		(at 41.91 83.82 180)
+		(fields_autoplaced yes)
 		(effects
 			(font
@@
 		(shape input)
 		(at 92.71 83.82 180)
+		(fields_autoplaced yes)
 		(effects
 			(font
@@
 		(shape input)
 		(at 39.37 53.34 180)
+		(fields_autoplaced yes)
 		(effects
 			(font
@@
 		(shape input)
 		(at 143.51 83.82 180)
+		(fields_autoplaced yes)
 		(effects
 			(font
@@
 		(shape input)
 		(at 27.94 100.33 180)
+		(fields_autoplaced yes)
 		(effects
 			(font
@@
 		(shape input)
 		(at 90.17 58.42 180)
+		(fields_autoplaced yes)
 		(effects
 			(font
@@
 		(shape input)
 		(at 191.77 60.96 180)
+		(fields_autoplaced yes)
 		(effects
 			(font
@@
 		(shape input)
 		(at 90.17 55.88 180)
+		(fields_autoplaced yes)
 		(effects
 			(font
@@
 		(shape input)
 		(at 245.11 53.34 180)
+		(fields_autoplaced yes)
 		(effects
 			(font
@@
 		(shape input)
 		(at 39.37 55.88 180)
+		(fields_autoplaced yes)
 		(effects
 			(font
@@
 		(shape input)
 		(at 140.97 53.34 180)
+		(fields_autoplaced yes)
 		(effects
 			(font
@@
 		(shape input)
 		(at 140.97 60.96 180)
+		(fields_autoplaced yes)
 		(effects
 			(font
@@
 		(shape input)
 		(at 39.37 58.42 180)
+		(fields_autoplaced yes)
 		(effects
 			(font
@@
 		(shape input)
 		(at 30.48 102.87 180)
+		(fields_autoplaced yes)
 		(effects
 			(font
@@
 			)
 		)
-		(property "Footprint" ""
+		(property "Footprint" "Package_DIP:DIP-16_W7.62mm_Socket"
 			(at 208.28 71.12 0)
 			(effects
@@
 			)
 		)
-		(property "Footprint" ""
+		(property "Footprint" "Package_DIP:DIP-16_W7.62mm_Socket"
 			(at 157.48 71.12 0)
 			(effects
@@
 			)
 		)
-		(property "Footprint" ""
+		(property "Footprint" "Package_DIP:DIP-16_W7.62mm_Socket"
 			(at 259.08 66.04 0)
 			(effects
@@
 			)
 		)
-		(property "Footprint" ""
+		(property "Footprint" "Package_DIP:DIP-16_W7.62mm_Socket"
 			(at 106.68 71.12 0)
 			(effects
@@
 			)
 		)
-		(property "Footprint" ""
+		(property "Footprint" "Package_DIP:DIP-16_W7.62mm_Socket"
 			(at 55.88 71.12 0)
 			(effects

Commit message: ICの配置を再検討
Parts:
- renumbered CP1 to CP3, CP2 to CP4, CP3 to CP5, CP4 to CP6, CP5 to CP7
Changed lines of the file:
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@@
 	(label "Internal_A1"
 		(at 234.95 60.96 0)
-		(fields_autoplaced yes)
 		(effects
 			(font
@@
 	(label "Internal_A2"
 		(at 130.81 53.34 180)
-		(fields_autoplaced yes)
 		(effects
 			(font
@@
 	(label "ALU_OUT1"
 		(at 280.67 55.88 180)
-		(fields_autoplaced yes)
 		(effects
 			(font
@@
 	(label "Internal_B3"
 		(at 80.01 71.12 180)
-		(fields_autoplaced yes)
 		(effects
 			(font
@@
 	(label "Internal_A0"
 		(at 234.95 58.42 0)
-		(fields_autoplaced yes)
 		(effects
 			(font
@@
 	(label "Internal_B3"
 		(at 234.95 78.74 0)
-		(fields_autoplaced yes)
 		(effects
 			(font
@@
 	(label "Internal_A2"
 		(at 234.95 63.5 0)
-		(fields_autoplaced yes)
 		(effects
 			(font
@@
 	(label "ALU_in_A1"
 		(at 135.89 88.9 0)
-		(fields_autoplaced yes)
 		(effects
 			(font
@@
 	(label "Internal_B2"
 		(at 234.95 76.2 0)
-		(fields_autoplaced yes)
 		(effects
 			(font
@@
 	(label "ALU_in_A2"
 		(at 85.09 88.9 0)
-		(fields_autoplaced yes)
 		(effects
 			(font
@@
 	(label "ALU_in_A3"
 		(at 34.29 88.9 0)
-		(fields_autoplaced yes)
 		(effects
 			(font
@@
 	(label "ALU_in_B2"
 		(at 85.09 91.44 0)
-		(fields_autoplaced yes)
 		(effects
 			(font
@@
 	(label "ALU_in_B0"
 		(at 186.69 91.44 0)
-		(fields_autoplaced yes)
 		(effects
 			(font
@@
 	(label "Internal_B2"
 		(at 130.81 71.12 180)
-		(fields_autoplaced yes)
 		(effects
 			(font
@@
 	(label "ALU_in_B3"
 		(at 34.29 91.44 0)
-		(fields_autoplaced yes)
 		(effects
 			(font
@@
 	(label "Internal_A1"
 		(at 181.61 53.34 180)
-		(fields_autoplaced yes)
 		(effects
 			(font
@@
 	(label "Internal_B0"
 		(at 232.41 71.12 180)
-		(fields_autoplaced yes)
 		(effects
 			(font
@@
 	(label "ALU_OUT0"
 		(at 280.67 53.34 180)
-		(fields_autoplaced yes)
 		(effects
 			(font
@@
 	(label "Internal_B0"
 		(at 234.95 71.12 0)
-		(fields_autoplaced yes)
 		(effects
 			(font
@@
 	(label "Internal_A3"
 		(at 80.01 53.34 180)
-		(fields_autoplaced yes)
 		(effects
 			(font
@@
 	(label "Internal_B1"
 		(at 181.61 71.12 180)
-		(fields_autoplaced yes)
 		(effects
 			(font
@@
 	(label "Internal_B1"
 		(at 234.95 73.66 0)
-		(fields_autoplaced yes)
 		(effects
 			(font
@@
 	(label "Internal_A3"
 		(at 234.95 66.04 0)
-		(fields_autoplaced yes)
 		(effects
 			(font
@@
 	(label "ALU_in_A0"
 		(at 186.69 88.9 0)
-		(fields_autoplaced yes)
 		(effects
 			(font
@@
 	(label "Internal_A0"
 		(at 232.41 53.34 180)
-		(fields_autoplaced yes)
 		(effects
 			(font
@@
 	(label "ALU_in_B1"
 		(at 135.89 91.44 0)
-		(fields_autoplaced yes)
 		(effects
 			(font
@@
 	(label "ALU_OUT3"
 		(at 280.67 60.96 180)
-		(fields_autoplaced yes)
 		(effects
 			(font
@@
 	(label "ALU_OUT2"
 		(at 280.67 58.42 180)
-		(fields_autoplaced yes)
 		(effects
 			(font
@@
 		(shape input)
 		(at 191.77 55.88 180)
-		(fields_autoplaced yes)
 		(effects
 			(font
@@
 		(shape input)
 		(at 191.77 53.34 180)
-		(fields_autoplaced yes)
 		(effects
 			(font
@@
 		(shape input)
 		(at 90.17 53.34 180)
-		(fields_autoplaced yes)
 		(effects
 			(font
@@
 		(shape input)
 		(at 191.77 58.42 180)
-		(fields_autoplaced yes)
 		(effects
 			(font
@@
 		(shape input)
 		(at 90.17 60.96 180)
-		(fields_autoplaced yes)
 		(effects
 			(font
@@
 		(shape input)
 		(at 140.97 55.88 180)
-		(fields_autoplaced yes)
 		(effects
 			(font
@@
 		(shape input)
 		(at 194.31 83.82 180)
-		(fields_autoplaced yes)
 		(effects
 			(font
@@
 		(shape input)
 		(at 194.31 83.82 180)
-		(fields_autoplaced yes)
 		(effects
 			(font
@@
 		(shape input)
 		(at 143.51 83.82 180)
-		(fields_autoplaced yes)
 		(effects
 			(font
@@
 		(shape output)
 		(at 275.59 69.85 270)
-		(fields_autoplaced yes)
 		(effects
 			(font
@@
 		(shape input)
 		(at 39.37 60.96 180)
-		(fields_autoplaced yes)
 		(effects
 			(font
@@
 		(shape input)
 		(at 140.97 58.42 180)
-		(fields_autoplaced yes)
 		(effects
 			(font
@@
 		(shape input)
 		(at 92.71 83.82 180)
-		(fields_autoplaced yes)
 		(effects
 			(font
@@
 		(shape output)
 		(at 283.21 69.85 270)
-		(fields_autoplaced yes)
 		(effects
 			(font
@@
 		(shape input)
 		(at 41.91 83.82 180)
-		(fields_autoplaced yes)
 		(effects
 			(font
@@
 		(shape input)
 		(at 92.71 83.82 180)
-		(fields_autoplaced yes)
 		(effects
 			(font
@@
 		(shape input)
 		(at 39.37 53.34 180)
-		(fields_autoplaced yes)
 		(effects
 			(font
@@
 		(shape input)
 		(at 143.51 83.82 180)
-		(fields_autoplaced yes)
 		(effects
 			(font
@@
 		(shape input)
 		(at 27.94 100.33 180)
-		(fields_autoplaced yes)
 		(effects
 			(font
@@
 		(shape input)
 		(at 90.17 58.42 180)
-		(fields_autoplaced yes)
 		(effects
 			(font
@@
 		(shape input)
 		(at 191.77 60.96 180)
-		(fields_autoplaced yes)
 		(effects
 			(font
@@
 		(shape input)
 		(at 90.17 55.88 180)
-		(fields_autoplaced yes)
 		(effects
 			(font
@@
 		(shape input)
 		(at 245.11 53.34 180)
-		(fields_autoplaced yes)
 		(effects
 			(font
@@
 		(shape input)
 		(at 39.37 55.88 180)
-		(fields_autoplaced yes)
 		(effects
 			(font
@@
 		(shape input)
 		(at 140.97 53.34 180)
-		(fields_autoplaced yes)
 		(effects
 			(font
@@
 		(shape input)
 		(at 140.97 60.96 180)
-		(fields_autoplaced yes)
 		(effects
 			(font
@@
 		(shape input)
 		(at 39.37 58.42 180)
-		(fields_autoplaced yes)
 		(effects
 			(font
@@
 		(shape input)
 		(at 30.48 102.87 180)
-		(fields_autoplaced yes)
 		(effects
 			(font
@@
 		(dnp no)
 		(fields_autoplaced yes)
-		(property "Reference" "CP3"
+		(property "Reference" "CP5"
 			(at 80.01 170.1799 0)
 			(effects
@@
 			(project "HC4_KiCad"
 				(path "/33731ded-38c0-4297-bdd8-92b082f46ff8/51fb15b9-2319-4d69-a07a-a04158a23ae2"
-					(reference "CP3")
+					(reference "CP5")
 					(unit 1)
 				)
@@
 		(dnp no)
 		(fields_autoplaced yes)
-		(property "Reference" "CP4"
+		(property "Reference" "CP6"
 			(at 92.71 170.1799 0)
 			(effects
@@
 			(project "HC4_KiCad"
 				(path "/33731ded-38c0-4297-bdd8-92b082f46ff8/51fb15b9-2319-4d69-a07a-a04158a23ae2"
-					(reference "CP4")
+					(reference "CP6")
 					(unit 1)
 				)
@@
 		(dnp no)
 		(fields_autoplaced yes)
-		(property "Reference" "CP1"
+		(property "Reference" "CP3"
 			(at 54.61 170.1799 0)
 			(effects
@@
 			(project ""
 				(path "/33731ded-38c0-4297-bdd8-92b082f46ff8/51fb15b9-2319-4d69-a07a-a04158a23ae2"
-					(reference "CP1")
+					(reference "CP3")
 					(unit 1)
 				)
@@
 		(dnp no)
 		(fields_autoplaced yes)
-		(property "Reference" "CP5"
+		(property "Reference" "CP7"
 			(at 105.41 170.1799 0)
 			(effects
@@
 			(project "HC4_KiCad"
 				(path "/33731ded-38c0-4297-bdd8-92b082f46ff8/51fb15b9-2319-4d69-a07a-a04158a23ae2"
-					(reference "CP5")
+					(reference "CP7")
 					(unit 1)
 				)
@@
 		(dnp no)
 		(fields_autoplaced yes)
-		(property "Reference" "CP2"
+		(property "Reference" "CP4"
 			(at 67.31 170.1799 0)
 			(effects
@@
 			(project "HC4_KiCad"
 				(path "/33731ded-38c0-4297-bdd8-92b082f46ff8/51fb15b9-2319-4d69-a07a-a04158a23ae2"
-					(reference "CP2")
+					(reference "CP4")
 					(unit 1)
 				)
