File: HC4_KiCad/instructiondecode.kicad_sch (KiCad schematic)
At the start: 4 parts, among them IC17 74HC74, IC18 74HC273, IC19 74HC4053, IC20 74HC151

Commit message: 進捗コミット2
Parts:
- removed IC18: 74HC273, symbol 74xx_2:74HC273
- added D10, D3, D4, D5, D6, D7, D8, D9: D, symbol Device:D
- added IC17: 74HC04, symbol 74xx_2:74HC04
- renumbered IC17 to IC18
Connections:
- net Instruction_0: now also IC19.10 (B), IC17.1
- net Instruction_1: now also IC17.3
- net Instruction_2: now also IC17.5
- net Instruction_3: now also IC17.9
- net VCC: now also IC18.4 (~{S})
- net ~{JMP}: now also IC20.7 (~{E})
- net ~{RESET}: now also IC18.1 (~{R})
- net ~{CLK} renamed CLK
- new net: D10.1 (K), D7.1 (K), D8.1 (K), D9.1 (K)
- new net: D3.1 (K), D4.1 (K), D5.1 (K), D6.1 (K)

Commit message: I'm tired. あとは任せた　頑張りたまえ
Parts:
- removed unit 5 of IC17
- added CP16, CP17, CP18, CP19, CP20, CP21: 0.1u, Capacitor_THT:C_Disc_D3.0mm_W1.6mm_P2.50mm, symbol Device2:C_Bypass
- added D11, D12, D13, D14, D15, D16, D17, D18, D19, D20, D21, D22, D23, D24, D25, D26, D27, D28, D29, D30, D31, D32, D33, D34, D35, D36, D37, D38, D39, D40, D41, D42, D43, D44, D45, D6: D, Diode_THT:D_DO-35_SOD27_P2.54mm_Vertical_AnodeUp, symbol Device:D
- added IC10: 74HC4002, symbol 74xx_2:74HC4002
- added IC18: 74HC00, symbol 74xx_2:74HC00
- added unit 3 of IC21
- added IC23: 74HC32, symbol 74xx_2:74HC32
- added R3, R4, R5: 10k, Resistor_THT:R_Axial_DIN0207_L6.3mm_D2.5mm_P7.62mm_Horizontal, symbol Device:R
- added RN6: 10k, Resistor_THT:R_Array_SIP9, symbol Device:R_Network08_Split
- D10, D7, D8, D9: footprint (none) -> Diode_THT:D_DO-35_SOD27_P2.54mm_Vertical_AnodeUp
- D2: renamed from D3; footprint (none) -> Diode_THT:D_DO-35_SOD27_P2.54mm_Vertical_AnodeUp
- D3: renamed from D4; footprint (none) -> Diode_THT:D_DO-35_SOD27_P2.54mm_Vertical_AnodeUp
- D4: renamed from D5; footprint (none) -> Diode_THT:D_DO-35_SOD27_P2.54mm_Vertical_AnodeUp
- D5: renamed from D6; footprint (none) -> Diode_THT:D_DO-35_SOD27_P2.54mm_Vertical_AnodeUp
- renumbered IC18 to IC19, IC19 to IC20, IC17 to IC21, IC20 to IC22
Connections:
- net Oprand_0 is gone; now on net Instruction_2: IC22.11 (S0)
- net Oprand_1 is gone; now on net Instruction_1: IC22.10 (S1)
- net Oprand_2 is gone; now on net Instruction_0: IC22.9 (S2)
- net CLK: now also IC19.3 (C)
- net GND: now also IC20.9 (C), IC21.7 (GND), IC22.12 (I7), IC22.13 (I6), CP16.2, CP17.2, CP18.2, CP19.2, CP20.2, CP21.2, IC10.7 (VSS), IC23.7 (GND)
- net Instruction_0: no longer IC21.1
- net Instruction_1: no longer IC21.3
- net Instruction_2: no longer IC21.5
- net Instruction_3: no longer IC21.9
- net Instruction_4: now also IC21.11, D25.2 (A), D33.2 (A), IC23.12
- net Instruction_5: now also D8.2 (A), IC21.3, D12.2 (A), D24.2 (A), D28.2 (A), D36.2 (A), IC18.12
- net Instruction_6: now also IC21.13, D11.2 (A), D19.2 (A), D27.2 (A), D35.2 (A)
- net Instruction_7: now also D10.2 (A), IC21.1, D38.2 (A), D6.2 (A), IC23.1
- net VCC: now also IC21.14 (VCC), CP16.1, CP17.1, CP18.1, CP19.1, CP20.1, CP21.1, IC10.14 (VDD), IC23.14 (VCC), R3.1, R4.1, R5.1, RN6.1 (R1), RN6.1 (R1), RN6.1 (R1), RN6.1 (R1), RN6.1 (R1), RN6.1 (R1), RN6.1 (R1), RN6.1 (R1)
- net ~{JMP}: no longer IC22.7 (~{E})
- net at D7.1 (K), D8.1 (K), D9.1 (K): now also IC21.9, D6.1 (K), RN6.3 (R2.2); no longer D10.1 (K)
- net at D7.2 (A): now also D3.2 (A), IC21.12, D15.2 (A), D23.2 (A), D31.2 (A), D39.2 (A), D43.2 (A), IC18.13
- net at D2.1 (K), D3.1 (K), D4.1 (K)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: now also IC23.2, RN6.2 (R1.2)
- net ~{Zero_Flg}: now reaches IC22.14 (I5)
- net ~{Zero_Flg}: now also IC19.6 (~{Q})
- net Zero_Flg: now reaches IC22.15 (I4)
- net Zero_Flg: now also IC19.5 (Q), IC20.1 (Y1)
- net at IC19.2 (D): now also IC20.15 (Y)
- net at D4.2 (A): now also IC21.4, D16.2 (A), D20.2 (A), D40.2 (A), D44.2 (A), IC23.9
- net at IC21.2: now also D42.2 (A), IC23.4
- net ALU_~{Eb}: now reaches IC20.11 (A)
- net ALU_~{Eb}: now also IC18.11
- net BUS_Zero: now reaches IC20.2 (Y0)
- new net: D42.1 (K), D43.1 (K), D44.1 (K), D45.1 (K), IC18.10, IC18.9, R5.2
- new net: D30.1 (K), D31.1 (K), D32.1 (K), D33.1 (K), IC23.10, RN6.9 (R8.2)
- new net: D34.1 (K), D35.1 (K), D36.1 (K), D37.1 (K), IC23.13, R3.2
- new net: D10.1 (K), D11.1 (K), D12.1 (K), D13.1 (K), IC21.5, IC23.5, RN6.4 (R3.2)
- new net: D22.1 (K), D23.1 (K), D24.1 (K), D25.1 (K), IC10.10, IC10.9, RN6.7 (R6.2)
- new net: D26.1 (K), D27.1 (K), D28.1 (K), D29.1 (K), IC10.11, IC10.12, RN6.8 (R7.2)
- new net: D17.2 (A), D21.2 (A), D29.2 (A), IC21.10
- new net I0a: D18.1 (K), D19.1 (K), D20.1 (K), D21.1 (K), RN6.6 (R5.2)
- new net I1a: IC10.13
- new net I2a: IC23.8
- new net I3a: IC23.11
- new net MEMMode: D14.1 (K), D15.1 (K), D16.1 (K), D17.1 (K), RN6.5 (R4.2)
- new net READ: D38.1 (K), D39.1 (K), D40.1 (K), D41.1 (K), R4.2
- new net ~{ALU_OE}: IC23.3
- new net ~{Imm_OE}: IC21.8
- new net ~{LevelC_OE}: IC18.8
- new net ~{STACK_LE}: IC23.6
- new net ~{is_JP_inst}: IC21.6, IC22.7 (~{E})
- no-connect marks 1 -> 19
Other:
- note added: "I0a"
- note added: "I1a"
- note added: "I2a"
- note added: "I3a"
- note added: "MEMMode"
- note added: "READ"
- note added: "~{ALU_OE}"
- note added: "~{Imm_OE}"
- note added: "~{LevelC_OE}"
- note added: "~{STACK_LE}"
- note added: "~{is_JP_inst}"
- title: (none) -> CPU
- moved on the sheet: D2, D3, D4, D5, IC19A, IC19B, IC19C, IC21A, IC21B, IC21D, IC21E, IC21F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

Commit message: 回路図の修正
Parts:
- removed D2, D3, D4, D5: D, Diode_THT:D_DO-35_SOD27_P2.54mm_Vertical_AnodeUp, symbol Device:D
- removed unit 1 of IC23
- removed R3: 10k, Resistor_THT:R_Axial_DIN0207_L6.3mm_D2.5mm_P7.62mm_Horizontal, symbol Device:R
- added unit 1 of IC19
- IC18: now not fitted
- renumbered D14 to D10, D15 to D11, D16 to D12, D17 to D13, D18 to D14, D19 to D15, D20 to D16, D21 to D17, D22 to D18, D23 to D19, D6 to D2, D24 to D20, D25 to D21, D26 to D22, D27 to D23, D28 to D24, D29 to D25, D30 to D26, D31 to D27, D32 to D28, D33 to D29, D7 to D3, D34 to D30, D35 to D31, D36 to D32, D37 to D33, D38 to D34, D39 to D35, D40 to D36, D41 to D37, D42 to D38, D43 to D39, D8 to D4, D44 to D40, D45 to D41, D9 to D5, D10 to D6, D11 to D7, D12 to D8, D13 to D9, IC23 to IC19, IC19 to IC20, IC20 to IC21, IC21 to IC22, IC22 to IC23, R4 to R5, R5 to R6
Connections:
- net Instruction_7 is gone; now on net ~{ALU_OE}: D2.2 (A), D34.2 (A), D6.2 (A), IC22.1
- net Instruction_0: now also IC23.11 (S0); no longer IC23.9 (S2)
- net Instruction_2: now also IC23.9 (S2); no longer IC23.11 (S0)
- net VCC: now also IC18.10, IC18.9, IC19.1, IC19.2
- net LevelC_OE: now reaches D38.1 (K), D39.1 (K), D40.1 (K), D41.1 (K), R6.2
- net LevelC_OE: no longer IC18.10, IC18.9
- net at D30.1 (K), D31.1 (K), D32.1 (K)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: now also RN6.2 (R1.2)
- net at IC19.4, IC22.2: no longer D38.2 (A)
- net ~{LevelC_OE}: no longer names the net of IC18.8

Commit message: フットプリントの割り当て修正
Parts:
- IC10, IC18, IC20, IC22: footprint (none) -> Package_DIP:DIP-14_W7.62mm_Socket
- IC19, IC21, IC23: footprint (none) -> Package_DIP:DIP-16_W7.62mm_Socket
Changed lines of the file:
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@@
 	(label "Zero_Flg"
 		(at 52.07 140.97 0)
+		(fields_autoplaced yes)
 		(effects
 			(font
@@
 	(label "Instruction_6"
 		(at 93.98 49.53 0)
+		(fields_autoplaced yes)
 		(effects
 			(font
@@
 	(label "Instruction_1"
 		(at 105.41 173.99 0)
+		(fields_autoplaced yes)
 		(effects
 			(font
@@
 	(label "Instruction_4"
 		(at 36.83 45.72 180)
+		(fields_autoplaced yes)
 		(effects
 			(font
@@
 	(label "~{is_JP_inst}"
 		(at 157.48 133.35 90)
+		(fields_autoplaced yes)
 		(effects
 			(font
@@
 	(label "Instruction_7"
 		(at 36.83 38.1 180)
+		(fields_autoplaced yes)
 		(effects
 			(font
@@
 	(label "Instruction_2"
 		(at 105.41 176.53 0)
+		(fields_autoplaced yes)
 		(effects
 			(font
@@
 	(label "Instruction_0"
 		(at 105.41 171.45 0)
+		(fields_autoplaced yes)
 		(effects
 			(font
@@
 	(label "Carry_Flg"
 		(at 105.41 116.84 0)
+		(fields_autoplaced yes)
 		(effects
 			(font
@@
 	(label "~{Carry_Flg}"
 		(at 121.92 135.89 180)
+		(fields_autoplaced yes)
 		(effects
 			(font
@@
 	(label "Instruction_4"
 		(at 93.98 87.63 0)
+		(fields_autoplaced yes)
 		(effects
 			(font
@@
 	(label "~{Zero_Flg}"
 		(at 59.69 146.05 180)
+		(fields_autoplaced yes)
 		(effects
 			(font
@@
 	(label "ALU_~{Eb}"
 		(at 48.26 156.21 0)
+		(fields_autoplaced yes)
 		(effects
 			(font
@@
 	(label "Zero_Flg"
 		(at 107.95 158.75 0)
+		(fields_autoplaced yes)
 		(effects
 			(font
@@
 	(label "~{Zero_Flg}"
 		(at 107.95 161.29 0)
+		(fields_autoplaced yes)
 		(effects
 			(font
@@
 	(label "Instruction_0"
 		(at 48.26 158.75 0)
+		(fields_autoplaced yes)
 		(effects
 			(font
@@
 	(label "Zero_Flg"
 		(at 44.45 181.61 0)
+		(fields_autoplaced yes)
 		(effects
 			(font
@@
 	(label "Instruction_1"
 		(at 36.83 53.34 180)
+		(fields_autoplaced yes)
 		(effects
 			(font
@@
 	(label "~{Carry_Flg}"
 		(at 107.95 156.21 0)
+		(fields_autoplaced yes)
 		(effects
 			(font
@@
 	(label "Instruction_2"
 		(at 36.83 50.8 180)
+		(fields_autoplaced yes)
 		(effects
 			(font
@@
 	(label "Instruction_6"
 		(at 36.83 40.64 180)
+		(fields_autoplaced yes)
 		(effects
 			(font
@@
 	(label "ALU_~{Eb}"
 		(at 281.94 127 180)
+		(fields_autoplaced yes)
 		(effects
 			(font
@@
 	(label "Instruction_5"
 		(at 36.83 43.18 180)
+		(fields_autoplaced yes)
 		(effects
 			(font
@@
 	(label "Instruction_0"
 		(at 36.83 55.88 180)
+		(fields_autoplaced yes)
 		(effects
 			(font
@@
 	(label "~{is_JP_inst}"
 		(at 107.95 181.61 0)
+		(fields_autoplaced yes)
 		(effects
 			(font
@@
 	(label "Instruction_5"
 		(at 93.98 68.58 0)
+		(fields_autoplaced yes)
 		(effects
 			(font
@@
 	(label "Instruction_7"
 		(at 93.98 30.48 0)
+		(fields_autoplaced yes)
 		(effects
 			(font
@@
 	(label "Carry_Flg"
 		(at 107.95 153.67 0)
+		(fields_autoplaced yes)
 		(effects
 			(font
@@
 	(label "Instruction_3"
 		(at 36.83 48.26 180)
+		(fields_autoplaced yes)
 		(effects
 			(font
@@
 		(shape output)
 		(at 168.91 125.73 0)
+		(fields_autoplaced yes)
 		(effects
 			(font
@@
 		(shape output)
 		(at 261.62 115.57 270)
+		(fields_autoplaced yes)
 		(effects
 			(font
@@
 		(shape input)
 		(at 59.69 137.16 180)
+		(fields_autoplaced yes)
 		(effects
 			(font
@@
 		(shape output)
 		(at 207.01 130.81 0)
+		(fields_autoplaced yes)
 		(effects
 			(font
@@
 		(shape output)
 		(at 115.57 130.81 0)
+		(fields_autoplaced yes)
 		(effects
 			(font
@@
 		(shape output)
 		(at 228.6 130.81 0)
+		(fields_autoplaced yes)
 		(effects
 			(font
@@
 		(shape output)
 		(at 54.61 181.61 0)
+		(fields_autoplaced yes)
 		(effects
 			(font
@@
 		(shape input)
 		(at 20.32 34.29 90)
+		(fields_autoplaced yes)
 		(effects
 			(font
@@
 		(shape input)
 		(at 55.88 130.81 180)
+		(fields_autoplaced yes)
 		(effects
 			(font
@@
 		(shape output)
 		(at 138.43 110.49 270)
+		(fields_autoplaced yes)
 		(effects
 			(font
@@
 		(shape output)
 		(at 147.32 151.13 0)
+		(fields_autoplaced yes)
 		(effects
 			(font
@@
 		(shape output)
 		(at 250.19 105.41 0)
+		(fields_autoplaced yes)
 		(effects
 			(font
@@
 		(shape output)
 		(at 148.59 135.89 0)
+		(fields_autoplaced yes)
 		(effects
 			(font
@@
 		(shape output)
 		(at 281.94 128.27 270)
+		(fields_autoplaced yes)
 		(effects
 			(font
@@
 		(shape output)
 		(at 175.26 106.68 0)
+		(fields_autoplaced yes)
 		(effects
 			(font
@@
 		(shape output)
 		(at 245.11 130.81 0)
+		(fields_autoplaced yes)
 		(effects
 			(font
@@
 		(shape output)
 		(at 187.96 130.81 0)
+		(fields_autoplaced yes)
 		(effects
 			(font
@@
 			)
 		)
-		(property "Footprint" ""
+		(property "Footprint" "Package_DIP:DIP-14_W7.62mm_Socket"
 			(at 118.11 63.5 0)
 			(effects
@@
 			)
 		)
-		(property "Footprint" ""
+		(property "Footprint" "Package_DIP:DIP-14_W7.62mm_Socket"
 			(at 104.14 133.35 0)
 			(effects
@@
 			)
 		)
-		(property "Footprint" ""
+		(property "Footprint" "Package_DIP:DIP-14_W7.62mm_Socket"
 			(at 274.32 147.32 0)
 			(effects
@@
 			)
 		)
-		(property "Footprint" ""
+		(property "Footprint" "Package_DIP:DIP-14_W7.62mm_Socket"
 			(at 254 147.32 0)
 			(effects
@@
 			)
 		)
-		(property "Footprint" ""
+		(property "Footprint" "Package_DIP:DIP-14_W7.62mm_Socket"
 			(at 118.11 82.55 0)
 			(effects
@@
 			)
 		)
-		(property "Footprint" ""
+		(property "Footprint" "Package_DIP:DIP-14_W7.62mm_Socket"
 			(at 118.11 101.6 0)
 			(effects
@@
 			)
 		)
-		(property "Footprint" ""
+		(property "Footprint" "Package_DIP:DIP-16_W7.62mm_Socket"
 			(at 130.81 163.83 0)
 			(effects
@@
 			)
 		)
-		(property "Footprint" ""
+		(property "Footprint" "Package_DIP:DIP-14_W7.62mm_Socket"
 			(at 43.18 143.51 0)
 			(effects
@@
 			)
 		)
-		(property "Footprint" ""
+		(property "Footprint" "Package_DIP:DIP-16_W7.62mm_Socket"
 			(at 243.84 115.57 0)
 			(effects
@@
 			)
 		)
-		(property "Footprint" ""
+		(property "Footprint" "Package_DIP:DIP-14_W7.62mm_Socket"
 			(at 281.94 116.84 0)
 			(effects
@@
 			)
 		)
-		(property "Footprint" ""
+		(property "Footprint" "Package_DIP:DIP-14_W7.62mm_Socket"
 			(at 148.59 125.73 0)
 			(effects
@@
 			)
 		)
-		(property "Footprint" ""
+		(property "Footprint" "Package_DIP:DIP-16_W7.62mm_Socket"
 			(at 167.64 115.57 0)
 			(effects
@@
 			)
 		)
-		(property "Footprint" ""
+		(property "Footprint" "Package_DIP:DIP-14_W7.62mm_Socket"
 			(at 118.11 44.45 0)
 			(effects
@@
 			)
 		)
-		(property "Footprint" ""
+		(property "Footprint" "Package_DIP:DIP-16_W7.62mm_Socket"
 			(at 40.64 92.71 0)
 			(effects
@@
 			)
 		)
-		(property "Footprint" ""
+		(property "Footprint" "Package_DIP:DIP-14_W7.62mm_Socket"
 			(at 205.74 120.65 0)
 			(effects
@@
 			)
 		)
-		(property "Footprint" ""
+		(property "Footprint" "Package_DIP:DIP-16_W7.62mm_Socket"
 			(at 227.33 115.57 0)
 			(effects
@@
 			)
 		)
-		(property "Footprint" ""
+		(property "Footprint" "Package_DIP:DIP-16_W7.62mm_Socket"
 			(at 73.66 147.32 0)
 			(effects
@@
 			)
 		)
-		(property "Footprint" ""
+		(property "Footprint" "Package_DIP:DIP-14_W7.62mm_Socket"
 			(at 234.95 147.32 0)
 			(effects
@@
 			)
 		)
-		(property "Footprint" ""
+		(property "Footprint" "Package_DIP:DIP-14_W7.62mm_Socket"
 			(at 157.48 115.57 0)
 			(effects
@@
 			)
 		)
-		(property "Footprint" ""
+		(property "Footprint" "Package_DIP:DIP-16_W7.62mm_Socket"
 			(at 215.9 147.32 0)
 			(effects
@@
 			)
 		)
-		(property "Footprint" ""
+		(property "Footprint" "Package_DIP:DIP-14_W7.62mm_Socket"
 			(at 69.85 92.71 0)
 			(effects

Commit message: Adress Bus完成(芸術点Up)
Parts:
- IC19: footprint Package_DIP:DIP-16_W7.62mm_Socket -> Package_DIP:DIP-14_W7.62mm_Socket
Changed lines of the file:
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@@
 			)
 		)
-		(property "Footprint" "Package_DIP:DIP-16_W7.62mm_Socket"
+		(property "Footprint" "Package_DIP:DIP-14_W7.62mm_Socket"
 			(at 243.84 115.57 0)
 			(effects
@@
 			)
 		)
-		(property "Footprint" "Package_DIP:DIP-16_W7.62mm_Socket"
+		(property "Footprint" "Package_DIP:DIP-14_W7.62mm_Socket"
 			(at 167.64 115.57 0)
 			(effects
@@
 			)
 		)
-		(property "Footprint" "Package_DIP:DIP-16_W7.62mm_Socket"
+		(property "Footprint" "Package_DIP:DIP-14_W7.62mm_Socket"
 			(at 40.64 92.71 0)
 			(effects
@@
 			)
 		)
-		(property "Footprint" "Package_DIP:DIP-16_W7.62mm_Socket"
+		(property "Footprint" "Package_DIP:DIP-14_W7.62mm_Socket"
 			(at 227.33 115.57 0)
 			(effects
@@
 			)
 		)
-		(property "Footprint" "Package_DIP:DIP-16_W7.62mm_Socket"
+		(property "Footprint" "Package_DIP:DIP-14_W7.62mm_Socket"
 			(at 215.9 147.32 0)
 			(effects

Commit message: ICの配置を再検討
Parts:
- added CP17: 0.1u, Capacitor_THT:C_Disc_D3.0mm_W1.6mm_P2.50mm, symbol Device2:C_Bypass
- added unit 1 of IC20
- added unit 5 of IC20
- added unit 2 of IC20
- renumbered CP16 to CP18, CP17 to CP19, CP18 to CP20, CP19 to CP21, CP20 to CP22, CP21 to CP23, IC19 to IC18, IC20 to IC19, IC18 to IC20
Connections:
- net GND: now also CP17.2, IC20.7 (GND)
- net READ: now also IC20.1
- net VCC: now also CP17.1, IC20.14 (VCC)
- net ~{ALU_OE}: now also IC20.4
- new net CLK2: IC20.2, IC20.5
- new net ~{RAM_RD}: IC20.3
- new net ~{RAM_WR}: IC20.6
Other:
- moved on the sheet: CP18, CP19, CP20, CP21, CP22, CP23, IC10C, IC18E, IC19C, IC22G

Commit message: 基板ぬ
Parts:
- D10, D11, D12, D13, D14, D15, D16, D17, D18, D19, D2, D20, D21, D22, D23, D24, D25, D26, D27, D28, D29, D3, D30, D31, D32, D33, D34, D35, D36, D37, D38, D39, D4, D40, D41, D5, D6, D7, D8, D9: footprint Diode_THT:D_DO-35_SOD27_P2.54mm_Vertical_AnodeUp -> Library:DO-35_horizontal_anodeup_Smallhole
Connections:
- net ~{i6}: now reaches D11.2 (A), D19.2 (A), D27.2 (A), D3.2 (A), D35.2 (A), D39.2 (A), IC20.13, IC22.12
- net ~{i5}: now reaches D12.2 (A), D16.2 (A), D36.2 (A), D40.2 (A), IC18.9, IC22.4
- net ~{i4}: now reaches D13.2 (A), D17.2 (A), D25.2 (A), IC22.10
- net ~{i7}: now reaches IC18.4, IC22.2
