File: HC4_KiCad/programcounter.kicad_sch (KiCad schematic)
At the start: 20 parts, among them IC13 74HC161, IC14 74HC161, IC15 74HC161

Commit message: 再配置ほぼ完了
Connections:
- net at RN4.4 (R3.2): now also LD13.1 (K); no longer LD16.1 (K)
- net at RN4.5 (R4.2): now also LD10.1 (K); no longer LD19.1 (K)
- net at RN4.3 (R2.2): now also LD16.1 (K); no longer LD13.1 (K)
- net at RN4.2 (R1.2): now also LD19.1 (K); no longer LD10.1 (K)
Other:
- moved on the sheet: RN4A, RN4B, RN4C, RN4D
Changed lines of the file:
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@@
 	)
 	(junction
-		(at 115.57 119.38)
+		(at 157.48 170.18)
 		(diameter 0)
 		(color 0 0 0 0)
 	)
 	(junction
-		(at 157.48 170.18)
+		(at 115.57 119.38)
 		(diameter 0)
 		(color 0 0 0 0)
 	)
 	(junction
-		(at 157.48 125.73)
+		(at 148.59 170.18)
 		(diameter 0)
 		(color 0 0 0 0)
 	)
 	(junction
-		(at 148.59 170.18)
+		(at 157.48 125.73)
 		(diameter 0)
 		(color 0 0 0 0)
@@
 	(wire
 		(pts
-			(xy 148.59 170.18) (xy 157.48 170.18)
-		)
-		(stroke
-			(width 0)
-			(type default)
-		)
-	)
-	(wire
-		(pts
 			(xy 118.11 175.26) (xy 118.11 173.99)
 		)
@@
 	(wire
 		(pts
+			(xy 148.59 170.18) (xy 157.48 170.18)
+		)
+		(stroke
+			(width 0)
+			(type default)
+		)
+	)
+	(wire
+		(pts
 			(xy 104.14 57.15) (xy 116.84 57.15)
 		)
@@
 		)
 	)
+	(wire
+		(pts
+			(xy 157.48 170.18) (xy 166.37 170.18)
+		)
+		(stroke
+			(width 0)
+			(type default)
+		)
+	)
 	(bus
 		(pts
@@
 	(wire
 		(pts
-			(xy 157.48 170.18) (xy 166.37 170.18)
-		)
-		(stroke
-			(width 0)
-			(type default)
-		)
-	)
-	(wire
-		(pts
 			(xy 148.59 74.93) (xy 148.59 73.66)
 		)
@@
 	(label "Level_B2"
 		(at 104.14 97.79 0)
+		(fields_autoplaced yes)
 		(effects
 			(font
@@
 	(label "Level_A0"
 		(at 107.95 147.32 0)
+		(fields_autoplaced yes)
 		(effects
 			(font
@@
 	(label "PC_3"
 		(at 149.86 139.7 0)
+		(fields_autoplaced yes)
 		(effects
 			(font
@@
 	(label "Level_C3"
 		(at 104.14 52.07 0)
+		(fields_autoplaced yes)
 		(effects
 			(font
@@
 	(label "Level_B0"
 		(at 104.14 102.87 0)
+		(fields_autoplaced yes)
 		(effects
 			(font
@@
 	(label "PC_0"
 		(at 149.86 147.32 0)
+		(fields_autoplaced yes)
 		(effects
 			(font
@@
 	(label "Level_A2"
 		(at 107.95 142.24 0)
+		(fields_autoplaced yes)
 		(effects
 			(font
@@
 	(label "PC_6"
 		(at 149.86 97.79 0)
+		(fields_autoplaced yes)
 		(effects
 			(font
@@
 	(label "PC_5"
 		(at 149.86 100.33 0)
+		(fields_autoplaced yes)
 		(effects
 			(font
@@
 	(label "PC_9"
 		(at 149.86 57.15 0)
+		(fields_autoplaced yes)
 		(effects
 			(font
@@
 	(label "Level_A1"
 		(at 107.95 144.78 0)
+		(fields_autoplaced yes)
 		(effects
 			(font
@@
 	(label "PC_1"
 		(at 149.86 144.78 0)
+		(fields_autoplaced yes)
 		(effects
 			(font
@@
 	(label "Level_B3"
 		(at 104.14 95.25 0)
+		(fields_autoplaced yes)
 		(effects
 			(font
@@
 	(label "PC_11"
 		(at 149.86 52.07 0)
+		(fields_autoplaced yes)
 		(effects
 			(font
@@
 	(label "PC_4"
 		(at 149.86 102.87 0)
+		(fields_autoplaced yes)
 		(effects
 			(font
@@
 	(label "PC_7"
 		(at 149.86 95.25 0)
+		(fields_autoplaced yes)
 		(effects
 			(font
@@
 	(label "Level_C2"
 		(at 104.14 54.61 0)
+		(fields_autoplaced yes)
 		(effects
 			(font
@@
 	(label "Level_B1"
 		(at 104.14 100.33 0)
+		(fields_autoplaced yes)
 		(effects
 			(font
@@
 	(label "PC_10"
 		(at 149.86 54.61 0)
+		(fields_autoplaced yes)
 		(effects
 			(font
@@
 	(label "Level_A3"
 		(at 107.95 139.7 0)
+		(fields_autoplaced yes)
 		(effects
 			(font
@@
 	(label "Level_C0"
 		(at 104.14 59.69 0)
+		(fields_autoplaced yes)
 		(effects
 			(font
@@
 	(label "PC_8"
 		(at 149.86 59.69 0)
+		(fields_autoplaced yes)
 		(effects
 			(font
@@
 	(label "Level_C1"
 		(at 104.14 57.15 0)
+		(fields_autoplaced yes)
 		(effects
 			(font
@@
 	(label "PC_2"
 		(at 149.86 142.24 0)
+		(fields_autoplaced yes)
 		(effects
 			(font
@@
 		(shape input)
 		(at 114.3 83.82 180)
+		(fields_autoplaced yes)
 		(effects
 			(font
@@
 		(shape input)
 		(at 102.87 134.62 180)
+		(fields_autoplaced yes)
 		(effects
 			(font
@@
 		(shape output)
 		(at 182.88 52.07 0)
+		(fields_autoplaced yes)
 		(effects
 			(font
@@
 		(shape input)
 		(at 99.06 90.17 180)
+		(fields_autoplaced yes)
 		(effects
 			(font
@@
 		(shape input)
 		(at 114.3 40.64 180)
+		(fields_autoplaced yes)
 		(effects
 			(font
@@
 		(shape input)
 		(at 99.06 46.99 180)
+		(fields_autoplaced yes)
 		(effects
 			(font
@@
 		(shape input)
 		(at 114.3 128.27 180)
+		(fields_autoplaced yes)
 		(effects
 			(font
@@
 	(symbol
 		(lib_id "Device:R_Network08_Split")
-		(at 157.48 166.37 0)
-		(mirror x)
+		(at 148.59 166.37 180)
 		(unit 3)
 		(exclude_from_sim no)
@@
 		(on_board yes)
 		(dnp no)
-		(fields_autoplaced yes)
 		(property "Reference" "RN4"
-			(at 154.94 165.0999 0)
+			(at 151.13 165.0999 0)
 			(effects
 				(font
 					(size 1.27 1.27)
 				)
-				(justify right)
+				(justify left)
 			)
 		)
 		(property "Value" "1k"
-			(at 154.94 167.6399 0)
+			(at 151.13 167.6399 0)
 			(effects
 				(font
@@
 		)
 		(property "Footprint" "Resistor_THT:R_Array_SIP9"
-			(at 155.448 166.37 90)
+			(at 150.622 166.37 90)
 			(effects
 				(font
@@
 		)
 		(property "Datasheet" "http://www.vishay.com/docs/31509/csc.pdf"
-			(at 157.48 166.37 0)
+			(at 148.59 166.37 0)
 			(effects
 				(font
@@
 		)
 		(property "Description" "8 resistor network, star topology, bussed resistors, split"
-			(at 157.48 166.37 0)
+			(at 148.59 166.37 0)
 			(effects
 				(font
@@
 	(symbol
 		(lib_id "Device:R_Network08_Split")
-		(at 166.37 166.37 0)
-		(mirror x)
+		(at 139.7 166.37 180)
 		(unit 4)
 		(exclude_from_sim no)
@@
 		(fields_autoplaced yes)
 		(property "Reference" "RN4"
-			(at 163.83 165.0999 0)
+			(at 142.24 165.0999 0)
 			(effects
 				(font
@@
 		)
 		(property "Value" "1k"
-			(at 163.83 167.6399 0)
+			(at 142.24 167.6399 0)
 			(effects
 				(font
@@
 		)
 		(property "Footprint" "Resistor_THT:R_Array_SIP9"
-			(at 164.338 166.37 90)
+			(at 141.732 166.37 90)
 			(effects
 				(font
@@
 		)
 		(property "Datasheet" "http://www.vishay.com/docs/31509/csc.pdf"
-			(at 166.37 166.37 0)
+			(at 139.7 166.37 0)
 			(effects
 				(font
@@
 		)
 		(property "Description" "8 resistor network, star topology, bussed resistors, split"
-			(at 166.37 166.37 0)
+			(at 139.7 166.37 0)
 			(effects
 				(font
@@
 	(symbol
 		(lib_id "Device:R_Network08_Split")
-		(at 148.59 166.37 0)
-		(mirror x)
+		(at 157.48 166.37 180)
 		(unit 2)
 		(exclude_from_sim no)
@@
 		(fields_autoplaced yes)
 		(property "Reference" "RN4"
-			(at 146.05 165.0999 0)
+			(at 160.02 165.0999 0)
 			(effects
 				(font
@@
 		)
 		(property "Value" "1k"
-			(at 146.05 167.6399 0)
+			(at 160.02 167.6399 0)
 			(effects
 				(font
@@
 		)
 		(property "Footprint" "Resistor_THT:R_Array_SIP9"
-			(at 146.558 166.37 90)
+			(at 159.512 166.37 90)
 			(effects
 				(font
@@
 		)
 		(property "Datasheet" "http://www.vishay.com/docs/31509/csc.pdf"
-			(at 148.59 166.37 0)
+			(at 157.48 166.37 0)
 			(effects
 				(font
@@
 		)
 		(property "Description" "8 resistor network, star topology, bussed resistors, split"
-			(at 148.59 166.37 0)
+			(at 157.48 166.37 0)
 			(effects
 				(font
@@
 	(symbol
 		(lib_id "Device:R_Network08_Split")
-		(at 139.7 166.37 0)
-		(mirror x)
+		(at 166.37 166.37 180)
 		(unit 1)
 		(exclude_from_sim no)
@@
 		(fields_autoplaced yes)
 		(property "Reference" "RN4"
-			(at 137.16 165.0999 0)
+			(at 168.91 165.0999 0)
 			(effects
 				(font
@@
 		)
 		(property "Value" "1k"
-			(at 137.16 167.6399 0)
+			(at 168.91 167.6399 0)
 			(effects
 				(font
@@
 		)
 		(property "Footprint" "Resistor_THT:R_Array_SIP9"
-			(at 137.668 166.37 90)
+			(at 168.402 166.37 90)
 			(effects
 				(font
@@
 		)
 		(property "Datasheet" "http://www.vishay.com/docs/31509/csc.pdf"
-			(at 139.7 166.37 0)
+			(at 166.37 166.37 0)
 			(effects
 				(font
@@
 		)
 		(property "Description" "8 resistor network, star topology, bussed resistors, split"
-			(at 139.7 166.37 0)
+			(at 166.37 166.37 0)
 			(effects
 				(font

Commit message: またも手直し
Parts:
- renumbered LD8 to LD20, LD9 to LD21, LD10 to LD22, LD11 to LD23, LD12 to LD24, LD13 to LD25, LD14 to LD26, LD15 to LD27, LD16 to LD28, LD17 to LD29, LD18 to LD30, LD19 to LD31, RN3 to RN5, RN4 to RN6
Other:
- title: CPU -> HC4_CPU

Commit message: 回路の改良　試験は明日やる
Parts:
- removed RN5: 1k, Resistor_THT:R_Array_SIP5, symbol Device:R_Network04_Split
- removed RN6: 1k, Resistor_THT:R_Array_SIP9, symbol Device:R_Network08_Split
- added RN4, RN5: 1k, Resistor_THT:R_Array_SIP9, symbol Device:R_Network08_Split
Connections:
- net GND: now also RN4.1 (R1), RN4.1 (R1), RN4.1 (R1), RN4.1 (R1), RN5.1 (R1), RN5.1 (R1), RN5.1 (R1), RN5.1 (R1), RN5.1 (R1), RN5.1 (R1), RN5.1 (R1), RN5.1 (R1)
- net Level_A0: now also IC15.3 (A); no longer IC15.6 (D)
- net Level_A1: now also IC15.4 (B); no longer IC15.5 (C)
- net Level_A2: now also IC15.5 (C); no longer IC15.4 (B)
- net Level_A3: now also IC15.6 (D); no longer IC15.3 (A)
- net Level_B0: now also IC14.3 (A); no longer IC14.6 (D)
- net Level_B1: now also IC14.4 (B); no longer IC14.5 (C)
- net Level_B2: now also IC14.5 (C); no longer IC14.4 (B)
- net Level_B3: now also IC14.6 (D); no longer IC14.3 (A)
- net Level_C0: now also IC13.3 (A); no longer IC13.6 (D)
- net Level_C1: now also IC13.4 (B); no longer IC13.5 (C)
- net Level_C2: now also IC13.5 (C); no longer IC13.4 (B)
- net Level_C3: now also IC13.6 (D); no longer IC13.3 (A)
- net PC_0: now also IC15.14 (QA), LD22.2; no longer IC15.11 (QD), LD31.2
- net PC_1: now also IC15.13 (QB), LD25.2; no longer IC15.12 (QC), LD28.2
- net PC_10: now also IC13.12 (QC), LD26.2; no longer IC13.13 (QB), LD23.2
- net PC_11: now also IC13.11 (QD), LD29.2; no longer IC13.14 (QA), LD20.2
- net PC_2: now also IC15.12 (QC), LD28.2; no longer IC15.13 (QB), LD25.2
- net PC_3: now also IC15.11 (QD), LD31.2; no longer IC15.14 (QA), LD22.2
- net PC_4: now also IC14.14 (QA), LD21.2; no longer IC14.11 (QD), LD30.2
- net PC_5: now also IC14.13 (QB), LD24.2; no longer IC14.12 (QC), LD27.2
- net PC_6: now also IC14.12 (QC), LD27.2; no longer IC14.13 (QB), LD24.2
- net PC_7: now also IC14.11 (QD), LD30.2; no longer IC14.14 (QA), LD21.2
- net PC_8: now also IC13.14 (QA), LD20.2; no longer IC13.11 (QD), LD29.2
- net PC_9: now also IC13.13 (QB), LD23.2; no longer IC13.12 (QC), LD26.2
- net at LD26.1 (K): now also RN4.8 (R7.2)
- net at LD30.1 (K): now also RN5.5 (R4.2)
- net at LD29.1 (K): now also RN4.9 (R8.2)
- net at LD24.1 (K): now also RN5.3 (R2.2)
- net at LD23.1 (K): now also RN4.7 (R6.2)
- net at LD20.1 (K): now also RN4.6 (R5.2)
- net at LD27.1 (K): now also RN5.4 (R3.2)
- net at LD25.1 (K): now also RN5.7 (R6.2)
- net at LD21.1 (K): now also RN5.2 (R1.2)
- net at LD22.1 (K): now also RN5.6 (R5.2)
- net at LD28.1 (K): now also RN5.8 (R7.2)
- net at LD31.1 (K): now also RN5.9 (R8.2)
