File: HC4_KiCad/addressbus.kicad_sch (KiCad schematic)
At the start: 15 parts, among them IC16 74HC257, IC17 74HC257, SW2 Bus_Open

Commit message: 回路の改良　試験は明日やる
Parts:
- renumbered RN7 to RN6
Changed lines of the file:
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@@
 	(title_block
 		(title "HC4_CPU")
-		(date "2025-02-23")
-		(rev "1.2")
+		(date "2025-03-31")
+		(rev "1.3")
 	)
 	(junction
@@
 		(dnp no)
 		(fields_autoplaced yes)
-		(property "Reference" "RN7"
+		(property "Reference" "RN6"
 			(at 208.28 154.9401 0)
 			(effects
@@
 			(project ""
 				(path "/33731ded-38c0-4297-bdd8-92b082f46ff8/06be0d13-f4ff-478c-92b4-64c4ff1b6880"
-					(reference "RN7")
+					(reference "RN6")
 					(unit 7)
 				)
@@
 		(dnp no)
 		(fields_autoplaced yes)
-		(property "Reference" "RN7"
+		(property "Reference" "RN6"
 			(at 153.67 154.9401 0)
 			(effects
@@
 			(project ""
 				(path "/33731ded-38c0-4297-bdd8-92b082f46ff8/06be0d13-f4ff-478c-92b4-64c4ff1b6880"
-					(reference "RN7")
+					(reference "RN6")
 					(unit 1)
 				)
@@
 		(dnp no)
 		(fields_autoplaced yes)
-		(property "Reference" "RN7"
+		(property "Reference" "RN6"
 			(at 190.5 154.9401 0)
 			(effects
@@
 			(project ""
 				(path "/33731ded-38c0-4297-bdd8-92b082f46ff8/06be0d13-f4ff-478c-92b4-64c4ff1b6880"
-					(reference "RN7")
+					(reference "RN6")
 					(unit 5)
 				)
@@
 		(dnp no)
 		(fields_autoplaced yes)
-		(property "Reference" "RN7"
+		(property "Reference" "RN6"
 			(at 162.56 154.9401 0)
 			(effects
@@
 			(project ""
 				(path "/33731ded-38c0-4297-bdd8-92b082f46ff8/06be0d13-f4ff-478c-92b4-64c4ff1b6880"
-					(reference "RN7")
+					(reference "RN6")
 					(unit 2)
 				)
@@
 		(dnp no)
 		(fields_autoplaced yes)
-		(property "Reference" "RN7"
+		(property "Reference" "RN6"
 			(at 217.17 154.9401 0)
 			(effects
@@
 			(project ""
 				(path "/33731ded-38c0-4297-bdd8-92b082f46ff8/06be0d13-f4ff-478c-92b4-64c4ff1b6880"
-					(reference "RN7")
+					(reference "RN6")
 					(unit 8)
 				)
@@
 		(dnp no)
 		(fields_autoplaced yes)
-		(property "Reference" "RN7"
+		(property "Reference" "RN6"
 			(at 171.45 154.9401 0)
 			(effects
@@
 			(project ""
 				(path "/33731ded-38c0-4297-bdd8-92b082f46ff8/06be0d13-f4ff-478c-92b4-64c4ff1b6880"
-					(reference "RN7")
+					(reference "RN6")
 					(unit 3)
 				)
@@
 		(dnp no)
 		(fields_autoplaced yes)
-		(property "Reference" "RN7"
+		(property "Reference" "RN6"
 			(at 199.39 154.9401 0)
 			(effects
@@
 			(project ""
 				(path "/33731ded-38c0-4297-bdd8-92b082f46ff8/06be0d13-f4ff-478c-92b4-64c4ff1b6880"
-					(reference "RN7")
+					(reference "RN6")
 					(unit 6)
 				)
@@
 		(dnp no)
 		(fields_autoplaced yes)
-		(property "Reference" "RN7"
+		(property "Reference" "RN6"
 			(at 180.34 154.9401 0)
 			(effects
@@
 			(project ""
 				(path "/33731ded-38c0-4297-bdd8-92b082f46ff8/06be0d13-f4ff-478c-92b4-64c4ff1b6880"
-					(reference "RN7")
+					(reference "RN6")
 					(unit 4)
 				)

Commit message: フットプリントをSOPに変更
Parts:
- CP15, CP16: footprint Capacitor_THT:C_Disc_D3.0mm_W1.6mm_P2.50mm -> Capacitor_SMD:C_0603_1608Metric
- IC16, IC17: footprint Package_DIP:DIP-16_W7.62mm_Socket -> Package_SO:SO-16_5.3x10.2mm_P1.27mm
- R4: footprint Resistor_THT:R_Axial_DIN0207_L6.3mm_D2.5mm_P7.62mm_Horizontal -> Resistor_SMD:R_0603_1608Metric
Changed lines of the file:
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@@
 			)
 		)
-		(property "Footprint" "Package_DIP:DIP-16_W7.62mm_Socket"
+		(property "Footprint" "Package_SO:SO-16_5.3x10.2mm_P1.27mm"
 			(at 121.92 80.01 0)
 			(effects
@@
 			)
 		)
-		(property "Footprint" "Capacitor_THT:C_Disc_D3.0mm_W1.6mm_P2.50mm"
+		(property "Footprint" "Capacitor_SMD:C_0603_1608Metric"
 			(at 150.8252 185.42 0)
 			(effects
@@
 			)
 		)
-		(property "Footprint" "Resistor_THT:R_Axial_DIN0207_L6.3mm_D2.5mm_P7.62mm_Horizontal"
+		(property "Footprint" "Resistor_SMD:R_0603_1608Metric"
 			(at 88.392 182.88 90)
 			(effects
@@
 			)
 		)
-		(property "Footprint" "Capacitor_THT:C_Disc_D3.0mm_W1.6mm_P2.50mm"
+		(property "Footprint" "Capacitor_SMD:C_0603_1608Metric"
 			(at 140.6652 185.42 0)
 			(effects
@@
 			)
 		)
-		(property "Footprint" "Package_DIP:DIP-16_W7.62mm_Socket"
+		(property "Footprint" "Package_SO:SO-16_5.3x10.2mm_P1.27mm"
 			(at 121.92 146.05 0)
 			(effects
