File: HC4_KiCad/addressbus.kicad_sch (KiCad schematic)
At the start: 15 parts, among them IC16 74HC257, IC17 74HC257, SW2 Bus_Open

Commit message: Added output port for blink
Parts:
- renumbered LD32 to LD36, LD33 to LD37, LD34 to LD38, LD35 to LD39, LD36 to LD40, LD37 to LD41, LD38 to LD42, LD39 to LD43, SW2 to SW1
Changed lines of the file:
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@@
 		(on_board yes)
 		(dnp no)
-		(property "Reference" "#PWR061"
+		(property "Reference" "#PWR060"
 			(at 144.78 194.31 0)
 			(effects
@@
 			(project ""
 				(path "/33731ded-38c0-4297-bdd8-92b082f46ff8/06be0d13-f4ff-478c-92b4-64c4ff1b6880"
-					(reference "#PWR061")
+					(reference "#PWR060")
 					(unit 1)
 				)
@@
 		(dnp no)
 		(fields_autoplaced yes)
-		(property "Reference" "LD32"
+		(property "Reference" "LD36"
 			(at 154.94 145.0974 90)
 			(effects
@@
 			)
 		)
-		(property "Datasheet" "~"
+		(property "Datasheet" ""
 			(at 151.13 144.78 0)
 			(effects
@@
 			(project "HC4_KiCad"
 				(path "/33731ded-38c0-4297-bdd8-92b082f46ff8/06be0d13-f4ff-478c-92b4-64c4ff1b6880"
-					(reference "LD32")
+					(reference "LD36")
 					(unit 1)
 				)
@@
 		(dnp no)
 		(fields_autoplaced yes)
-		(property "Reference" "LD35"
+		(property "Reference" "LD39"
 			(at 181.61 145.0974 90)
 			(effects
@@
 			)
 		)
-		(property "Datasheet" "~"
+		(property "Datasheet" ""
 			(at 177.8 144.78 0)
 			(effects
@@
 			(project "HC4_KiCad"
 				(path "/33731ded-38c0-4297-bdd8-92b082f46ff8/06be0d13-f4ff-478c-92b4-64c4ff1b6880"
-					(reference "LD35")
+					(reference "LD39")
 					(unit 1)
 				)
@@
 		(dnp no)
 		(fields_autoplaced yes)
-		(property "Reference" "#PWR056"
+		(property "Reference" "#PWR055"
 			(at 121.92 59.69 0)
 			(effects
@@
 			(project ""
 				(path "/33731ded-38c0-4297-bdd8-92b082f46ff8/06be0d13-f4ff-478c-92b4-64c4ff1b6880"
-					(reference "#PWR056")
+					(reference "#PWR055")
 					(unit 1)
 				)
@@
 		(dnp no)
 		(fields_autoplaced yes)
-		(property "Reference" "LD39"
+		(property "Reference" "LD43"
 			(at 218.44 145.0974 90)
 			(effects
@@
 			)
 		)
-		(property "Datasheet" "~"
+		(property "Datasheet" ""
 			(at 214.63 144.78 0)
 			(effects
@@
 			(project "HC4_KiCad"
 				(path "/33731ded-38c0-4297-bdd8-92b082f46ff8/06be0d13-f4ff-478c-92b4-64c4ff1b6880"
-					(reference "LD39")
+					(reference "LD43")
 					(unit 1)
 				)
@@
 		(dnp no)
 		(fields_autoplaced yes)
-		(property "Reference" "#PWR057"
+		(property "Reference" "#PWR056"
 			(at 121.92 114.3 0)
 			(effects
@@
 			(project ""
 				(path "/33731ded-38c0-4297-bdd8-92b082f46ff8/06be0d13-f4ff-478c-92b4-64c4ff1b6880"
-					(reference "#PWR057")
+					(reference "#PWR056")
 					(unit 1)
 				)
@@
 		(on_board yes)
 		(dnp no)
-		(property "Reference" "SW2"
+		(property "Reference" "SW1"
 			(at 78.74 166.37 0)
 			(effects
@@
 			(project ""
 				(path "/33731ded-38c0-4297-bdd8-92b082f46ff8/06be0d13-f4ff-478c-92b4-64c4ff1b6880"
-					(reference "SW2")
+					(reference "SW1")
 					(unit 1)
 				)
@@
 		(dnp no)
 		(fields_autoplaced yes)
-		(property "Reference" "LD38"
+		(property "Reference" "LD42"
 			(at 209.55 145.0974 90)
 			(effects
@@
 			)
 		)
-		(property "Datasheet" "~"
+		(property "Datasheet" ""
 			(at 205.74 144.78 0)
 			(effects
@@
 			(project "HC4_KiCad"
 				(path "/33731ded-38c0-4297-bdd8-92b082f46ff8/06be0d13-f4ff-478c-92b4-64c4ff1b6880"
-					(reference "LD38")
+					(reference "LD42")
 					(unit 1)
 				)
@@
 		(dnp no)
 		(fields_autoplaced yes)
-		(property "Reference" "LD34"
+		(property "Reference" "LD38"
 			(at 172.72 145.0974 90)
 			(effects
@@
 			)
 		)
-		(property "Datasheet" "~"
+		(property "Datasheet" ""
 			(at 168.91 144.78 0)
 			(effects
@@
 			(project "HC4_KiCad"
 				(path "/33731ded-38c0-4297-bdd8-92b082f46ff8/06be0d13-f4ff-478c-92b4-64c4ff1b6880"
-					(reference "LD34")
+					(reference "LD38")
 					(unit 1)
 				)
@@
 		(on_board yes)
 		(dnp no)
-		(property "Reference" "#PWR060"
+		(property "Reference" "#PWR059"
 			(at 144.78 172.72 0)
 			(effects
@@
 			(project ""
 				(path "/33731ded-38c0-4297-bdd8-92b082f46ff8/06be0d13-f4ff-478c-92b4-64c4ff1b6880"
-					(reference "#PWR060")
+					(reference "#PWR059")
 					(unit 1)
 				)
@@
 		(dnp no)
 		(fields_autoplaced yes)
-		(property "Reference" "LD33"
+		(property "Reference" "LD37"
 			(at 163.83 145.0974 90)
 			(effects
@@
 			)
 		)
-		(property "Datasheet" "~"
+		(property "Datasheet" ""
 			(at 160.02 144.78 0)
 			(effects
@@
 			(project "HC4_KiCad"
 				(path "/33731ded-38c0-4297-bdd8-92b082f46ff8/06be0d13-f4ff-478c-92b4-64c4ff1b6880"
-					(reference "LD33")
+					(reference "LD37")
 					(unit 1)
 				)
@@
 		(dnp no)
 		(fields_autoplaced yes)
-		(property "Reference" "#PWR062"
+		(property "Reference" "#PWR061"
 			(at 168.91 166.37 0)
 			(effects
@@
 			(project ""
 				(path "/33731ded-38c0-4297-bdd8-92b082f46ff8/06be0d13-f4ff-478c-92b4-64c4ff1b6880"
-					(reference "#PWR062")
+					(reference "#PWR061")
 					(unit 1)
 				)
@@
 		(dnp no)
 		(fields_autoplaced yes)
-		(property "Reference" "#PWR055"
+		(property "Reference" "#PWR054"
 			(at 90.17 196.85 0)
 			(effects
@@
 			(project ""
 				(path "/33731ded-38c0-4297-bdd8-92b082f46ff8/06be0d13-f4ff-478c-92b4-64c4ff1b6880"
-					(reference "#PWR055")
+					(reference "#PWR054")
 					(unit 1)
 				)
@@
 		(dnp no)
 		(fields_autoplaced yes)
-		(property "Reference" "LD37"
+		(property "Reference" "LD41"
 			(at 200.66 145.0974 90)
 			(effects
@@
 			)
 		)
-		(property "Datasheet" "~"
+		(property "Datasheet" ""
 			(at 196.85 144.78 0)
 			(effects
@@
 			(project "HC4_KiCad"
 				(path "/33731ded-38c0-4297-bdd8-92b082f46ff8/06be0d13-f4ff-478c-92b4-64c4ff1b6880"
-					(reference "LD37")
+					(reference "LD41")
 					(unit 1)
 				)
@@
 		(dnp no)
 		(fields_autoplaced yes)
-		(property "Reference" "#PWR058"
+		(property "Reference" "#PWR057"
 			(at 121.92 125.73 0)
 			(effects
@@
 			(project ""
 				(path "/33731ded-38c0-4297-bdd8-92b082f46ff8/06be0d13-f4ff-478c-92b4-64c4ff1b6880"
-					(reference "#PWR058")
+					(reference "#PWR057")
 					(unit 1)
 				)
@@
 		(dnp no)
 		(fields_autoplaced yes)
-		(property "Reference" "LD36"
+		(property "Reference" "LD40"
 			(at 191.77 145.0974 90)
 			(effects
@@
 			)
 		)
-		(property "Datasheet" "~"
+		(property "Datasheet" ""
 			(at 187.96 144.78 0)
 			(effects
@@
 			(project "HC4_KiCad"
 				(path "/33731ded-38c0-4297-bdd8-92b082f46ff8/06be0d13-f4ff-478c-92b4-64c4ff1b6880"
-					(reference "LD36")
+					(reference "LD40")
 					(unit 1)
 				)
@@
 		(dnp no)
 		(fields_autoplaced yes)
-		(property "Reference" "#PWR059"
+		(property "Reference" "#PWR058"
 			(at 121.92 179.07 0)
 			(effects
@@
 			(project ""
 				(path "/33731ded-38c0-4297-bdd8-92b082f46ff8/06be0d13-f4ff-478c-92b4-64c4ff1b6880"
-					(reference "#PWR059")
+					(reference "#PWR058")
 					(unit 1)
 				)
@@
 		(dnp no)
 		(fields_autoplaced yes)
-		(property "Reference" "#PWR054"
+		(property "Reference" "#PWR053"
 			(at 71.12 175.26 0)
 			(effects
@@
 			(project ""
 				(path "/33731ded-38c0-4297-bdd8-92b082f46ff8/06be0d13-f4ff-478c-92b4-64c4ff1b6880"
-					(reference "#PWR054")
-					(unit 1)
-				)
+					(reference "#PWR053")
+					(unit 1)
+				)

Commit message: moti
Parts:
- IC15: renamed from IC16; footprint Package_SO:SO-16_5.3x10.2mm_P1.27mm -> Package_DIP:DIP-16_W7.62mm
- IC16: renamed from IC17; footprint Package_SO:SO-16_5.3x10.2mm_P1.27mm -> Package_DIP:DIP-16_W7.62mm
- renumbered CP15 to CP14, CP16 to CP15
Changed lines of the file:
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@@
 		(on_board yes)
 		(dnp no)
-		(property "Reference" "#PWR060"
+		(property "Reference" "#PWR061"
 			(at 144.78 194.31 0)
 			(effects
@@
 			(project ""
 				(path "/33731ded-38c0-4297-bdd8-92b082f46ff8/06be0d13-f4ff-478c-92b4-64c4ff1b6880"
-					(reference "#PWR060")
+					(reference "#PWR061")
 					(unit 1)
 				)
@@
 		(dnp no)
 		(fields_autoplaced yes)
-		(property "Reference" "IC16"
+		(property "Reference" "IC15"
 			(at 124.1141 57.15 0)
 			(effects
@@
 			)
 		)
-		(property "Footprint" "Package_SO:SO-16_5.3x10.2mm_P1.27mm"
+		(property "Footprint" "Package_DIP:DIP-16_W7.62mm"
 			(at 121.92 80.01 0)
 			(effects
@@
 			(project ""
 				(path "/33731ded-38c0-4297-bdd8-92b082f46ff8/06be0d13-f4ff-478c-92b4-64c4ff1b6880"
-					(reference "IC16")
+					(reference "IC15")
 					(unit 1)
 				)
@@
 		(on_board yes)
 		(dnp no)
-		(property "Reference" "CP16"
+		(property "Reference" "CP15"
 			(at 154.432 180.594 0)
 			(effects
@@
 			(project "HC4_KiCad"
 				(path "/33731ded-38c0-4297-bdd8-92b082f46ff8/06be0d13-f4ff-478c-92b4-64c4ff1b6880"
-					(reference "CP16")
+					(reference "CP15")
 					(unit 1)
 				)
@@
 		(dnp no)
 		(fields_autoplaced yes)
-		(property "Reference" "#PWR055"
+		(property "Reference" "#PWR056"
 			(at 121.92 59.69 0)
 			(effects
@@
 			(project ""
 				(path "/33731ded-38c0-4297-bdd8-92b082f46ff8/06be0d13-f4ff-478c-92b4-64c4ff1b6880"
-					(reference "#PWR055")
+					(reference "#PWR056")
 					(unit 1)
 				)
@@
 		(dnp no)
 		(fields_autoplaced yes)
-		(property "Reference" "#PWR056"
+		(property "Reference" "#PWR057"
 			(at 121.92 114.3 0)
 			(effects
@@
 			(project ""
 				(path "/33731ded-38c0-4297-bdd8-92b082f46ff8/06be0d13-f4ff-478c-92b4-64c4ff1b6880"
-					(reference "#PWR056")
+					(reference "#PWR057")
 					(unit 1)
 				)
@@
 		(on_board yes)
 		(dnp no)
-		(property "Reference" "CP15"
+		(property "Reference" "CP14"
 			(at 131.318 179.578 0)
 			(effects
@@
 			(project "HC4_KiCad"
 				(path "/33731ded-38c0-4297-bdd8-92b082f46ff8/06be0d13-f4ff-478c-92b4-64c4ff1b6880"
-					(reference "CP15")
+					(reference "CP14")
 					(unit 1)
 				)
@@
 		(on_board yes)
 		(dnp no)
-		(property "Reference" "#PWR059"
+		(property "Reference" "#PWR060"
 			(at 144.78 172.72 0)
 			(effects
@@
 			(project ""
 				(path "/33731ded-38c0-4297-bdd8-92b082f46ff8/06be0d13-f4ff-478c-92b4-64c4ff1b6880"
-					(reference "#PWR059")
+					(reference "#PWR060")
 					(unit 1)
 				)
@@
 		(dnp no)
 		(fields_autoplaced yes)
-		(property "Reference" "#PWR061"
+		(property "Reference" "#PWR062"
 			(at 168.91 166.37 0)
 			(effects
@@
 			(project ""
 				(path "/33731ded-38c0-4297-bdd8-92b082f46ff8/06be0d13-f4ff-478c-92b4-64c4ff1b6880"
-					(reference "#PWR061")
+					(reference "#PWR062")
 					(unit 1)
 				)
@@
 		(dnp no)
 		(fields_autoplaced yes)
-		(property "Reference" "IC17"
+		(property "Reference" "IC16"
 			(at 124.1141 123.19 0)
 			(effects
@@
 			)
 		)
-		(property "Footprint" "Package_SO:SO-16_5.3x10.2mm_P1.27mm"
+		(property "Footprint" "Package_DIP:DIP-16_W7.62mm"
 			(at 121.92 146.05 0)
 			(effects
@@
 			(project "HC4_KiCad"
 				(path "/33731ded-38c0-4297-bdd8-92b082f46ff8/06be0d13-f4ff-478c-92b4-64c4ff1b6880"
-					(reference "IC17")
+					(reference "IC16")
 					(unit 1)
 				)
@@
 		(dnp no)
 		(fields_autoplaced yes)
-		(property "Reference" "#PWR054"
+		(property "Reference" "#PWR055"
 			(at 90.17 196.85 0)
 			(effects
@@
 			(project ""
 				(path "/33731ded-38c0-4297-bdd8-92b082f46ff8/06be0d13-f4ff-478c-92b4-64c4ff1b6880"
-					(reference "#PWR054")
+					(reference "#PWR055")
 					(unit 1)
 				)
@@
 		(dnp no)
 		(fields_autoplaced yes)
-		(property "Reference" "#PWR057"
+		(property "Reference" "#PWR058"
 			(at 121.92 125.73 0)
 			(effects
@@
 			(project ""
 				(path "/33731ded-38c0-4297-bdd8-92b082f46ff8/06be0d13-f4ff-478c-92b4-64c4ff1b6880"
-					(reference "#PWR057")
+					(reference "#PWR058")
 					(unit 1)
 				)
@@
 		(dnp no)
 		(fields_autoplaced yes)
-		(property "Reference" "#PWR058"
+		(property "Reference" "#PWR059"
 			(at 121.92 179.07 0)
 			(effects
@@
 			(project ""
 				(path "/33731ded-38c0-4297-bdd8-92b082f46ff8/06be0d13-f4ff-478c-92b4-64c4ff1b6880"
-					(reference "#PWR058")
+					(reference "#PWR059")
 					(unit 1)
 				)
@@
 		(dnp no)
 		(fields_autoplaced yes)
-		(property "Reference" "#PWR053"
+		(property "Reference" "#PWR054"
 			(at 71.12 175.26 0)
 			(effects
@@
 			(project ""
 				(path "/33731ded-38c0-4297-bdd8-92b082f46ff8/06be0d13-f4ff-478c-92b4-64c4ff1b6880"
-					(reference "#PWR053")
-					(unit 1)
-				)
+					(reference "#PWR054")
+					(unit 1)
+				)

Commit message: 基板途中
Parts:
- renumbered CP14 to CP13, CP15 to CP14

Commit message: 仮
Parts:
- renumbered IC15 to IC14, IC16 to IC15, LD36 to LD32, LD37 to LD33, LD38 to LD34, LD39 to LD35, LD40 to LD36, LD41 to LD37, LD42 to LD38, LD43 to LD39
Changed lines of the file:
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@@
 		(in_pos_files yes)
 		(dnp no)
-		(property "Reference" "#PWR058"
+		(property "Reference" "#PWR055"
 			(at 144.78 194.31 0)
 			(hide yes)
@@
 			(project "HC4_KiCad"
 				(path "/33731ded-38c0-4297-bdd8-92b082f46ff8/06be0d13-f4ff-478c-92b4-64c4ff1b6880"
-					(reference "#PWR058")
+					(reference "#PWR055")
 					(unit 1)
 				)
@@
 		(dnp no)
 		(fields_autoplaced yes)
-		(property "Reference" "IC15"
+		(property "Reference" "IC14"
 			(at 124.1141 57.15 0)
 			(show_name no)
@@
 			(project "HC4_KiCad"
 				(path "/33731ded-38c0-4297-bdd8-92b082f46ff8/06be0d13-f4ff-478c-92b4-64c4ff1b6880"
-					(reference "IC15")
+					(reference "IC14")
 					(unit 1)
 				)
@@
 		(dnp no)
 		(fields_autoplaced yes)
-		(property "Reference" "LD36"
+		(property "Reference" "LD32"
 			(at 154.94 145.0974 90)
 			(show_name no)
@@
 			(project "HC4_KiCad"
 				(path "/33731ded-38c0-4297-bdd8-92b082f46ff8/06be0d13-f4ff-478c-92b4-64c4ff1b6880"
-					(reference "LD36")
+					(reference "LD32")
 					(unit 1)
 				)
@@
 		(dnp no)
 		(fields_autoplaced yes)
-		(property "Reference" "LD39"
+		(property "Reference" "LD35"
 			(at 181.61 145.0974 90)
 			(show_name no)
@@
 			(project "HC4_KiCad"
 				(path "/33731ded-38c0-4297-bdd8-92b082f46ff8/06be0d13-f4ff-478c-92b4-64c4ff1b6880"
-					(reference "LD39")
+					(reference "LD35")
 					(unit 1)
 				)
@@
 		(dnp no)
 		(fields_autoplaced yes)
-		(property "Reference" "#PWR053"
+		(property "Reference" "#PWR050"
 			(at 121.92 59.69 0)
 			(hide yes)
@@
 			(project "HC4_KiCad"
 				(path "/33731ded-38c0-4297-bdd8-92b082f46ff8/06be0d13-f4ff-478c-92b4-64c4ff1b6880"
-					(reference "#PWR053")
+					(reference "#PWR050")
 					(unit 1)
 				)
@@
 		(dnp no)
 		(fields_autoplaced yes)
-		(property "Reference" "LD43"
+		(property "Reference" "LD39"
 			(at 218.44 145.0974 90)
 			(show_name no)
@@
 			(project "HC4_KiCad"
 				(path "/33731ded-38c0-4297-bdd8-92b082f46ff8/06be0d13-f4ff-478c-92b4-64c4ff1b6880"
-					(reference "LD43")
+					(reference "LD39")
 					(unit 1)
 				)
@@
 		(dnp no)
 		(fields_autoplaced yes)
-		(property "Reference" "#PWR054"
+		(property "Reference" "#PWR051"
 			(at 121.92 114.3 0)
 			(hide yes)
@@
 			(project "HC4_KiCad"
 				(path "/33731ded-38c0-4297-bdd8-92b082f46ff8/06be0d13-f4ff-478c-92b4-64c4ff1b6880"
-					(reference "#PWR054")
+					(reference "#PWR051")
 					(unit 1)
 				)
@@
 		(dnp no)
 		(fields_autoplaced yes)
-		(property "Reference" "LD42"
+		(property "Reference" "LD38"
 			(at 209.55 145.0974 90)
 			(show_name no)
@@
 			(project "HC4_KiCad"
 				(path "/33731ded-38c0-4297-bdd8-92b082f46ff8/06be0d13-f4ff-478c-92b4-64c4ff1b6880"
-					(reference "LD42")
+					(reference "LD38")
 					(unit 1)
 				)
@@
 		(dnp no)
 		(fields_autoplaced yes)
-		(property "Reference" "LD38"
+		(property "Reference" "LD34"
 			(at 172.72 145.0974 90)
 			(show_name no)
@@
 			(project "HC4_KiCad"
 				(path "/33731ded-38c0-4297-bdd8-92b082f46ff8/06be0d13-f4ff-478c-92b4-64c4ff1b6880"
-					(reference "LD38")
+					(reference "LD34")
 					(unit 1)
 				)
@@
 		(in_pos_files yes)
 		(dnp no)
-		(property "Reference" "#PWR057"
+		(property "Reference" "#PWR054"
 			(at 144.78 172.72 0)
 			(hide yes)
@@
 			(project "HC4_KiCad"
 				(path "/33731ded-38c0-4297-bdd8-92b082f46ff8/06be0d13-f4ff-478c-92b4-64c4ff1b6880"
-					(reference "#PWR057")
+					(reference "#PWR054")
 					(unit 1)
 				)
@@
 		(dnp no)
 		(fields_autoplaced yes)
-		(property "Reference" "LD37"
+		(property "Reference" "LD33"
 			(at 163.83 145.0974 90)
 			(show_name no)
@@
 			(project "HC4_KiCad"
 				(path "/33731ded-38c0-4297-bdd8-92b082f46ff8/06be0d13-f4ff-478c-92b4-64c4ff1b6880"
-					(reference "LD37")
+					(reference "LD33")
 					(unit 1)
 				)
@@
 		(dnp no)
 		(fields_autoplaced yes)
-		(property "Reference" "#PWR059"
+		(property "Reference" "#PWR056"
 			(at 168.91 166.37 0)
 			(hide yes)
@@
 			(project "HC4_KiCad"
 				(path "/33731ded-38c0-4297-bdd8-92b082f46ff8/06be0d13-f4ff-478c-92b4-64c4ff1b6880"
-					(reference "#PWR059")
+					(reference "#PWR056")
 					(unit 1)
 				)
@@
 		(dnp no)
 		(fields_autoplaced yes)
-		(property "Reference" "IC16"
+		(property "Reference" "IC15"
 			(at 124.1141 123.19 0)
 			(show_name no)
@@
 			(project "HC4_KiCad"
 				(path "/33731ded-38c0-4297-bdd8-92b082f46ff8/06be0d13-f4ff-478c-92b4-64c4ff1b6880"
-					(reference "IC16")
+					(reference "IC15")
 					(unit 1)
 				)
@@
 		(dnp no)
 		(fields_autoplaced yes)
-		(property "Reference" "#PWR052"
+		(property "Reference" "#PWR049"
 			(at 90.17 196.85 0)
 			(hide yes)
@@
 			(project "HC4_KiCad"
 				(path "/33731ded-38c0-4297-bdd8-92b082f46ff8/06be0d13-f4ff-478c-92b4-64c4ff1b6880"
-					(reference "#PWR052")
+					(reference "#PWR049")
 					(unit 1)
 				)
@@
 		(dnp no)
 		(fields_autoplaced yes)
-		(property "Reference" "LD41"
+		(property "Reference" "LD37"
 			(at 200.66 145.0974 90)
 			(show_name no)
@@
 			(project "HC4_KiCad"
 				(path "/33731ded-38c0-4297-bdd8-92b082f46ff8/06be0d13-f4ff-478c-92b4-64c4ff1b6880"
-					(reference "LD41")
+					(reference "LD37")
 					(unit 1)
 				)
@@
 		(dnp no)
 		(fields_autoplaced yes)
-		(property "Reference" "#PWR055"
+		(property "Reference" "#PWR052"
 			(at 121.92 125.73 0)
 			(hide yes)
@@
 			(project "HC4_KiCad"
 				(path "/33731ded-38c0-4297-bdd8-92b082f46ff8/06be0d13-f4ff-478c-92b4-64c4ff1b6880"
-					(reference "#PWR055")
+					(reference "#PWR052")
 					(unit 1)
 				)
@@
 		(dnp no)
 		(fields_autoplaced yes)
-		(property "Reference" "LD40"
+		(property "Reference" "LD36"
 			(at 191.77 145.0974 90)
 			(show_name no)
@@
 			(project "HC4_KiCad"
 				(path "/33731ded-38c0-4297-bdd8-92b082f46ff8/06be0d13-f4ff-478c-92b4-64c4ff1b6880"
-					(reference "LD40")
+					(reference "LD36")
 					(unit 1)
 				)
@@
 		(dnp no)
 		(fields_autoplaced yes)
-		(property "Reference" "#PWR056"
+		(property "Reference" "#PWR053"
 			(at 121.92 179.07 0)
 			(hide yes)
@@
 			(project "HC4_KiCad"
 				(path "/33731ded-38c0-4297-bdd8-92b082f46ff8/06be0d13-f4ff-478c-92b4-64c4ff1b6880"
-					(reference "#PWR056")
+					(reference "#PWR053")
 					(unit 1)
 				)
@@
 		(dnp no)
 		(fields_autoplaced yes)
-		(property "Reference" "#PWR051"
+		(property "Reference" "#PWR048"
 			(at 71.12 175.26 0)
 			(hide yes)
@@
 			(project "HC4_KiCad"
 				(path "/33731ded-38c0-4297-bdd8-92b082f46ff8/06be0d13-f4ff-478c-92b4-64c4ff1b6880"
-					(reference "#PWR051")
+					(reference "#PWR048")
 					(unit 1)
 				)
