File: HC4_KiCad/clockandreset.kicad_sch (KiCad schematic)
At the start: 16 parts, among them IC24 74HC14, SW3 SW_Push, SW4 SW_Push, SW5 SW_SPDT

Commit message: 基板ぬ
Parts:
- renumbered R7 to R15, R8 to R16, R9 to R17, R10 to R18, R11 to R19, RN8 to RN7
Changed lines of the file:
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@@
 		(dnp no)
 		(fields_autoplaced yes)
-		(property "Reference" "R7"
+		(property "Reference" "R15"
 			(at 46.99 86.36 90)
 			(effects
@@
 			(project ""
 				(path "/33731ded-38c0-4297-bdd8-92b082f46ff8/3d67359d-c55c-4207-8a6b-ff7c83e276f6"
-					(reference "R7")
+					(reference "R15")
 					(unit 1)
 				)
@@
 		(dnp no)
 		(fields_autoplaced yes)
-		(property "Reference" "RN8"
+		(property "Reference" "RN7"
 			(at 40.64 144.7799 0)
 			(effects
@@
 			(project ""
 				(path "/33731ded-38c0-4297-bdd8-92b082f46ff8/3d67359d-c55c-4207-8a6b-ff7c83e276f6"
-					(reference "RN8")
+					(reference "RN7")
 					(unit 2)
 				)
@@
 		(dnp no)
 		(fields_autoplaced yes)
-		(property "Reference" "RN8"
+		(property "Reference" "RN7"
 			(at 120.65 116.8399 0)
 			(effects
@@
 			(project ""
 				(path "/33731ded-38c0-4297-bdd8-92b082f46ff8/3d67359d-c55c-4207-8a6b-ff7c83e276f6"
-					(reference "RN8")
+					(reference "RN7")
 					(unit 4)
 				)
@@
 		(dnp no)
 		(fields_autoplaced yes)
-		(property "Reference" "R10"
+		(property "Reference" "R18"
 			(at 95.25 83.82 90)
 			(effects
@@
 			(project "HC4_KiCad"
 				(path "/33731ded-38c0-4297-bdd8-92b082f46ff8/3d67359d-c55c-4207-8a6b-ff7c83e276f6"
-					(reference "R10")
+					(reference "R18")
 					(unit 1)
 				)
@@
 		(dnp no)
 		(fields_autoplaced yes)
-		(property "Reference" "R8"
+		(property "Reference" "R16"
 			(at 48.26 144.78 90)
 			(effects
@@
 			(project "HC4_KiCad"
 				(path "/33731ded-38c0-4297-bdd8-92b082f46ff8/3d67359d-c55c-4207-8a6b-ff7c83e276f6"
-					(reference "R8")
+					(reference "R16")
 					(unit 1)
 				)
@@
 		(dnp no)
 		(fields_autoplaced yes)
-		(property "Reference" "RN8"
+		(property "Reference" "RN7"
 			(at 40.64 86.3599 0)
 			(effects
@@
 			(project ""
 				(path "/33731ded-38c0-4297-bdd8-92b082f46ff8/3d67359d-c55c-4207-8a6b-ff7c83e276f6"
-					(reference "RN8")
+					(reference "RN7")
 					(unit 1)
 				)
@@
 		(dnp no)
 		(fields_autoplaced yes)
-		(property "Reference" "R11"
+		(property "Reference" "R19"
 			(at 128.27 83.82 90)
 			(effects
@@
 			(project "HC4_KiCad"
 				(path "/33731ded-38c0-4297-bdd8-92b082f46ff8/3d67359d-c55c-4207-8a6b-ff7c83e276f6"
-					(reference "R11")
+					(reference "R19")
 					(unit 1)
 				)
@@
 		(dnp no)
 		(fields_autoplaced yes)
-		(property "Reference" "RN8"
+		(property "Reference" "RN7"
 			(at 110.49 116.8399 0)
 			(effects
@@
 			(project ""
 				(path "/33731ded-38c0-4297-bdd8-92b082f46ff8/3d67359d-c55c-4207-8a6b-ff7c83e276f6"
-					(reference "RN8")
+					(reference "RN7")
 					(unit 3)
 				)
@@
 		(dnp no)
 		(fields_autoplaced yes)
-		(property "Reference" "R9"
+		(property "Reference" "R17"
 			(at 58.42 48.2599 0)
 			(effects
@@
 			(project ""
 				(path "/33731ded-38c0-4297-bdd8-92b082f46ff8/3d67359d-c55c-4207-8a6b-ff7c83e276f6"
-					(reference "R9")
-					(unit 1)
-				)
+					(reference "R17")
+					(unit 1)
+				)

Commit message: Added output port for blink
Parts:
- renumbered LD40 to LD44, LD41 to LD45, SW3 to SW2, SW4 to SW3, SW5 to SW4
Changed lines of the file:
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@@
 		(on_board yes)
 		(dnp no)
-		(property "Reference" "SW5"
+		(property "Reference" "SW4"
 			(at 85.09 81.28 0)
 			(effects
@@
 			(project ""
 				(path "/33731ded-38c0-4297-bdd8-92b082f46ff8/3d67359d-c55c-4207-8a6b-ff7c83e276f6"
-					(reference "SW5")
+					(reference "SW4")
 					(unit 1)
 				)
@@
 		(on_board yes)
 		(dnp no)
-		(property "Reference" "SW3"
+		(property "Reference" "SW2"
 			(at 34.29 97.7899 90)
 			(effects
@@
 			(project "HC4_KiCad"
 				(path "/33731ded-38c0-4297-bdd8-92b082f46ff8/3d67359d-c55c-4207-8a6b-ff7c83e276f6"
-					(reference "SW3")
+					(reference "SW2")
 					(unit 1)
 				)
@@
 		(dnp no)
 		(fields_autoplaced yes)
-		(property "Reference" "#PWR083"
+		(property "Reference" "#PWR082"
 			(at 118.11 116.84 0)
 			(effects
@@
 			(project ""
 				(path "/33731ded-38c0-4297-bdd8-92b082f46ff8/3d67359d-c55c-4207-8a6b-ff7c83e276f6"
-					(reference "#PWR083")
+					(reference "#PWR082")
 					(unit 1)
 				)
@@
 		(dnp no)
 		(fields_autoplaced yes)
-		(property "Reference" "#PWR077"
+		(property "Reference" "#PWR076"
 			(at 38.1 111.76 0)
 			(effects
@@
 			(project "HC4_KiCad"
 				(path "/33731ded-38c0-4297-bdd8-92b082f46ff8/3d67359d-c55c-4207-8a6b-ff7c83e276f6"
-					(reference "#PWR077")
+					(reference "#PWR076")
 					(unit 1)
 				)
@@
 		(dnp no)
 		(fields_autoplaced yes)
-		(property "Reference" "#PWR080"
+		(property "Reference" "#PWR079"
 			(at 57.15 111.76 0)
 			(effects
@@
 			(project ""
 				(path "/33731ded-38c0-4297-bdd8-92b082f46ff8/3d67359d-c55c-4207-8a6b-ff7c83e276f6"
-					(reference "#PWR080")
+					(reference "#PWR079")
 					(unit 1)
 				)
@@
 		(dnp no)
 		(fields_autoplaced yes)
-		(property "Reference" "#PWR081"
+		(property "Reference" "#PWR080"
 			(at 57.15 170.18 0)
 			(effects
@@
 			(project "HC4_KiCad"
 				(path "/33731ded-38c0-4297-bdd8-92b082f46ff8/3d67359d-c55c-4207-8a6b-ff7c83e276f6"
-					(reference "#PWR081")
+					(reference "#PWR080")
 					(unit 1)
 				)
@@
 		(dnp no)
 		(fields_autoplaced yes)
-		(property "Reference" "LD40"
+		(property "Reference" "LD44"
 			(at 111.76 127.9524 90)
 			(effects
@@
 			(project ""
 				(path "/33731ded-38c0-4297-bdd8-92b082f46ff8/3d67359d-c55c-4207-8a6b-ff7c83e276f6"
-					(reference "LD40")
+					(reference "LD44")
 					(unit 1)
 				)
@@
 		(dnp no)
 		(fields_autoplaced yes)
-		(property "Reference" "#PWR079"
+		(property "Reference" "#PWR078"
 			(at 38.1 170.18 0)
 			(effects
@@
 			(project ""
 				(path "/33731ded-38c0-4297-bdd8-92b082f46ff8/3d67359d-c55c-4207-8a6b-ff7c83e276f6"
-					(reference "#PWR079")
+					(reference "#PWR078")
 					(unit 1)
 				)
@@
 		(dnp no)
 		(fields_autoplaced yes)
-		(property "Reference" "#PWR082"
+		(property "Reference" "#PWR081"
 			(at 107.95 116.84 0)
 			(effects
@@
 			(project "HC4_KiCad"
 				(path "/33731ded-38c0-4297-bdd8-92b082f46ff8/3d67359d-c55c-4207-8a6b-ff7c83e276f6"
-					(reference "#PWR082")
+					(reference "#PWR081")
 					(unit 1)
 				)
@@
 		(dnp no)
 		(fields_autoplaced yes)
-		(property "Reference" "LD41"
+		(property "Reference" "LD45"
 			(at 121.92 127.9524 90)
 			(effects
@@
 			(project "HC4_KiCad"
 				(path "/33731ded-38c0-4297-bdd8-92b082f46ff8/3d67359d-c55c-4207-8a6b-ff7c83e276f6"
-					(reference "LD41")
+					(reference "LD45")
 					(unit 1)
 				)
@@
 		(dnp no)
 		(fields_autoplaced yes)
-		(property "Reference" "#PWR078"
+		(property "Reference" "#PWR077"
 			(at 38.1 144.78 0)
 			(effects
@@
 			(project ""
 				(path "/33731ded-38c0-4297-bdd8-92b082f46ff8/3d67359d-c55c-4207-8a6b-ff7c83e276f6"
-					(reference "#PWR078")
+					(reference "#PWR077")
 					(unit 1)
 				)
@@
 		(dnp no)
 		(fields_autoplaced yes)
-		(property "Reference" "#PWR076"
+		(property "Reference" "#PWR075"
 			(at 38.1 86.36 0)
 			(effects
@@
 			(project "HC4_KiCad"
 				(path "/33731ded-38c0-4297-bdd8-92b082f46ff8/3d67359d-c55c-4207-8a6b-ff7c83e276f6"
-					(reference "#PWR076")
+					(reference "#PWR075")
 					(unit 1)
 				)
@@
 		(on_board yes)
 		(dnp no)
-		(property "Reference" "SW4"
+		(property "Reference" "SW3"
 			(at 34.29 156.2099 90)
 			(effects
@@
 			(project ""
 				(path "/33731ded-38c0-4297-bdd8-92b082f46ff8/3d67359d-c55c-4207-8a6b-ff7c83e276f6"
-					(reference "SW4")
+					(reference "SW3")
 					(unit 1)
 				)
@@
 		(dnp no)
 		(fields_autoplaced yes)
-		(property "Reference" "#PWR085"
+		(property "Reference" "#PWR084"
 			(at 156.21 196.85 0)
 			(effects
@@
 			(project ""
 				(path "/33731ded-38c0-4297-bdd8-92b082f46ff8/3d67359d-c55c-4207-8a6b-ff7c83e276f6"
-					(reference "#PWR085")
+					(reference "#PWR084")
 					(unit 1)
 				)
@@
 		(dnp no)
 		(fields_autoplaced yes)
-		(property "Reference" "#PWR084"
+		(property "Reference" "#PWR083"
 			(at 156.21 166.37 0)
 			(effects
@@
 			(project ""
 				(path "/33731ded-38c0-4297-bdd8-92b082f46ff8/3d67359d-c55c-4207-8a6b-ff7c83e276f6"
-					(reference "#PWR084")
-					(unit 1)
-				)
+					(reference "#PWR083")
+					(unit 1)
+				)

Commit message: ガーバーファイルを出力
Parts:
- C4: footprint Capacitor_THT:C_Radial_D5.0mm_H5.0mm_P2.00mm -> Capacitor_THT:C_Radial_D6.3mm_H5.0mm_P2.50mm
Changed lines of the file:
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@@
 			)
 		)
-		(property "Footprint" "Capacitor_THT:C_Radial_D5.0mm_H5.0mm_P2.00mm"
+		(property "Footprint" "Capacitor_THT:C_Radial_D6.3mm_H5.0mm_P2.50mm"
 			(at 68.58 40.9448 0)
 			(effects

Commit message: moti
Parts:
- IC23: renamed from IC24; footprint Package_SO:SO-14_5.3x10.2mm_P1.27mm -> Package_DIP:DIP-14_W7.62mm
- renumbered CP24 to CP23, R18 to R10, R19 to R11, R15 to R7, R16 to R8, R17 to R9, RN7 to RN8

Commit message: 基板途中
Parts:
- added D41: D, Diode_SMD:D_SOD-323_HandSoldering, symbol Device:D
- renumbered CP23 to CP22
Connections:
- net ~{RESET}: now also D41.1 (K)
- net at C4.1, IC23.1, R9.1: now also D41.2 (A)

Commit message: 仮
Parts:
- renumbered IC23 to IC22, LD44 to LD40, LD45 to LD41
Changed lines of the file:
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@@
 		(dnp no)
 		(fields_autoplaced yes)
-		(property "Reference" "IC23"
+		(property "Reference" "IC22"
 			(at 114.3 81.28 0)
 			(show_name no)
@@
 			(project "HC4_KiCad"
 				(path "/33731ded-38c0-4297-bdd8-92b082f46ff8/3d67359d-c55c-4207-8a6b-ff7c83e276f6"
-					(reference "IC23")
+					(reference "IC22")
 					(unit 6)
 				)
@@
 		(dnp no)
 		(fields_autoplaced yes)
-		(property "Reference" "IC23"
+		(property "Reference" "IC22"
 			(at 68.58 142.24 0)
 			(show_name no)
@@
 			(project "HC4_KiCad"
 				(path "/33731ded-38c0-4297-bdd8-92b082f46ff8/3d67359d-c55c-4207-8a6b-ff7c83e276f6"
-					(reference "IC23")
+					(reference "IC22")
 					(unit 3)
 				)
@@
 		(dnp no)
 		(fields_autoplaced yes)
-		(property "Reference" "#PWR080"
+		(property "Reference" "#PWR077"
 			(at 118.11 116.84 0)
 			(hide yes)
@@
 			(project "HC4_KiCad"
 				(path "/33731ded-38c0-4297-bdd8-92b082f46ff8/3d67359d-c55c-4207-8a6b-ff7c83e276f6"
-					(reference "#PWR080")
+					(reference "#PWR077")
 					(unit 1)
 				)
@@
 		(dnp no)
 		(fields_autoplaced yes)
-		(property "Reference" "IC23"
+		(property "Reference" "IC22"
 			(at 68.58 83.82 0)
 			(show_name no)
@@
 			(project "HC4_KiCad"
 				(path "/33731ded-38c0-4297-bdd8-92b082f46ff8/3d67359d-c55c-4207-8a6b-ff7c83e276f6"
-					(reference "IC23")
+					(reference "IC22")
 					(unit 5)
 				)
@@
 		(dnp no)
 		(fields_autoplaced yes)
-		(property "Reference" "#PWR074"
+		(property "Reference" "#PWR071"
 			(at 38.1 111.76 0)
 			(hide yes)
@@
 			(project "HC4_KiCad"
 				(path "/33731ded-38c0-4297-bdd8-92b082f46ff8/3d67359d-c55c-4207-8a6b-ff7c83e276f6"
-					(reference "#PWR074")
+					(reference "#PWR071")
 					(unit 1)
 				)
@@
 		(dnp no)
 		(fields_autoplaced yes)
-		(property "Reference" "#PWR077"
+		(property "Reference" "#PWR074"
 			(at 57.15 111.76 0)
 			(hide yes)
@@
 			(project "HC4_KiCad"
 				(path "/33731ded-38c0-4297-bdd8-92b082f46ff8/3d67359d-c55c-4207-8a6b-ff7c83e276f6"
-					(reference "#PWR077")
+					(reference "#PWR074")
 					(unit 1)
 				)
@@
 		(dnp no)
 		(fields_autoplaced yes)
-		(property "Reference" "#PWR078"
+		(property "Reference" "#PWR075"
 			(at 57.15 170.18 0)
 			(hide yes)
@@
 			(project "HC4_KiCad"
 				(path "/33731ded-38c0-4297-bdd8-92b082f46ff8/3d67359d-c55c-4207-8a6b-ff7c83e276f6"
-					(reference "#PWR078")
+					(reference "#PWR075")
 					(unit 1)
 				)
@@
 		(dnp no)
 		(fields_autoplaced yes)
-		(property "Reference" "LD44"
+		(property "Reference" "LD40"
 			(at 111.76 127.9524 90)
 			(show_name no)
@@
 			(project "HC4_KiCad"
 				(path "/33731ded-38c0-4297-bdd8-92b082f46ff8/3d67359d-c55c-4207-8a6b-ff7c83e276f6"
-					(reference "LD44")
+					(reference "LD40")
 					(unit 1)
 				)
@@
 		(dnp no)
 		(fields_autoplaced yes)
-		(property "Reference" "#PWR076"
+		(property "Reference" "#PWR073"
 			(at 38.1 170.18 0)
 			(hide yes)
@@
 			(project "HC4_KiCad"
 				(path "/33731ded-38c0-4297-bdd8-92b082f46ff8/3d67359d-c55c-4207-8a6b-ff7c83e276f6"
-					(reference "#PWR076")
+					(reference "#PWR073")
 					(unit 1)
 				)
@@
 		(dnp no)
 		(fields_autoplaced yes)
-		(property "Reference" "#PWR079"
+		(property "Reference" "#PWR076"
 			(at 107.95 116.84 0)
 			(hide yes)
@@
 			(project "HC4_KiCad"
 				(path "/33731ded-38c0-4297-bdd8-92b082f46ff8/3d67359d-c55c-4207-8a6b-ff7c83e276f6"
-					(reference "#PWR079")
+					(reference "#PWR076")
 					(unit 1)
 				)
@@
 		(dnp no)
 		(fields_autoplaced yes)
-		(property "Reference" "LD45"
+		(property "Reference" "LD41"
 			(at 121.92 127.9524 90)
 			(show_name no)
@@
 			(project "HC4_KiCad"
 				(path "/33731ded-38c0-4297-bdd8-92b082f46ff8/3d67359d-c55c-4207-8a6b-ff7c83e276f6"
-					(reference "LD45")
+					(reference "LD41")
 					(unit 1)
 				)
@@
 		(dnp no)
 		(fields_autoplaced yes)
-		(property "Reference" "IC23"
+		(property "Reference" "IC22"
 			(at 64.77 54.61 0)
 			(show_name no)
@@
 			(project "HC4_KiCad"
 				(path "/33731ded-38c0-4297-bdd8-92b082f46ff8/3d67359d-c55c-4207-8a6b-ff7c83e276f6"
-					(reference "IC23")
+					(reference "IC22")
 					(unit 2)
 				)
@@
 		(dnp no)
 		(fields_autoplaced yes)
-		(property "Reference" "#PWR075"
+		(property "Reference" "#PWR072"
 			(at 38.1 144.78 0)
 			(hide yes)
@@
 			(project "HC4_KiCad"
 				(path "/33731ded-38c0-4297-bdd8-92b082f46ff8/3d67359d-c55c-4207-8a6b-ff7c83e276f6"
-					(reference "#PWR075")
+					(reference "#PWR072")
 					(unit 1)
 				)
@@
 		(dnp no)
 		(fields_autoplaced yes)
-		(property "Reference" "IC23"
+		(property "Reference" "IC22"
 			(at 162.56 175.2599 0)
 			(show_name no)
@@
 			(project "HC4_KiCad"
 				(path "/33731ded-38c0-4297-bdd8-92b082f46ff8/3d67359d-c55c-4207-8a6b-ff7c83e276f6"
-					(reference "IC23")
+					(reference "IC22")
 					(unit 7)
 				)
@@
 		(dnp no)
 		(fields_autoplaced yes)
-		(property "Reference" "#PWR073"
+		(property "Reference" "#PWR070"
 			(at 38.1 86.36 0)
 			(hide yes)
@@
 			(project "HC4_KiCad"
 				(path "/33731ded-38c0-4297-bdd8-92b082f46ff8/3d67359d-c55c-4207-8a6b-ff7c83e276f6"
-					(reference "#PWR073")
+					(reference "#PWR070")
 					(unit 1)
 				)
@@
 		(dnp no)
 		(fields_autoplaced yes)
-		(property "Reference" "IC23"
+		(property "Reference" "IC22"
 			(at 46.99 54.61 0)
 			(show_name no)
@@
 			(project "HC4_KiCad"
 				(path "/33731ded-38c0-4297-bdd8-92b082f46ff8/3d67359d-c55c-4207-8a6b-ff7c83e276f6"
-					(reference "IC23")
+					(reference "IC22")
 					(unit 1)
 				)
@@
 		(dnp no)
 		(fields_autoplaced yes)
-		(property "Reference" "IC23"
+		(property "Reference" "IC22"
 			(at 85.09 142.24 0)
 			(show_name no)
@@
 			(project "HC4_KiCad"
 				(path "/33731ded-38c0-4297-bdd8-92b082f46ff8/3d67359d-c55c-4207-8a6b-ff7c83e276f6"
-					(reference "IC23")
+					(reference "IC22")
 					(unit 4)
 				)
@@
 		(dnp no)
 		(fields_autoplaced yes)
-		(property "Reference" "#PWR082"
+		(property "Reference" "#PWR079"
 			(at 156.21 196.85 0)
 			(hide yes)
@@
 			(project "HC4_KiCad"
 				(path "/33731ded-38c0-4297-bdd8-92b082f46ff8/3d67359d-c55c-4207-8a6b-ff7c83e276f6"
-					(reference "#PWR082")
+					(reference "#PWR079")
 					(unit 1)
 				)
@@
 		(dnp no)
 		(fields_autoplaced yes)
-		(property "Reference" "#PWR081"
+		(property "Reference" "#PWR078"
 			(at 156.21 166.37 0)
 			(hide yes)
@@
 			(project "HC4_KiCad"
 				(path "/33731ded-38c0-4297-bdd8-92b082f46ff8/3d67359d-c55c-4207-8a6b-ff7c83e276f6"
-					(reference "#PWR081")
+					(reference "#PWR078")
 					(unit 1)
 				)
