File: HC4_KiCad/HC4_KiCad.kicad_sch (KiCad schematic)
At the start: 17 parts, among them IC1 ROM, J1 Power

Commit message: 配線完了とみられる
Changed lines of the file:
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@@
 (kicad_sch
-	(version 20231120)
+	(version 20250114)
 	(generator "eeschema")
-	(generator_version "8.0")
+	(generator_version "9.0")
 	(paper "A4")
 	(title_block
@@
 		(rev "1.3")
 	)
+	(text "When using a 6116 type SRAM, \nClose 2-3 of JP1"
+		(exclude_from_sim no)
+		(at 45.466 118.872 0)
+		(effects
+			(font
+				(size 1.27 1.27)
+			)
+		)
+	)
+	(text "DATA BUS"
+		(exclude_from_sim yes)
+		(at 164.338 36.068 0)
+		(effects
+			(font
+				(size 5.08 5.08)
+				(thickness 1.016)
+				(bold yes)
+			)
+		)
+	)
 	(junction
 		(at 161.29 116.84)
@@
 		)
 	)
-	(text "When using a 6116 type SRAM, \nClose 2-3 of JP1"
-		(exclude_from_sim no)
-		(at 45.466 118.872 0)
-		(effects
-			(font
-				(size 1.27 1.27)
-			)
-		)
-	)
-	(text "DATA BUS"
-		(exclude_from_sim yes)
-		(at 164.338 36.068 0)
-		(effects
-			(font
-				(size 5.08 5.08)
-				(thickness 1.016)
-				(bold yes)
-			)
-		)
-	)
 	(label "Instruction_4"
 		(at 251.46 101.6 180)
@@
 		(at 30.48 144.78)
 		(size 134.62 7.62)
+		(exclude_from_sim no)
+		(in_bom yes)
+		(on_board yes)
+		(dnp no)
 		(stroke
 			(width 0.1524)
@@
 		(at 160.02 48.26)
 		(size 78.74 27.94)
+		(exclude_from_sim no)
+		(in_bom yes)
+		(on_board yes)
+		(dnp no)
 		(stroke
 			(width 0.1524)
@@
 		(at 96.52 50.8)
 		(size 46.99 20.32)
+		(exclude_from_sim no)
+		(in_bom yes)
+		(on_board yes)
+		(dnp no)
 		(stroke
 			(width 0.1524)
@@
 		(at 25.4 31.75)
 		(size 245.11 7.62)
+		(exclude_from_sim no)
+		(in_bom yes)
+		(on_board yes)
+		(dnp no)
 		(fields_autoplaced yes)
 		(stroke
@@
 		(at 248.92 148.59)
 		(size 25.4 11.43)
+		(exclude_from_sim no)
+		(in_bom yes)
+		(on_board yes)
+		(dnp no)
 		(fields_autoplaced yes)
 		(stroke
@@
 		(at 96.52 82.55)
 		(size 46.99 31.75)
+		(exclude_from_sim no)
+		(in_bom yes)
+		(on_board yes)
+		(dnp no)
 		(stroke
 			(width 0.1524)
@@
 		(at 156.21 118.11)
 		(size 34.29 13.97)
+		(exclude_from_sim no)
+		(in_bom yes)
+		(on_board yes)
+		(dnp no)
 		(stroke
 			(width 0.1524)
@@
 		)
 	)
+	(embedded_fonts no)
 )

Commit message: リビジョン番号いれた
Other:
- note removed: "When using a 6116 type SRAM, Close 2-3 of JP1"
Changed lines of the file:
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@@
 	(title_block
 		(title "HC4_CPU")
-		(date "2025-03-31")
-		(rev "1.3")
-	)
-	(text "When using a 6116 type SRAM, \nClose 2-3 of JP1"
-		(exclude_from_sim no)
-		(at 45.466 118.872 0)
-		(effects
-			(font
-				(size 1.27 1.27)
-			)
-		)
+		(date "2025-04-17")
+		(rev "2.0")
 	)
 	(text "DATA BUS"
@@
 	(bus
 		(pts
-			(xy 161.29 116.84) (xy 144.78 116.84)
+			(xy 161.29 116.84) (xy 146.05 116.84)
 		)
 		(stroke
@@
 	(bus
 		(pts
-			(xy 165.1 146.05) (xy 205.74 146.05)
+			(xy 176.53 146.05) (xy 210.82 146.05)
 		)
 		(stroke
@@
 	(wire
 		(pts
-			(xy 199.39 148.59) (xy 165.1 148.59)
-		)
-		(stroke
-			(width 0)
-			(type default)
-		)
-	)
-	(wire
-		(pts
 			(xy 190.5 99.06) (xy 190.5 76.2)
 		)
@@
 	(bus
 		(pts
-			(xy 205.74 156.21) (xy 246.38 156.21)
+			(xy 210.82 156.21) (xy 246.38 156.21)
 		)
 		(stroke
@@
 	(polyline
 		(pts
-			(xy 15.24 35.56) (xy 25.4 45.72)
+			(xy 25.4 35.56) (xy 35.56 45.72)
 		)
 		(stroke
@@
 	(bus
 		(pts
-			(xy 44.45 144.78) (xy 44.45 127)
-		)
-		(stroke
-			(width 0)
-			(type default)
-		)
-	)
-	(bus
-		(pts
 			(xy 254 39.37) (xy 254 71.12)
 		)
@@
 		)
 	)
-	(bus
-		(pts
-			(xy 55.88 48.26) (xy 22.86 48.26)
-		)
-		(stroke
-			(width 0)
-			(type default)
-		)
-	)
 	(wire
 		(pts
@@
 	(polyline
 		(pts
-			(xy 30.48 143.51) (xy 30.48 144.78)
+			(xy 38.1 143.51) (xy 38.1 144.78)
 		)
 		(stroke
@@
 	(polyline
 		(pts
-			(xy 30.48 138.43) (xy 30.48 144.78)
+			(xy 38.1 138.43) (xy 38.1 144.78)
 		)
 		(stroke
@@
 	(polyline
 		(pts
-			(xy 165.1 143.51) (xy 165.1 144.78)
+			(xy 176.53 143.51) (xy 176.53 144.78)
 		)
 		(stroke
@@
 	(polyline
 		(pts
-			(xy 15.24 35.56) (xy 25.4 25.4)
+			(xy 25.4 35.56) (xy 35.56 25.4)
 		)
 		(stroke
@@
 	(polyline
 		(pts
-			(xy 165.1 152.4) (xy 165.1 158.75)
+			(xy 176.53 152.4) (xy 176.53 158.75)
 		)
 		(stroke
@@
 	(polyline
 		(pts
-			(xy 20.32 148.59) (xy 30.48 158.75)
+			(xy 27.94 148.59) (xy 38.1 158.75)
 		)
 		(stroke
@@
 	(bus
 		(pts
-			(xy 44.45 127) (xy 22.86 127)
-		)
-		(stroke
-			(width 0)
-			(type default)
-		)
-	)
-	(bus
-		(pts
 			(xy 101.6 71.12) (xy 101.6 81.28)
 		)
@@
 	(wire
 		(pts
+			(xy 176.53 148.59) (xy 199.39 148.59)
+		)
+		(stroke
+			(width 0)
+			(type default)
+		)
+	)
+	(wire
+		(pts
 			(xy 208.28 109.22) (xy 217.17 109.22)
 		)
@@
 	(polyline
 		(pts
-			(xy 25.4 25.4) (xy 25.4 31.75)
+			(xy 35.56 25.4) (xy 35.56 31.75)
 		)
 		(stroke
@@
 	(bus
 		(pts
-			(xy 144.78 116.84) (xy 144.78 144.78)
+			(xy 146.05 116.84) (xy 146.05 144.78)
 		)
 		(stroke
@@
 	(polyline
 		(pts
-			(xy 25.4 39.37) (xy 25.4 45.72)
+			(xy 35.56 39.37) (xy 35.56 45.72)
 		)
 		(stroke
@@
 	(bus
 		(pts
-			(xy 55.88 39.37) (xy 55.88 48.26)
+			(xy 55.88 39.37) (xy 55.88 144.78)
 		)
 		(stroke
@@
 	(bus
 		(pts
-			(xy 142.24 115.57) (xy 142.24 144.78)
+			(xy 143.51 115.57) (xy 143.51 144.78)
 		)
 		(stroke
@@
 	(polyline
 		(pts
-			(xy 175.26 148.59) (xy 165.1 158.75)
+			(xy 186.69 148.59) (xy 176.53 158.75)
 		)
 		(stroke
@@
 	(polyline
 		(pts
-			(xy 30.48 152.4) (xy 30.48 158.75)
+			(xy 38.1 152.4) (xy 38.1 158.75)
 		)
 		(stroke
@@
 		)
 	)
-	(bus
-		(pts
-			(xy 22.86 48.26) (xy 22.86 127)
-		)
-		(stroke
-			(width 0)
-			(type default)
-		)
-	)
 	(wire
 		(pts
@@
 	(polyline
 		(pts
-			(xy 175.26 148.59) (xy 165.1 138.43)
+			(xy 186.69 148.59) (xy 176.53 138.43)
 		)
 		(stroke
@@
 	(bus
 		(pts
-			(xy 205.74 146.05) (xy 205.74 156.21)
+			(xy 210.82 146.05) (xy 210.82 156.21)
 		)
 		(stroke
@@
 	(polyline
 		(pts
-			(xy 20.32 148.59) (xy 30.48 138.43)
+			(xy 27.94 148.59) (xy 38.1 138.43)
 		)
 		(stroke
@@
 	(polyline
 		(pts
-			(xy 165.1 138.43) (xy 165.1 144.78)
+			(xy 176.53 138.43) (xy 176.53 144.78)
 		)
 		(stroke
@@
 	(polyline
 		(pts
-			(xy 25.4 30.48) (xy 25.4 31.75)
+			(xy 35.56 30.48) (xy 35.56 31.75)
 		)
 		(stroke
@@
 	(bus
 		(pts
-			(xy 142.24 115.57) (xy 158.75 115.57)
+			(xy 143.51 115.57) (xy 158.75 115.57)
 		)
 		(stroke
@@
 	)
 	(sheet
-		(at 30.48 144.78)
-		(size 134.62 7.62)
+		(at 38.1 144.78)
+		(size 138.43 7.62)
 		(exclude_from_sim no)
 		(in_bom yes)
@@
 		)
 		(property "Sheetname" "Address BUS"
-			(at 75.438 144.272 0)
+			(at 83.058 144.272 0)
 			(effects
 				(font
@@
 		)
 		(property "Sheetfile" "addressbus.kicad_sch"
-			(at 74.422 153.162 0)
+			(at 82.042 153.162 0)
 			(effects
 				(font
@@
 		)
 		(pin "Instruction_[0..7]" input
-			(at 165.1 146.05 0)
+			(at 176.53 146.05 0)
 			(effects
 				(font
@@
 		)
 		(pin "Level_A[0..3]" input
-			(at 142.24 144.78 90)
+			(at 143.51 144.78 90)
 			(effects
 				(font
@@
 		)
 		(pin "Level_B[0..3]" input
-			(at 144.78 144.78 90)
+			(at 146.05 144.78 90)
 			(effects
 				(font
@@
 		)
 		(pin "MEMMode" input
-			(at 165.1 148.59 0)
+			(at 176.53 148.59 0)
 			(effects
 				(font
@@
 		)
 		(pin "RAM_A[0..7]" output
-			(at 44.45 144.78 90)
+			(at 55.88 144.78 90)
 			(effects
 				(font
@@
 	)
 	(sheet
-		(at 25.4 31.75)
-		(size 245.11 7.62)
+		(at 35.56 31.75)
+		(size 234.95 7.62)
 		(exclude_from_sim no)
 		(in_bom yes)
 		(on_board yes)
 		(dnp no)
-		(fields_autoplaced yes)
 		(stroke
 			(width 0.1524)
@@
 		)
 		(property "Sheetname" "Data BUS"
-			(at 25.4 31.0384 0)
+			(at 35.814 31.242 0)
 			(effects
 				(font
@@
 		)
 		(property "Sheetfile" "databus.kicad_sch"
-			(at 25.4 39.9546 0)
+			(at 58.674 29.972 0)
 			(effects
 				(font

Commit message: moti
Parts:
- removed CP2: 0.1u, Capacitor_SMD:C_0603_1608Metric, symbol Device2:C_Bypass
- removed D1: 5.6V, Diode_THT:D_DO-34_SOD68_P7.62mm_Horizontal, symbol Device:D_Zener
- removed IC1: ROM, Socket:DIP_Socket-28_W11.9_W12.7_W15.24_W17.78_W18.5_3M_228-1277-00-0602J, symbol Memory_EPROM:27256
- added J2: ROMCard, Connector_PinHeader_2.54mm:PinHeader_2x20_P2.54mm_Vertical, symbol Connector_Generic:Conn_02x20_Top_Bottom
Connections:
- net GND: now also J2.19 (Pin_19), J2.20 (Pin_20), J2.39 (Pin_39), J2.40 (Pin_40)
- net Instruction_0: now also J2.21 (Pin_21)
- net Instruction_1: now also J2.22 (Pin_22)
- net Instruction_2: now also J2.23 (Pin_23)
- net Instruction_3: now also J2.24 (Pin_24)
- net Instruction_4: now also J2.25 (Pin_25)
- net Instruction_5: now also J2.26 (Pin_26)
- net Instruction_6: now also J2.27 (Pin_27)
- net Instruction_7: now also J2.28 (Pin_28)
- net PC_0: now also J2.3 (Pin_3)
- net PC_1: now also J2.4 (Pin_4)
- net PC_10: now also J2.13 (Pin_13)
- net PC_11: now also J2.14 (Pin_14)
- net PC_2: now also J2.5 (Pin_5)
- net PC_3: now also J2.6 (Pin_6)
- net PC_4: now also J2.7 (Pin_7)
- net PC_5: now also J2.8 (Pin_8)
- net PC_6: now also J2.9 (Pin_9)
- net PC_7: now also J2.10 (Pin_10)
- net PC_8: now also J2.11 (Pin_11)
- net PC_9: now also J2.12 (Pin_12)
- net VCC: now also J2.1 (Pin_1), J2.15 (Pin_15), J2.16 (Pin_16), J2.17 (Pin_17), J2.18 (Pin_18), J2.2 (Pin_2)
- no-connect marks 0 -> 10
Other:
- note added: "~{CE}"
- note added: "~{OE}"

Commit message: 基板途中
Parts:
- removed CP1: 0.1u, Capacitor_SMD:C_0603_1608Metric, symbol Device2:C_Bypass
- removed J2: ROMCard, Connector_PinHeader_2.54mm:PinHeader_2x20_P2.54mm_Vertical, symbol Connector_Generic:Conn_02x20_Top_Bottom
- added J2: Conn_02x12_Odd_Even, Connector_PinHeader_2.54mm:PinHeader_2x12_P2.54mm_Vertical, symbol Connector_Generic:Conn_02x12_Odd_Even
Connections:
- net GND: now also J2.18 (Pin_18), J2.20 (Pin_20), J2.22 (Pin_22)
- net Instruction_0: now also J2.2 (Pin_2)
- net Instruction_1: now also J2.4 (Pin_4)
- net Instruction_2: now also J2.6 (Pin_6)
- net Instruction_3: now also J2.8 (Pin_8)
- net Instruction_4: now also J2.10 (Pin_10)
- net Instruction_5: now also J2.12 (Pin_12)
- net Instruction_6: now also J2.14 (Pin_14)
- net Instruction_7: now also J2.16 (Pin_16)
- net PC_0: now also J2.1 (Pin_1)
- net PC_1: now also J2.3 (Pin_3)
- net PC_10: now also J2.21 (Pin_21)
- net PC_11: now also J2.23 (Pin_23)
- net PC_2: now also J2.5 (Pin_5)
- net PC_3: now also J2.7 (Pin_7)
- net PC_4: now also J2.9 (Pin_9)
- net PC_5: now also J2.11 (Pin_11)
- net PC_6: now also J2.13 (Pin_13)
- net PC_7: now also J2.15 (Pin_15)
- net PC_8: now also J2.17 (Pin_17)
- net PC_9: now also J2.19 (Pin_19)
- net VCC: now also J2.24 (Pin_24)
- no-connect marks 10 -> 0
Other:
- note removed: "~{CE}"
- note removed: "~{OE}"

Commit message: 仮
Parts:
- removed J2: Conn_02x12_Odd_Even, Connector_PinHeader_2.54mm:PinHeader_2x12_P2.54mm_Vertical, symbol Connector_Generic:Conn_02x12_Odd_Even
- added J2: Conn_02x12_Counter_Clockwise, Connector_PinHeader_2.54mm:PinHeader_2x12_P2.54mm_Vertical, symbol Connector_Generic:Conn_02x12_Counter_Clockwise
Connections:
- net GND: now also LD2.1 (K), LD3.1 (K), J2.22 (Pin_22), J2.23 (Pin_23), J2.24 (Pin_24); no longer R2.2, R3.2
- net Instruction Decoder/Carry_Flg: now also R3.1; no longer LD3.2
- net Instruction Decoder/Zero_Flg: now also R2.1; no longer LD2.2
- net Instruction_0: now also J2.20 (Pin_20)
- net Instruction_1: now also J2.19 (Pin_19)
- net Instruction_2: now also J2.18 (Pin_18)
- net Instruction_3: now also J2.17 (Pin_17)
- net Instruction_4: now also J2.16 (Pin_16)
- net Instruction_5: now also J2.15 (Pin_15)
- net Instruction_6: now also J2.14 (Pin_14)
- net Instruction_7: now also J2.13 (Pin_13)
- net PC_0: now also J2.1 (Pin_1)
- net PC_1: now also J2.2 (Pin_2)
- net PC_10: now also J2.11 (Pin_11)
- net PC_11: now also J2.12 (Pin_12)
- net PC_2: now also J2.3 (Pin_3)
- net PC_3: now also J2.4 (Pin_4)
- net PC_4: now also J2.5 (Pin_5)
- net PC_5: now also J2.6 (Pin_6)
- net PC_6: now also J2.7 (Pin_7)
- net PC_7: now also J2.8 (Pin_8)
- net PC_8: now also J2.9 (Pin_9)
- net PC_9: now also J2.10 (Pin_10)
- net VCC: now also J2.21 (Pin_21)
- new net: LD3.2, R3.2
- new net: LD2.2, R2.2
Other:
- moved on the sheet: LD2, LD3, R2, R3
