File: HC4_KiCad/databus.kicad_sch (KiCad schematic)
At the start: 18 parts, among them IC6 74HC257, IC7 74HC244, IC8 74HC4002, IC9 74HC374, J3 Expantion_Connector

Commit message: 基板途中
Parts:
- removed RN2: 10k, Resistor_THT:R_Array_SIP9, symbol Device:R_Network08_Split
- added RN2: 10k, Resistor_THT:R_Array_SIP5, symbol Device:R_Network04_Split
- renumbered CP7 to CP6, CP8 to CP7
Connections:
- net Databus0: now also RN2.2 (R1.2)
- net Databus1: now also RN2.3 (R2.2)
- net Databus2: now also RN2.4 (R3.2)
- net Databus3: now also RN2.5 (R4.2)
- net VCC: now also RN2.1 (R1), RN2.1 (R1), RN2.1 (R1), RN2.1 (R1)
- net Dummy4: no longer names the net of J3.7 (Pin_7)
- net Dummy5: no longer names the net of J3.8 (Pin_8)
- net Dummy6: no longer names the net of J3.9 (Pin_9)
- net Dummy7: no longer names the net of J3.10 (Pin_10)
- no-connect marks 14 -> 18

Commit message: 仮
Parts:
- removed IC9: 74HC374, Package_DIP:DIP-20_W7.62mm, symbol 74xx_2:74HC374
- removed JP1: Blink_EN, Connector_PinSocket_2.54mm:PinSocket_1x02_P2.54mm_Vertical, symbol Jumper:Jumper_2_Bridged
- removed LD10, LD11, LD8, LD9: LED, LED_THT:LED_Rectangular_W5.0mm_H2.0mm, symbol Device2:LED_
- removed RN1: 1k, Resistor_THT:R_Array_SIP9, symbol Device:R_Network08_Split
- added RN1: 1k, Resistor_THT:R_Array_SIP5, symbol Device:R_Network04_Split
Connections:
- net GND: now also RN1.2 (R1.2), RN1.3 (R2.2), RN1.4 (R3.2), RN1.5 (R4.2)
- net at LD6.1 (K): now also RN1.1 (R1)
- net at LD7.1 (K): now also RN1.1 (R1)
- net at LD5.1 (K): now also RN1.1 (R1)
- net at LD4.1 (K): now also RN1.1 (R1)
- net PA0: no longer names the net of J3.31 (Pin_31)
- net PA1: no longer names the net of J3.32 (Pin_32)
- net PA2: no longer names the net of J3.33 (Pin_33)
- net PA3: no longer names the net of J3.34 (Pin_34)
- no-connect marks 18 -> 22
