File: HC4_KiCad/stackunit.kicad_sch (KiCad schematic)
At the start: 18 parts, among them IC10 74HC161, IC11 74HC377

Commit message: 基板途中
Parts:
- renumbered CP9 to CP8, CP10 to CP9

Commit message: 仮
Parts:
- renumbered IC11 to IC10, IC10 to IC9, LD14 to LD10, LD15 to LD11, LD16 to LD12, LD17 to LD13, LD18 to LD14, LD19 to LD15, LD20 to LD16, LD21 to LD17, LD22 to LD18, LD23 to LD19, LD12 to LD8, LD13 to LD9
Changed lines of the file:
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@@
 		(in_pos_files yes)
 		(dnp no)
-		(property "Reference" "LD14"
+		(property "Reference" "LD10"
 			(at 148.59 143.8274 90)
 			(show_name no)
@@
 			(project "HC4_KiCad"
 				(path "/33731ded-38c0-4297-bdd8-92b082f46ff8/27e10803-908c-4418-a733-f902d25b5ad6"
-					(reference "LD14")
+					(reference "LD10")
 					(unit 1)
 				)
@@
 		(in_pos_files yes)
 		(dnp no)
-		(property "Reference" "#PWR038"
+		(property "Reference" "#PWR035"
 			(at 167.64 81.28 0)
 			(hide yes)
@@
 			(project "HC4_KiCad"
 				(path "/33731ded-38c0-4297-bdd8-92b082f46ff8/27e10803-908c-4418-a733-f902d25b5ad6"
-					(reference "#PWR038")
+					(reference "#PWR035")
 					(unit 1)
 				)
@@
 		(in_pos_files yes)
 		(dnp no)
-		(property "Reference" "LD15"
+		(property "Reference" "LD11"
 			(at 153.67 143.8274 90)
 			(show_name no)
@@
 			(project "HC4_KiCad"
 				(path "/33731ded-38c0-4297-bdd8-92b082f46ff8/27e10803-908c-4418-a733-f902d25b5ad6"
-					(reference "LD15")
+					(reference "LD11")
 					(unit 1)
 				)
@@
 		(in_pos_files yes)
 		(dnp no)
-		(property "Reference" "LD21"
+		(property "Reference" "LD17"
 			(at 184.15 143.8274 90)
 			(show_name no)
@@
 			(project "HC4_KiCad"
 				(path "/33731ded-38c0-4297-bdd8-92b082f46ff8/27e10803-908c-4418-a733-f902d25b5ad6"
-					(reference "LD21")
+					(reference "LD17")
 					(unit 1)
 				)
@@
 		(in_pos_files yes)
 		(dnp no)
-		(property "Reference" "LD23"
+		(property "Reference" "LD19"
 			(at 194.31 143.8274 90)
 			(show_name no)
@@
 			(project "HC4_KiCad"
 				(path "/33731ded-38c0-4297-bdd8-92b082f46ff8/27e10803-908c-4418-a733-f902d25b5ad6"
-					(reference "LD23")
+					(reference "LD19")
 					(unit 1)
 				)
@@
 		(dnp no)
 		(fields_autoplaced yes)
-		(property "Reference" "IC11"
+		(property "Reference" "IC10"
 			(at 169.8341 81.28 0)
 			(show_name no)
@@
 			(project "HC4_KiCad"
 				(path "/33731ded-38c0-4297-bdd8-92b082f46ff8/27e10803-908c-4418-a733-f902d25b5ad6"
-					(reference "IC11")
+					(reference "IC10")
 					(unit 1)
 				)
@@
 		(dnp no)
 		(fields_autoplaced yes)
-		(property "Reference" "#PWR035"
+		(property "Reference" "#PWR032"
 			(at 100.33 149.86 0)
 			(hide yes)
@@
 			(project "HC4_KiCad"
 				(path "/33731ded-38c0-4297-bdd8-92b082f46ff8/27e10803-908c-4418-a733-f902d25b5ad6"
-					(reference "#PWR035")
+					(reference "#PWR032")
 					(unit 1)
 				)
@@
 		(in_pos_files yes)
 		(dnp no)
-		(property "Reference" "LD19"
+		(property "Reference" "LD15"
 			(at 173.99 143.8274 90)
 			(show_name no)
@@
 			(project "HC4_KiCad"
 				(path "/33731ded-38c0-4297-bdd8-92b082f46ff8/27e10803-908c-4418-a733-f902d25b5ad6"
-					(reference "LD19")
+					(reference "LD15")
 					(unit 1)
 				)
@@
 		(in_pos_files yes)
 		(dnp no)
-		(property "Reference" "#PWR037"
+		(property "Reference" "#PWR034"
 			(at 137.16 165.1 0)
 			(hide yes)
@@
 			(project "HC4_KiCad"
 				(path "/33731ded-38c0-4297-bdd8-92b082f46ff8/27e10803-908c-4418-a733-f902d25b5ad6"
-					(reference "#PWR037")
+					(reference "#PWR034")
 					(unit 1)
 				)
@@
 		(in_pos_files yes)
 		(dnp no)
-		(property "Reference" "LD12"
+		(property "Reference" "LD8"
 			(at 138.43 143.8274 90)
 			(show_name no)
@@
 			(project "HC4_KiCad"
 				(path "/33731ded-38c0-4297-bdd8-92b082f46ff8/27e10803-908c-4418-a733-f902d25b5ad6"
-					(reference "LD12")
+					(reference "LD8")
 					(unit 1)
 				)
@@
 		(in_pos_files yes)
 		(dnp no)
-		(property "Reference" "#PWR036"
+		(property "Reference" "#PWR033"
 			(at 100.33 160.02 0)
 			(hide yes)
@@
 			(project "HC4_KiCad"
 				(path "/33731ded-38c0-4297-bdd8-92b082f46ff8/27e10803-908c-4418-a733-f902d25b5ad6"
-					(reference "#PWR036")
+					(reference "#PWR033")
 					(unit 1)
 				)
@@
 		(in_pos_files yes)
 		(dnp no)
-		(property "Reference" "LD20"
+		(property "Reference" "LD16"
 			(at 179.07 143.8274 90)
 			(show_name no)
@@
 			(project "HC4_KiCad"
 				(path "/33731ded-38c0-4297-bdd8-92b082f46ff8/27e10803-908c-4418-a733-f902d25b5ad6"
-					(reference "LD20")
+					(reference "LD16")
 					(unit 1)
 				)
@@
 		(in_pos_files yes)
 		(dnp no)
-		(property "Reference" "LD18"
+		(property "Reference" "LD14"
 			(at 168.91 143.8274 90)
 			(show_name no)
@@
 			(project "HC4_KiCad"
 				(path "/33731ded-38c0-4297-bdd8-92b082f46ff8/27e10803-908c-4418-a733-f902d25b5ad6"
-					(reference "LD18")
+					(reference "LD14")
 					(unit 1)
 				)
@@
 		(in_pos_files yes)
 		(dnp no)
-		(property "Reference" "LD16"
+		(property "Reference" "LD12"
 			(at 158.75 143.8274 90)
 			(show_name no)
@@
 			(project "HC4_KiCad"
 				(path "/33731ded-38c0-4297-bdd8-92b082f46ff8/27e10803-908c-4418-a733-f902d25b5ad6"
-					(reference "LD16")
+					(reference "LD12")
 					(unit 1)
 				)
@@
 		(dnp no)
 		(fields_autoplaced yes)
-		(property "Reference" "#PWR039"
+		(property "Reference" "#PWR036"
 			(at 167.64 129.54 0)
 			(hide yes)
@@
 			(project "HC4_KiCad"
 				(path "/33731ded-38c0-4297-bdd8-92b082f46ff8/27e10803-908c-4418-a733-f902d25b5ad6"
-					(reference "#PWR039")
+					(reference "#PWR036")
 					(unit 1)
 				)
@@
 		(in_pos_files yes)
 		(dnp no)
-		(property "Reference" "LD13"
+		(property "Reference" "LD9"
 			(at 143.51 143.8274 90)
 			(show_name no)
@@
 			(project "HC4_KiCad"
 				(path "/33731ded-38c0-4297-bdd8-92b082f46ff8/27e10803-908c-4418-a733-f902d25b5ad6"
-					(reference "LD13")
+					(reference "LD9")
 					(unit 1)
 				)
@@
 		(in_pos_files yes)
 		(dnp no)
-		(property "Reference" "IC10"
+		(property "Reference" "IC9"
 			(at 95.504 81.534 0)
 			(show_name no)
@@
 			(project "HC4_KiCad"
 				(path "/33731ded-38c0-4297-bdd8-92b082f46ff8/27e10803-908c-4418-a733-f902d25b5ad6"
-					(reference "IC10")
+					(reference "IC9")
 					(unit 1)
 				)
@@
 		(in_pos_files yes)
 		(dnp no)
-		(property "Reference" "#PWR033"
+		(property "Reference" "#PWR030"
 			(at 92.71 85.09 0)
 			(hide yes)
@@
 			(project "HC4_KiCad"
 				(path "/33731ded-38c0-4297-bdd8-92b082f46ff8/27e10803-908c-4418-a733-f902d25b5ad6"
-					(reference "#PWR033")
+					(reference "#PWR030")
 					(unit 1)
 				)
@@
 		(in_pos_files yes)
 		(dnp no)
-		(property "Reference" "LD22"
+		(property "Reference" "LD18"
 			(at 189.23 143.8274 90)
 			(show_name no)
@@
 			(project "HC4_KiCad"
 				(path "/33731ded-38c0-4297-bdd8-92b082f46ff8/27e10803-908c-4418-a733-f902d25b5ad6"
-					(reference "LD22")
+					(reference "LD18")
 					(unit 1)
 				)
@@
 		(in_pos_files yes)
 		(dnp no)
-		(property "Reference" "LD17"
+		(property "Reference" "LD13"
 			(at 163.83 143.8274 90)
 			(show_name no)
@@
 			(project "HC4_KiCad"
 				(path "/33731ded-38c0-4297-bdd8-92b082f46ff8/27e10803-908c-4418-a733-f902d25b5ad6"
-					(reference "LD17")
+					(reference "LD13")
 					(unit 1)
 				)
@@
 		(dnp no)
 		(fields_autoplaced yes)
-		(property "Reference" "#PWR034"
+		(property "Reference" "#PWR031"
 			(at 92.71 123.19 0)
 			(hide yes)
@@
 			(project "HC4_KiCad"
 				(path "/33731ded-38c0-4297-bdd8-92b082f46ff8/27e10803-908c-4418-a733-f902d25b5ad6"
-					(reference "#PWR034")
+					(reference "#PWR031")
 					(unit 1)
 				)
