File: HC4_KiCad/stackunit.kicad_sch (KiCad schematic)
At the start: 18 parts, among them IC10 74HC377, IC9 74HC161

Commit message: SPICEを復活です
Connections:
- net Level_C0: now also IC10.19 (Q7); no longer IC10.12 (Q4)
- net Level_C1: now also IC10.16 (Q6); no longer IC10.15 (Q5)
- net Level_C2: now also IC10.15 (Q5); no longer IC10.16 (Q6)
- net Level_C3: now also IC10.12 (Q4); no longer IC10.19 (Q7)
Changed lines of the file:
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@@
 	(title_block
 		(title "HC4_CPU")
-		(date "2025-04-17")
+		(date "2026-08-05")
 		(rev "2.0")
 	)
@@
 	)
 	(label "Level_C3"
-		(at 189.23 106.68 180)
+		(at 189.23 99.06 180)
 		(effects
 			(font
@@
 	)
 	(label "Level_C0"
-		(at 189.23 99.06 180)
+		(at 189.23 106.68 180)
 		(effects
 			(font
@@
 	)
 	(label "Level_C2"
-		(at 189.23 104.14 180)
+		(at 189.23 101.6 180)
 		(effects
 			(font
@@
 	)
 	(label "Level_C1"
-		(at 189.23 101.6 180)
-		(effects
-			(font
+		(at 189.23 104.14 180)
+		(effects
+			(font
