File: HC4_KiCad_EE/addressbus.kicad_sch (KiCad schematic)
At the start: 15 parts, among them IC16 74HC257, IC17 74HC257, SW2 Bus_Open

Commit message: 一部を整地
Parts:
- removed CP15, CP16: 0.1u, Capacitor_THT:C_Disc_D3.0mm_W1.6mm_P2.50mm, symbol Device2:C_Bypass
- removed IC16, IC17: 74HC257, Package_DIP:DIP-16_W7.62mm_Socket, symbol 74xx_2:74HC257
- removed LD32, LD33, LD34, LD35, LD36, LD37, LD38, LD39: LED, LED_THT:LED_Rectangular_W5.0mm_H2.0mm, symbol Device2:LED_
- removed R4: 10k, Resistor_THT:R_Axial_DIN0207_L6.3mm_D2.5mm_P7.62mm_Horizontal, symbol Device:R
- removed RN7: 1k, Resistor_THT:R_Array_SIP9, symbol Device:R_Network08_Split
- removed SW2: Bus_Open, Button_Switch_THT:SW_Slide-03_Wuerth-WS-SLTV_10x2.5x6.4_P2.54mm, symbol Switch:SW_SPDT_312
Connections:
- no-connect marks 1 -> 0
Other:
- note removed: "WRITE"
