File: HC4_KiCad_EE/alu.kicad_sch (KiCad schematic)
At the start: 8 parts, among them IC1 74HC86, IC2 74HC283, IC3 74HC253, IC4 74HC253

Commit message: たぶん完成！！！！！！！
Other:
- title: HC4_CPU -> HC4e_CPU
Changed lines of the file:
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@@
 	(paper "A4")
 	(title_block
-		(title "HC4_CPU")
-		(date "2025-06-16")
+		(title "HC4e_CPU")
+		(date "2025-07-21")
 		(rev "1.0")
 	)

Commit message: feat:HC4e改版,BOMを令和最新版に更新,KiCadを10に更新
Parts:
- IC1: footprint Package_SO:SO-14_5.3x10.2mm_P1.27mm -> (none)

Commit message: 基板を若干改版、フットプリントの指定が外れていたのを修正
Parts:
- IC1: footprint (none) -> Package_SO:SO-14_5.3x10.2mm_P1.27mm
Changed lines of the file:
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@@
 			)
 		)
-		(property "Footprint" ""
+		(property "Footprint" "Package_SO:SO-14_5.3x10.2mm_P1.27mm"
 			(at 151.13 101.6 0)
 			(hide yes)
@@
 			)
 		)
-		(property "Footprint" ""
+		(property "Footprint" "Package_SO:SO-14_5.3x10.2mm_P1.27mm"
 			(at 151.13 116.84 0)
 			(hide yes)
@@
 			)
 		)
-		(property "Footprint" ""
+		(property "Footprint" "Package_SO:SO-14_5.3x10.2mm_P1.27mm"
 			(at 151.13 148.59 0)
 			(hide yes)
@@
 			)
 		)
-		(property "Footprint" ""
+		(property "Footprint" "Package_SO:SO-14_5.3x10.2mm_P1.27mm"
 			(at 115.57 171.45 0)
 			(hide yes)
@@
 			)
 		)
-		(property "Footprint" ""
+		(property "Footprint" "Package_SO:SO-14_5.3x10.2mm_P1.27mm"
 			(at 151.13 133.35 0)
 			(hide yes)
