File: HC4_KiCad_EE/clockandreset.kicad_sch (KiCad schematic)
At the start: 18 parts, among them IC15 74HC14, SW2 SW_Push, SW3 SW_Push, SW4 FreqSel, SW5 SW_SPDT

Commit message: 自動配線前最終チェック
Connections:
- net at R4.1, SW2.2: now also RN15.3 (R3.1); no longer RN15.2 (R2.1)
- net at R5.1, SW3.2: now also RN15.2 (R2.1); no longer RN15.3 (R3.1)
Other:
- moved on the sheet: RN15B, RN15C
Changed lines of the file:
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@@
 	(symbol
 		(lib_id "Device:R_Pack04_Split")
-		(at 38.1 87.63 0)
+		(at 38.1 146.05 0)
 		(unit 2)
 		(exclude_from_sim no)
@@
 		(fields_autoplaced yes)
 		(property "Reference" "RN15"
-			(at 40.64 86.3599 0)
+			(at 40.64 144.7799 0)
 			(effects
 				(font
@@
 		)
 		(property "Value" "1k"
-			(at 40.64 88.8999 0)
+			(at 40.64 147.3199 0)
 			(effects
 				(font
@@
 		)
 		(property "Footprint" "Resistor_SMD:R_Array_Convex_4x0603"
-			(at 36.068 87.63 90)
+			(at 36.068 146.05 90)
 			(effects
 				(font
@@
 		)
 		(property "Datasheet" "~"
-			(at 38.1 87.63 0)
+			(at 38.1 146.05 0)
 			(effects
 				(font
@@
 		)
 		(property "Description" "4 resistor network, parallel topology, split"
-			(at 38.1 87.63 0)
+			(at 38.1 146.05 0)
 			(effects
 				(font
@@
 	(symbol
 		(lib_id "Device:R_Pack04_Split")
-		(at 38.1 146.05 0)
+		(at 38.1 87.63 0)
 		(unit 3)
 		(exclude_from_sim no)
@@
 		(fields_autoplaced yes)
 		(property "Reference" "RN15"
-			(at 40.64 144.7799 0)
+			(at 40.64 86.3599 0)
 			(effects
 				(font
@@
 		)
 		(property "Value" "1k"
-			(at 40.64 147.3199 0)
+			(at 40.64 88.8999 0)
 			(effects
 				(font
@@
 		)
 		(property "Footprint" "Resistor_SMD:R_Array_Convex_4x0603"
-			(at 36.068 146.05 90)
+			(at 36.068 87.63 90)
 			(effects
 				(font
@@
 		)
 		(property "Datasheet" "~"
-			(at 38.1 146.05 0)
+			(at 38.1 87.63 0)
 			(effects
 				(font
@@
 		)
 		(property "Description" "4 resistor network, parallel topology, split"
-			(at 38.1 146.05 0)
-			(effects
-				(font
+			(at 38.1 87.63 0)
+			(effects
+				(font
