File: HC4_KiCad_EE/clockandreset.kicad_sch (KiCad schematic)
At the start: 20 parts, among them IC15 74HC14, SW3 SW_Push, SW4 SW_Push, SW5 SW_SPDT, SW6 SW_SPDT

Commit message: HC4eRev2完成
Parts:
- R5: value 390k -> 330k
- R6: value 390 -> 330
Other:
- company: (none) -> Dengiken
Changed lines of the file:
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@@
 	(title_block
 		(title "HC4e_CPU")
-		(date "2026-03-19")
+		(date "2026-05-23")
 		(rev "2.0")
+		(company "Dengiken")
 	)
 	(junction
@@
 			)
 		)
-		(property "Value" "390"
+		(property "Value" "330"
 			(at 60.96 49.5299 0)
 			(show_name no)
@@
 			)
 		)
-		(property "Value" "390k"
+		(property "Value" "330k"
 			(at 50.8 49.5299 0)
 			(show_name no)
