File: HC4_KiCad_EE/HC4_KiCad_EE.kicad_pcb (KiCad board)
At the start: 2 copper layers, 100 x 100 mm, 126 parts, among them IC1 74HC86, IC10 74HC161, IC11 74HC74, IC12 74HC00, IC13 74HC4053, IC14 74HC02, IC15 74HC14, IC2 74HC283, IC3 74HC253, IC4 74HC253, IC5 74HC244, IC6 74HC377, IC7 4511, IC8 74HC377, IC9 74HC161, J1 USB_B_Mini, J2 Port_IN, J3 Port_A, J4 AVR-UPDI-6, SW1 SW_DIP_x04, SW2 SW_Push, SW3 SW_Push, SW4 FreqSel, SW5 SW_SPDT, U1 ATmega4809-A, U2 CH340E

Commit message: 自動配線前最終チェック
Parts:
- added SW6: SW_User, Button_Switch_THT:SW_PUSH_6mm, F.Cu at (123.2, 146.4)
- moved LD1 28.3 mm to (56.5, 152.4)
- moved LD46 23.9 mm to (78.5, 142.9)
- moved SW4 23.0 mm to (64.5, 125.7)
- moved RN7 15.1 mm to (94.2, 62.9)
- moved RN8 15.1 mm to (80.0, 57.8)
- moved SW3 14.1 mm to (66.8, 153.4)
- moved LD15 13.8 mm to (90.7, 58.4)
- moved LD16 13.8 mm to (88.1, 58.4)
- moved LD17 13.8 mm to (85.6, 58.4)
- moved LD18 13.8 mm to (83.1, 58.4)
- moved LD19 13.8 mm to (77.0, 58.4)
- moved LD20 13.8 mm to (74.4, 58.4)
- moved LD22 13.8 mm to (69.3, 58.4)
- moved LD21 13.8 mm to (71.9, 58.4)
- moved R8 10.9 mm to (62.2, 139.7)
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Connections:
- net /Data BUS/~{PORTA_OUT_OE} renamed /Data BUS/~{PORTA_OUT_WE}
- net /Data BUS/~{PORTB_OUT_OE} renamed /Data BUS/~{PORTB_OUT_WE}
- IC1 pad 10: /ALU/ALU_in_B2 -> /ALU/ALU_in_B3
- IC1 pad 11: /ALU/XOR3 -> /ALU/XOR2
- IC1 pad 12: /ALU/ALU_in_A3 -> /ALU/ALU_in_A2
- IC1 pad 13: /ALU/ALU_in_B3 -> /ALU/ALU_in_B2
- IC1 pad 8: /ALU/XOR2 -> /ALU/XOR3
- IC1 pad 9: /ALU/ALU_in_A2 -> /ALU/ALU_in_A3
- IC5 pad 11: /ALU/ALU_OUT3 -> /ALU/ALU_OUT0
- IC5 pad 12: /ALU/ALU_OUT3 -> /ALU/ALU_OUT0
- IC5 pad 13: /ALU/ALU_OUT2 -> /ALU/ALU_OUT1
- IC5 pad 14: /ALU/ALU_OUT2 -> /ALU/ALU_OUT1
- IC5 pad 15: /ALU/ALU_OUT1 -> /ALU/ALU_OUT2
- IC5 pad 16: /ALU/ALU_OUT1 -> /ALU/ALU_OUT2
- IC5 pad 17: /ALU/ALU_OUT0 -> /ALU/ALU_OUT3
- IC5 pad 18: /ALU/ALU_OUT0 -> /ALU/ALU_OUT3
- J2 pad 1: Net-(IC5-1A0) -> Net-(IC5-1A3)
- J2 pad 2: Net-(IC5-1A1) -> Net-(IC5-1A2)
- J2 pad 3: Net-(IC5-1A2) -> Net-(IC5-1A1)
- J2 pad 4: Net-(IC5-1A3) -> Net-(IC5-1A0)
- LD3 pad 2: Net-(IC5-2Y3) -> Net-(IC5-2Y0)
- LD4 pad 2: Net-(IC5-2Y2) -> Net-(IC5-2Y1)
- LD5 pad 2: Net-(IC5-2Y1) -> Net-(IC5-2Y2)
- LD6 pad 2: Net-(IC5-2Y0) -> Net-(IC5-2Y3)
- R4 pad 1: Net-(RN15B-R2.1) -> Net-(RN15C-R3.1)
- R5 pad 1: Net-(RN15C-R3.1) -> Net-(RN15B-R2.1)
- RN4 pad 5: Net-(LD14-K) -> Net-(LD9-K)
- RN4 pad 6: Net-(LD13-K) -> Net-(LD11-K)
- RN4 pad 7: Net-(LD11-K) -> Net-(LD13-K)
- RN4 pad 8: Net-(LD9-K) -> Net-(LD14-K)
- RN7 pad 5: Net-(LD18-K) -> Net-(LD15-K)
- RN7 pad 6: Net-(LD17-K) -> Net-(LD16-K)
- RN7 pad 7: Net-(LD16-K) -> Net-(LD17-K)
- RN7 pad 8: Net-(LD15-K) -> Net-(LD18-K)
- RN8 pad 5: Net-(LD19-K) -> Net-(LD22-K)
- RN8 pad 6: Net-(LD20-K) -> Net-(LD21-K)
- RN8 pad 7: Net-(LD21-K) -> Net-(LD20-K)
- RN8 pad 8: Net-(LD22-K) -> Net-(LD19-K)
- SW1 pad 1: Net-(IC5-1A0) -> Net-(IC5-1A3)
- SW1 pad 2: Net-(IC5-1A1) -> Net-(IC5-1A2)
- SW1 pad 3: Net-(IC5-1A2) -> Net-(IC5-1A1)
- SW1 pad 4: Net-(IC5-1A3) -> Net-(IC5-1A0)
- SW2 pad 2: Net-(RN15B-R2.1) -> Net-(RN15C-R3.1)
- SW3 pad 2: Net-(RN15C-R3.1) -> Net-(RN15B-R2.1)
Routing:
- net GND: track 473.7 -> 637.1 mm
- net VCC: track 427.8 -> 538.5 mm, vias 7 -> 11
Other:
- board text added: "↑B スタック A↑"
- board text added: "プログラムカウンタ"
- board text added: "繰り上げフラグ"

Commit message: 自動配線できた
Parts:
- moved F1 0.13 mm to (53.4, 133.4)
Routing:
- net GND: track 637.1 -> 944.0 mm, vias 2 -> 6
- net VCC: track 538.5 -> 731.2 mm, vias 11 -> 19
- net /Instruction Decoder/READ: track 0.00 -> 189.8 mm, vias 0 -> 9
- net CLK: track 0.00 -> 176.5 mm, vias 0 -> 8
- net /ALU/Instruction_1: track 0.00 -> 175.4 mm, vias 0 -> 7
- net ~{RESET}: track 0.00 -> 171.7 mm, vias 0 -> 6
- net /ALU/ALU_OUT1: track 0.00 -> 170.9 mm, vias 0 -> 12
- net /ALU/ALU_in_A0: track 0.00 -> 168.9 mm, vias 0 -> 4
- net /ALU/Instruction_0: track 0.00 -> 165.7 mm, vias 0 -> 6
- net /ALU/ALU_in_A2: track 0.00 -> 160.6 mm, vias 0 -> 6
- net /ALU/ALU_OUT3: track 0.00 -> 159.0 mm, vias 0 -> 9
- net /ALU/Instruction_2: track 0.00 -> 152.9 mm, vias 0 -> 5
- net /ALU/ALU_OUT2: track 0.00 -> 148.7 mm, vias 0 -> 8
- net /ALU/ALU_in_A1: track 0.00 -> 143.7 mm, vias 0 -> 6
- net /ALU/ALU_in_A3: track 0.00 -> 143.7 mm, vias 0 -> 9
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