File: HC4_KiCad_EE/instructiondecode.kicad_sch (KiCad schematic)
At the start: 28 parts, among them IC11 74HC02, IC12 74HC00, IC13 74HC4053, IC14 74HC74

Commit message: 基板を若干改版、フットプリントの指定が外れていたのを修正
Parts:
- CP11, CP12, CP13, CP14: LCSC PN (none) -> C14663
- IC11, IC12: footprint (none) -> Package_SO:SO-14_5.3x10.2mm_P1.27mm
- LD30, LD31, LD32, LD33, LD34, LD35, LD36, LD37, LD38, LD39, LD40, LD41, LD42, LD43, LD44, LD45: LCSC PN (none) -> C2289
- RN11, RN12, RN13, RN14: LCSC PN (none) -> C20197

Commit message: HC4eRev2完成
Connections:
- no-connect marks 3 -> 1
Other:
- company: (none) -> Dengiken
Changed lines of the file:
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@@
 	(title_block
 		(title "HC4e_CPU")
-		(date "2026-03-19")
+		(date "2026-05-23")
 		(rev "2.0")
+		(company "Dengiken")
 	)
 	(junction
@@
 		(at 123.19 168.91)
 	)
-	(no_connect
-		(at 256.54 92.71)
-	)
-	(no_connect
-		(at 259.08 92.71)
-	)
 	(bus_entry
