File: HC4_KiCad_EE/databus.kicad_sch (KiCad schematic)
At the start: 28 parts, among them IC5 74HC244, IC6 74HC377, IC7 4511, J2 Port_IN, J3 Port_A, SW1 SW_DIP_x04

Commit message: 自動配線前最終チェック
Parts:
- added SW6: SW_User, Button_Switch_THT:SW_PUSH_6mm, symbol Switch:SW_Push
Connections:
- net Databus0: now also IC5.11 (2A3), IC5.12 (1Y3); no longer IC5.17 (2A0), IC5.18 (1Y0)
- net Databus1: now also IC5.13 (2A2), IC5.14 (1Y2); no longer IC5.15 (2A1), IC5.16 (1Y1)
- net Databus2: now also IC5.15 (2A1), IC5.16 (1Y1); no longer IC5.13 (2A2), IC5.14 (1Y2)
- net Databus3: now also IC5.17 (2A0), IC5.18 (1Y0); no longer IC5.11 (2A3), IC5.12 (1Y3)
- net VCC: now also SW6.2
- net at LD5.2: now also IC5.7 (2Y2); no longer IC5.5 (2Y1)
- net at IC5.2 (1A0), RN1.5 (R4.2): now also J2.4 (Pin_4), SW1.4; no longer J2.1 (Pin_1), SW1.1
- net at IC5.4 (1A1), RN1.6 (R3.2): now also J2.3 (Pin_3), SW1.3; no longer J2.2 (Pin_2), SW1.2
- net at IC5.6 (1A2), RN1.7 (R2.2): now also J2.2 (Pin_2), SW1.2; no longer J2.3 (Pin_3), SW1.3
- net at IC5.8 (1A3), RN1.8 (R1.2): now also J2.1 (Pin_1), SW1.1, SW6.1; no longer J2.4 (Pin_4), SW1.4
- net at RN4.8 (R1.2): now also LD14.1 (K); no longer LD9.1 (K)
- net at LD13.1 (K): now also RN4.7 (R2.2); no longer RN4.6 (R3.2)
- net at LD6.2: now also IC5.9 (2Y3); no longer IC5.3 (2Y0)
- net at LD4.2: now also IC5.5 (2Y1); no longer IC5.7 (2Y2)
- net at LD3.2: now also IC5.3 (2Y0); no longer IC5.9 (2Y3)
- net at LD11.1 (K): now also RN4.6 (R3.2); no longer RN4.7 (R2.2)
- net at RN4.5 (R4.2): now also LD9.1 (K); no longer LD14.1 (K)
- net ~{PORTA_OUT_OE} renamed ~{PORTA_OUT_WE}
- net ~{PORTB_OUT_OE} renamed ~{PORTB_OUT_WE}
Other:
- moved on the sheet: RN4A, RN4B, RN4C, RN4D

Commit message: たぶん完成！！！！！！！
Parts:
- IC7: value 4511 -> 74HC4511
- J2: value Port_IN -> Port
- J3: value Port_A -> Port
- SW6: value SW_User -> SW_Push
Connections:
- net ~{PORTB_OUT_WE}: now also RN6.1 (R1.1); no longer RN6.4 (R4.1)
- net at RN6.2 (R2.1): now also IC7.9 (Qe); no longer IC7.15 (Qf)
- net at RN6.7 (R2.2): now also D1.1 (E); no longer D1.9 (F)
- net at RN6.8 (R1.2): now also D1.5 (DP); no longer D1.1 (E)
- net at D1.10 (G): now also RN6.5 (R4.2); no longer RN6.6 (R3.2)
- net at IC7.14 (Qg): now also RN6.4 (R4.1); no longer RN6.3 (R3.1)
- new net: D1.9 (F), RN6.6 (R3.2)
- new net: IC7.15 (Qf), RN6.3 (R3.1)
Other:
- title: HC4_CPU -> HC4e_CPU
- moved on the sheet: RN6A, RN6B, RN6C, RN6D
Changed lines of the file:
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@@
 	(paper "A4")
 	(title_block
-		(title "HC4_CPU")
-		(date "2025-06-16")
+		(title "HC4e_CPU")
+		(date "2025-07-21")
 		(rev "1.0")
 	)
@@
 			)
 		)
-		(property "Value" "SW_User"
+		(property "Value" "SW_Push"
 			(at 64.77 110.4899 90)
 			(effects
@@
 	(symbol
 		(lib_id "Device:R_Pack04_Split")
-		(at 248.92 87.63 270)
+		(at 248.92 85.09 270)
 		(mirror x)
 		(unit 2)
@@
 		(fields_autoplaced yes)
 		(property "Reference" "RN6"
-			(at 248.92 81.28 90)
+			(at 248.92 78.74 90)
 			(effects
 				(font
@@
 		)
 		(property "Value" "1k"
-			(at 248.92 83.82 90)
+			(at 248.92 81.28 90)
 			(effects
 				(font
@@
 		)
 		(property "Footprint" "Resistor_SMD:R_Array_Convex_4x0603"
-			(at 248.92 89.662 90)
+			(at 248.92 87.122 90)
 			(effects
 				(font
@@
 		)
 		(property "Datasheet" "~"
-			(at 248.92 87.63 0)
+			(at 248.92 85.09 0)
 			(effects
 				(font
@@
 		)
 		(property "Description" "4 resistor network, parallel topology, split"
-			(at 248.92 87.63 0)
+			(at 248.92 85.09 0)
 			(effects
 				(font
@@
 			)
 		)
-		(property "Value" "Port_IN"
+		(property "Value" "Port"
 			(at 39.37 115.824 0)
 			(effects
@@
 	(symbol
 		(lib_id "Device:R_Pack04_Split")
-		(at 248.92 92.71 270)
+		(at 248.92 90.17 270)
 		(mirror x)
 		(unit 4)
@@
 		(fields_autoplaced yes)
 		(property "Reference" "RN6"
-			(at 248.92 86.36 90)
+			(at 248.92 83.82 90)
 			(effects
 				(font
@@
 		)
 		(property "Value" "1k"
-			(at 248.92 88.9 90)
+			(at 248.92 86.36 90)
 			(effects
 				(font
@@
 		)
 		(property "Footprint" "Resistor_SMD:R_Array_Convex_4x0603"
-			(at 248.92 94.742 90)
+			(at 248.92 92.202 90)
 			(effects
 				(font
@@
 		)
 		(property "Datasheet" "~"
-			(at 248.92 92.71 0)
+			(at 248.92 90.17 0)
 			(effects
 				(font
@@
 		)
 		(property "Description" "4 resistor network, parallel topology, split"
-			(at 248.92 92.71 0)
+			(at 248.92 90.17 0)
 			(effects
 				(font
@@
 			)
 		)
-		(property "Value" "4511"
+		(property "Value" "74HC4511"
 			(at 234.5533 69.85 0)
 			(effects
@@
 	(symbol
 		(lib_id "Device:R_Pack04_Split")
-		(at 248.92 90.17 270)
+		(at 248.92 87.63 270)
 		(mirror x)
 		(unit 3)
@@
 		(fields_autoplaced yes)
 		(property "Reference" "RN6"
-			(at 248.92 83.82 90)
+			(at 248.92 81.28 90)
 			(effects
 				(font
@@
 		)
 		(property "Value" "1k"
-			(at 248.92 86.36 90)
+			(at 248.92 83.82 90)
 			(effects
 				(font
@@
 		)
 		(property "Footprint" "Resistor_SMD:R_Array_Convex_4x0603"
-			(at 248.92 92.202 90)
+			(at 248.92 89.662 90)
 			(effects
 				(font
@@
 		)
 		(property "Datasheet" "~"
-			(at 248.92 90.17 0)
+			(at 248.92 87.63 0)
 			(effects
 				(font
@@
 		)
 		(property "Description" "4 resistor network, parallel topology, split"
-			(at 248.92 90.17 0)
+			(at 248.92 87.63 0)
 			(effects
 				(font
@@
 	(symbol
 		(lib_id "Device:R_Pack04_Split")
-		(at 248.92 85.09 270)
+		(at 248.92 92.71 270)
 		(mirror x)
 		(unit 1)
@@
 		(fields_autoplaced yes)
 		(property "Reference" "RN6"
-			(at 248.92 78.74 90)
+			(at 248.92 86.36 90)
 			(effects
 				(font
@@
 		)
 		(property "Value" "1k"
-			(at 248.92 81.28 90)
+			(at 248.92 88.9 90)
 			(effects
 				(font
@@
 		)
 		(property "Footprint" "Resistor_SMD:R_Array_Convex_4x0603"
-			(at 248.92 87.122 90)
+			(at 248.92 94.742 90)
 			(effects
 				(font
@@
 		)
 		(property "Datasheet" "~"
-			(at 248.92 85.09 0)
+			(at 248.92 92.71 0)
 			(effects
 				(font
@@
 		)
 		(property "Description" "4 resistor network, parallel topology, split"
-			(at 248.92 85.09 0)
+			(at 248.92 92.71 0)
 			(effects
 				(font
@@
 			)
 		)
-		(property "Value" "Port_A"
+		(property "Value" "Port"
 			(at 176.53 80.0101 0)
 			(effects

Commit message: feat:HC4e改版,BOMを令和最新版に更新,KiCadを10に更新
Parts:
- renumbered J2 to J1, J3 to J2, LD11 to LD10, LD12 to LD11, LD13 to LD12, LD14 to LD13, LD3 to LD2, LD4 to LD3, LD5 to LD4, LD6 to LD5, LD7 to LD6, LD8 to LD7, LD9 to LD8, LD10 to LD9, SW6 to SW2

Commit message: 基板を若干改版、フットプリントの指定が外れていたのを修正
Parts:
- CP5, CP6, CP7: LCSC PN (none) -> C14663
- RN1: LCSC PN (none) -> C29718
- RN2, RN3, RN4, RN5, RN6: LCSC PN (none) -> C20197

Commit message: HC4eRev2完成
Parts:
- IC5, IC6: footprint Package_SO:TSSOP-20_4.4x6.5mm_P0.65mm -> Package_SO:SOIC-20W_7.5x12.8mm_P1.27mm
Other:
- company: (none) -> Dengiken
Changed lines of the file:
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@@
 	(title_block
 		(title "HC4e_CPU")
-		(date "2026-03-19")
+		(date "2026-05-23")
 		(rev "2.0")
+		(company "Dengiken")
 	)
 	(junction
@@
 			)
 		)
-		(property "Footprint" "Package_SO:TSSOP-20_4.4x6.5mm_P0.65mm"
+		(property "Footprint" "Package_SO:SOIC-20W_7.5x12.8mm_P1.27mm"
 			(at 156.21 90.17 0)
 			(hide yes)
@@
 			)
 		)
-		(property "Footprint" "Package_SO:TSSOP-20_4.4x6.5mm_P0.65mm"
+		(property "Footprint" "Package_SO:SOIC-20W_7.5x12.8mm_P1.27mm"
 			(at 99.06 133.35 0)
 			(hide yes)
