File: HC_MemoryBoard/HC_MemoryBoard.kicad_pcb (KiCad board)
At the start: 2 copper layers, 100 x 100 mm, 26 parts, among them IC1 HM62256BLP, IC2 74HC30, IC3 74HC138, IC4 74HC32, IC5 74HC541, J1 Expantion_Connector, J2 Conn_01x02_Pin, J3 Conn_01x08_Pin, J4 Expantion_Connector, J5 Conn_01x08_Pin, J6 Conn_01x02_Pin, J7 Conn_01x02_Pin, SW1 SW_DIP_x08

Commit message: 配線
Parts:
- added REF**: ThroughHole_d1.0_D1.7, ThroughHole:ThroughHole_d1.0_D1.7, F.Cu at (148.6, 109.9)
- added REF**: ThroughHole_d1.0_D1.7, ThroughHole:ThroughHole_d1.0_D1.7, F.Cu at (143.5, 142.9)
- added REF**: ThroughHole_d1.0_D1.7, ThroughHole:ThroughHole_d1.0_D1.7, F.Cu at (57.1, 142.9)
- added REF**: ThroughHole_d1.0_D1.7, ThroughHole:ThroughHole_d1.0_D1.7, F.Cu at (148.6, 112.4)
- added REF**10: ThroughHole_d1.0_D1.7, ThroughHole:ThroughHole_d1.0_D1.7, F.Cu at (74.9, 114.9)
- added REF**100: ThroughHole_d1.0_D1.7, ThroughHole:ThroughHole_d1.0_D1.7, F.Cu at (105.4, 120.0)
- added REF**101: ThroughHole_d1.0_D1.7, ThroughHole:ThroughHole_d1.0_D1.7, F.Cu at (108.0, 120.0)
- added REF**102: ThroughHole_d1.0_D1.7, ThroughHole:ThroughHole_d1.0_D1.7, F.Cu at (110.5, 120.0)
- added REF**103: ThroughHole_d1.0_D1.7, ThroughHole:ThroughHole_d1.0_D1.7, F.Cu at (113.0, 120.0)
- added REF**104: ThroughHole_d1.0_D1.7, ThroughHole:ThroughHole_d1.0_D1.7, F.Cu at (115.6, 120.0)
- added REF**105: ThroughHole_d1.0_D1.7, ThroughHole:ThroughHole_d1.0_D1.7, F.Cu at (118.1, 120.0)
- added REF**106: ThroughHole_d1.0_D1.7, ThroughHole:ThroughHole_d1.0_D1.7, F.Cu at (120.7, 120.0)
- added REF**107: ThroughHole_d1.0_D1.7, ThroughHole:ThroughHole_d1.0_D1.7, F.Cu at (123.2, 120.0)
- added REF**108: ThroughHole_d1.0_D1.7, ThroughHole:ThroughHole_d1.0_D1.7, F.Cu at (125.7, 120.0)
- added REF**109: ThroughHole_d1.0_D1.7, ThroughHole:ThroughHole_d1.0_D1.7, F.Cu at (128.3, 120.0)
- added REF**11: ThroughHole_d1.0_D1.7, ThroughHole:ThroughHole_d1.0_D1.7, F.Cu at (77.5, 114.9)
- added REF**110: ThroughHole_d1.0_D1.7, ThroughHole:ThroughHole_d1.0_D1.7, F.Cu at (130.8, 120.0)
- added REF**111: ThroughHole_d1.0_D1.7, ThroughHole:ThroughHole_d1.0_D1.7, F.Cu at (133.3, 120.0)
- added REF**112: ThroughHole_d1.0_D1.7, ThroughHole:ThroughHole_d1.0_D1.7, F.Cu at (135.9, 120.0)
- added REF**113: ThroughHole_d1.0_D1.7, ThroughHole:ThroughHole_d1.0_D1.7, F.Cu at (138.4, 120.0)
- added REF**114: ThroughHole_d1.0_D1.7, ThroughHole:ThroughHole_d1.0_D1.7, F.Cu at (141.0, 120.0)
- added REF**115: ThroughHole_d1.0_D1.7, ThroughHole:ThroughHole_d1.0_D1.7, F.Cu at (143.5, 120.0)
- added REF**116: ThroughHole_d1.0_D1.7, ThroughHole:ThroughHole_d1.0_D1.7, F.Cu at (146.1, 120.0)
- added REF**117: ThroughHole_d1.0_D1.7, ThroughHole:ThroughHole_d1.0_D1.7, F.Cu at (148.6, 120.0)
- added REF**118: ThroughHole_d1.0_D1.7, ThroughHole:ThroughHole_d1.0_D1.7, F.Cu at (52.1, 122.6)
- added REF**119: ThroughHole_d1.0_D1.7, ThroughHole:ThroughHole_d1.0_D1.7, F.Cu at (54.6, 122.6)
- added REF**12: ThroughHole_d1.0_D1.7, ThroughHole:ThroughHole_d1.0_D1.7, F.Cu at (80.0, 114.9)
- added REF**120: ThroughHole_d1.0_D1.7, ThroughHole:ThroughHole_d1.0_D1.7, F.Cu at (57.1, 122.6)
- added REF**121: ThroughHole_d1.0_D1.7, ThroughHole:ThroughHole_d1.0_D1.7, F.Cu at (59.7, 122.6)
- added REF**122: ThroughHole_d1.0_D1.7, ThroughHole:ThroughHole_d1.0_D1.7, F.Cu at (62.2, 122.6)
- added REF**123: ThroughHole_d1.0_D1.7, ThroughHole:ThroughHole_d1.0_D1.7, F.Cu at (64.8, 122.6)
- added REF**124: ThroughHole_d1.0_D1.7, ThroughHole:ThroughHole_d1.0_D1.7, F.Cu at (67.3, 122.6)
- added REF**125: ThroughHole_d1.0_D1.7, ThroughHole:ThroughHole_d1.0_D1.7, F.Cu at (69.8, 122.6)
- added REF**126: ThroughHole_d1.0_D1.7, ThroughHole:ThroughHole_d1.0_D1.7, F.Cu at (72.4, 122.6)
- added REF**127: ThroughHole_d1.0_D1.7, ThroughHole:ThroughHole_d1.0_D1.7, F.Cu at (74.9, 122.6)
- added REF**128: ThroughHole_d1.0_D1.7, ThroughHole:ThroughHole_d1.0_D1.7, F.Cu at (77.5, 122.6)
- added REF**129: ThroughHole_d1.0_D1.7, ThroughHole:ThroughHole_d1.0_D1.7, F.Cu at (80.0, 122.6)
- added REF**13: ThroughHole_d1.0_D1.7, ThroughHole:ThroughHole_d1.0_D1.7, F.Cu at (80.0, 109.9)
- added REF**13: ThroughHole_d1.0_D1.7, ThroughHole:ThroughHole_d1.0_D1.7, F.Cu at (80.0, 112.4)
- added REF**13: ThroughHole_d1.0_D1.7, ThroughHole:ThroughHole_d1.0_D1.7, F.Cu at (82.5, 114.9)
- added REF**130: ThroughHole_d1.0_D1.7, ThroughHole:ThroughHole_d1.0_D1.7, F.Cu at (82.5, 122.6)
- added REF**131: ThroughHole_d1.0_D1.7, ThroughHole:ThroughHole_d1.0_D1.7, F.Cu at (85.1, 122.6)
- added REF**132: ThroughHole_d1.0_D1.7, ThroughHole:ThroughHole_d1.0_D1.7, F.Cu at (87.6, 122.6)
- added REF**133: ThroughHole_d1.0_D1.7, ThroughHole:ThroughHole_d1.0_D1.7, F.Cu at (90.2, 122.6)
- added REF**134: ThroughHole_d1.0_D1.7, ThroughHole:ThroughHole_d1.0_D1.7, F.Cu at (92.7, 122.6)
- added REF**135: ThroughHole_d1.0_D1.7, ThroughHole:ThroughHole_d1.0_D1.7, F.Cu at (95.2, 122.6)
- added REF**136: ThroughHole_d1.0_D1.7, ThroughHole:ThroughHole_d1.0_D1.7, F.Cu at (97.8, 122.6)
- added REF**137: ThroughHole_d1.0_D1.7, ThroughHole:ThroughHole_d1.0_D1.7, F.Cu at (100.3, 122.6)
- added REF**138: ThroughHole_d1.0_D1.7, ThroughHole:ThroughHole_d1.0_D1.7, F.Cu at (102.9, 122.6)
- added REF**139: ThroughHole_d1.0_D1.7, ThroughHole:ThroughHole_d1.0_D1.7, F.Cu at (105.4, 122.6)
- added REF**14: ThroughHole_d1.0_D1.7, ThroughHole:ThroughHole_d1.0_D1.7, F.Cu at (85.1, 114.9)
- added REF**14: ThroughHole_d1.0_D1.7, ThroughHole:ThroughHole_d1.0_D1.7, F.Cu at (82.5, 112.4)
- added REF**14: ThroughHole_d1.0_D1.7, ThroughHole:ThroughHole_d1.0_D1.7, F.Cu at (82.5, 109.9)
- added REF**140: ThroughHole_d1.0_D1.7, ThroughHole:ThroughHole_d1.0_D1.7, F.Cu at (108.0, 122.6)
- added REF**141: ThroughHole_d1.0_D1.7, ThroughHole:ThroughHole_d1.0_D1.7, F.Cu at (110.5, 122.6)
- added REF**142: ThroughHole_d1.0_D1.7, ThroughHole:ThroughHole_d1.0_D1.7, F.Cu at (113.0, 122.6)
- added REF**143: ThroughHole_d1.0_D1.7, ThroughHole:ThroughHole_d1.0_D1.7, F.Cu at (115.6, 122.6)
- added REF**144: ThroughHole_d1.0_D1.7, ThroughHole:ThroughHole_d1.0_D1.7, F.Cu at (118.1, 122.6)
- added REF**145: ThroughHole_d1.0_D1.7, ThroughHole:ThroughHole_d1.0_D1.7, F.Cu at (120.7, 122.6)
- added REF**146: ThroughHole_d1.0_D1.7, ThroughHole:ThroughHole_d1.0_D1.7, F.Cu at (123.2, 122.6)
- added REF**147: ThroughHole_d1.0_D1.7, ThroughHole:ThroughHole_d1.0_D1.7, F.Cu at (125.7, 122.6)
- added REF**148: ThroughHole_d1.0_D1.7, ThroughHole:ThroughHole_d1.0_D1.7, F.Cu at (128.3, 122.6)
- added REF**149: ThroughHole_d1.0_D1.7, ThroughHole:ThroughHole_d1.0_D1.7, F.Cu at (130.8, 122.6)
- added REF**15: ThroughHole_d1.0_D1.7, ThroughHole:ThroughHole_d1.0_D1.7, F.Cu at (87.6, 114.9)
- added REF**15: ThroughHole_d1.0_D1.7, ThroughHole:ThroughHole_d1.0_D1.7, F.Cu at (85.1, 112.4)
- added REF**15: ThroughHole_d1.0_D1.7, ThroughHole:ThroughHole_d1.0_D1.7, F.Cu at (85.1, 109.9)
- added REF**150: ThroughHole_d1.0_D1.7, ThroughHole:ThroughHole_d1.0_D1.7, F.Cu at (133.3, 122.6)
- added REF**151: ThroughHole_d1.0_D1.7, ThroughHole:ThroughHole_d1.0_D1.7, F.Cu at (135.9, 122.6)
- added REF**152: ThroughHole_d1.0_D1.7, ThroughHole:ThroughHole_d1.0_D1.7, F.Cu at (138.4, 122.6)
- added REF**153: ThroughHole_d1.0_D1.7, ThroughHole:ThroughHole_d1.0_D1.7, F.Cu at (141.0, 122.6)
- added REF**154: ThroughHole_d1.0_D1.7, ThroughHole:ThroughHole_d1.0_D1.7, F.Cu at (143.5, 122.6)
- added REF**155: ThroughHole_d1.0_D1.7, ThroughHole:ThroughHole_d1.0_D1.7, F.Cu at (146.1, 122.6)
- added REF**156: ThroughHole_d1.0_D1.7, ThroughHole:ThroughHole_d1.0_D1.7, F.Cu at (148.6, 122.6)
- added REF**157: ThroughHole_d1.0_D1.7, ThroughHole:ThroughHole_d1.0_D1.7, F.Cu at (52.1, 125.1)
- added REF**158: ThroughHole_d1.0_D1.7, ThroughHole:ThroughHole_d1.0_D1.7, F.Cu at (54.6, 125.1)
- added REF**159: ThroughHole_d1.0_D1.7, ThroughHole:ThroughHole_d1.0_D1.7, F.Cu at (57.1, 125.1)
- added REF**16: ThroughHole_d1.0_D1.7, ThroughHole:ThroughHole_d1.0_D1.7, F.Cu at (87.6, 112.4)
- added REF**16: ThroughHole_d1.0_D1.7, ThroughHole:ThroughHole_d1.0_D1.7, F.Cu at (87.6, 109.9)
- added REF**16: ThroughHole_d1.0_D1.7, ThroughHole:ThroughHole_d1.0_D1.7, F.Cu at (90.2, 114.9)
- added REF**160: ThroughHole_d1.0_D1.7, ThroughHole:ThroughHole_d1.0_D1.7, F.Cu at (59.7, 125.1)
- added REF**161: ThroughHole_d1.0_D1.7, ThroughHole:ThroughHole_d1.0_D1.7, F.Cu at (62.2, 125.1)
- added REF**162: ThroughHole_d1.0_D1.7, ThroughHole:ThroughHole_d1.0_D1.7, F.Cu at (64.8, 125.1)
- added REF**163: ThroughHole_d1.0_D1.7, ThroughHole:ThroughHole_d1.0_D1.7, F.Cu at (67.3, 125.1)
- added REF**164: ThroughHole_d1.0_D1.7, ThroughHole:ThroughHole_d1.0_D1.7, F.Cu at (69.8, 125.1)
- added REF**165: ThroughHole_d1.0_D1.7, ThroughHole:ThroughHole_d1.0_D1.7, F.Cu at (72.4, 125.1)
- added REF**166: ThroughHole_d1.0_D1.7, ThroughHole:ThroughHole_d1.0_D1.7, F.Cu at (74.9, 125.1)
- added REF**167: ThroughHole_d1.0_D1.7, ThroughHole:ThroughHole_d1.0_D1.7, F.Cu at (77.5, 125.1)
- added REF**168: ThroughHole_d1.0_D1.7, ThroughHole:ThroughHole_d1.0_D1.7, F.Cu at (80.0, 125.1)
- added REF**169: ThroughHole_d1.0_D1.7, ThroughHole:ThroughHole_d1.0_D1.7, F.Cu at (82.5, 125.1)
- added REF**17: ThroughHole_d1.0_D1.7, ThroughHole:ThroughHole_d1.0_D1.7, F.Cu at (92.7, 114.9)
- added REF**17: ThroughHole_d1.0_D1.7, ThroughHole:ThroughHole_d1.0_D1.7, F.Cu at (90.2, 112.4)
- added REF**17: ThroughHole_d1.0_D1.7, ThroughHole:ThroughHole_d1.0_D1.7, F.Cu at (90.2, 109.9)
- added REF**170: ThroughHole_d1.0_D1.7, ThroughHole:ThroughHole_d1.0_D1.7, F.Cu at (85.1, 125.1)
- added REF**171: ThroughHole_d1.0_D1.7, ThroughHole:ThroughHole_d1.0_D1.7, F.Cu at (87.6, 125.1)
- added REF**172: ThroughHole_d1.0_D1.7, ThroughHole:ThroughHole_d1.0_D1.7, F.Cu at (90.2, 125.1)
- added REF**173: ThroughHole_d1.0_D1.7, ThroughHole:ThroughHole_d1.0_D1.7, F.Cu at (92.7, 125.1)
- added REF**174: ThroughHole_d1.0_D1.7, ThroughHole:ThroughHole_d1.0_D1.7, F.Cu at (95.2, 125.1)
- added REF**175: ThroughHole_d1.0_D1.7, ThroughHole:ThroughHole_d1.0_D1.7, F.Cu at (97.8, 125.1)
- added REF**176: ThroughHole_d1.0_D1.7, ThroughHole:ThroughHole_d1.0_D1.7, F.Cu at (100.3, 125.1)
- added REF**177: ThroughHole_d1.0_D1.7, ThroughHole:ThroughHole_d1.0_D1.7, F.Cu at (102.9, 125.1)
- added REF**178: ThroughHole_d1.0_D1.7, ThroughHole:ThroughHole_d1.0_D1.7, F.Cu at (105.4, 125.1)
- added REF**179: ThroughHole_d1.0_D1.7, ThroughHole:ThroughHole_d1.0_D1.7, F.Cu at (108.0, 125.1)
- added REF**18: ThroughHole_d1.0_D1.7, ThroughHole:ThroughHole_d1.0_D1.7, F.Cu at (92.7, 112.4)
- added REF**18: ThroughHole_d1.0_D1.7, ThroughHole:ThroughHole_d1.0_D1.7, F.Cu at (95.2, 114.9)
- added REF**18: ThroughHole_d1.0_D1.7, ThroughHole:ThroughHole_d1.0_D1.7, F.Cu at (92.7, 109.9)
- added REF**180: ThroughHole_d1.0_D1.7, ThroughHole:ThroughHole_d1.0_D1.7, F.Cu at (110.5, 125.1)
- added REF**181: ThroughHole_d1.0_D1.7, ThroughHole:ThroughHole_d1.0_D1.7, F.Cu at (113.0, 125.1)
- added REF**182: ThroughHole_d1.0_D1.7, ThroughHole:ThroughHole_d1.0_D1.7, F.Cu at (115.6, 125.1)
- added REF**183: ThroughHole_d1.0_D1.7, ThroughHole:ThroughHole_d1.0_D1.7, F.Cu at (118.1, 125.1)
- added REF**184: ThroughHole_d1.0_D1.7, ThroughHole:ThroughHole_d1.0_D1.7, F.Cu at (120.7, 125.1)
- added REF**185: ThroughHole_d1.0_D1.7, ThroughHole:ThroughHole_d1.0_D1.7, F.Cu at (123.2, 125.1)
- added REF**186: ThroughHole_d1.0_D1.7, ThroughHole:ThroughHole_d1.0_D1.7, F.Cu at (125.7, 125.1)
- added REF**187: ThroughHole_d1.0_D1.7, ThroughHole:ThroughHole_d1.0_D1.7, F.Cu at (128.3, 125.1)
- added REF**188: ThroughHole_d1.0_D1.7, ThroughHole:ThroughHole_d1.0_D1.7, F.Cu at (130.8, 125.1)
- added REF**189: ThroughHole_d1.0_D1.7, ThroughHole:ThroughHole_d1.0_D1.7, F.Cu at (133.3, 125.1)
- added REF**19: ThroughHole_d1.0_D1.7, ThroughHole:ThroughHole_d1.0_D1.7, F.Cu at (95.2, 109.9)
- added REF**19: ThroughHole_d1.0_D1.7, ThroughHole:ThroughHole_d1.0_D1.7, F.Cu at (95.2, 112.4)
- added REF**19: ThroughHole_d1.0_D1.7, ThroughHole:ThroughHole_d1.0_D1.7, F.Cu at (97.8, 114.9)
- added REF**190: ThroughHole_d1.0_D1.7, ThroughHole:ThroughHole_d1.0_D1.7, F.Cu at (135.9, 125.1)
- added REF**191: ThroughHole_d1.0_D1.7, ThroughHole:ThroughHole_d1.0_D1.7, F.Cu at (138.4, 125.1)
- added REF**192: ThroughHole_d1.0_D1.7, ThroughHole:ThroughHole_d1.0_D1.7, F.Cu at (141.0, 125.1)
- added REF**193: ThroughHole_d1.0_D1.7, ThroughHole:ThroughHole_d1.0_D1.7, F.Cu at (143.5, 125.1)
- added REF**194: ThroughHole_d1.0_D1.7, ThroughHole:ThroughHole_d1.0_D1.7, F.Cu at (146.1, 125.1)
- added REF**195: ThroughHole_d1.0_D1.7, ThroughHole:ThroughHole_d1.0_D1.7, F.Cu at (148.6, 125.1)
- added REF**196: ThroughHole_d1.0_D1.7, ThroughHole:ThroughHole_d1.0_D1.7, F.Cu at (52.1, 127.6)
- added REF**197: ThroughHole_d1.0_D1.7, ThroughHole:ThroughHole_d1.0_D1.7, F.Cu at (54.6, 127.6)
- added REF**198: ThroughHole_d1.0_D1.7, ThroughHole:ThroughHole_d1.0_D1.7, F.Cu at (57.1, 127.6)
- added REF**199: ThroughHole_d1.0_D1.7, ThroughHole:ThroughHole_d1.0_D1.7, F.Cu at (59.7, 127.6)
- added REF**20: ThroughHole_d1.0_D1.7, ThroughHole:ThroughHole_d1.0_D1.7, F.Cu at (97.8, 112.4)
- added REF**20: ThroughHole_d1.0_D1.7, ThroughHole:ThroughHole_d1.0_D1.7, F.Cu at (97.8, 109.9)
- added REF**20: ThroughHole_d1.0_D1.7, ThroughHole:ThroughHole_d1.0_D1.7, F.Cu at (100.3, 114.9)
- added REF**200: ThroughHole_d1.0_D1.7, ThroughHole:ThroughHole_d1.0_D1.7, F.Cu at (62.2, 127.6)
- added REF**201: ThroughHole_d1.0_D1.7, ThroughHole:ThroughHole_d1.0_D1.7, F.Cu at (64.8, 127.6)
- added REF**202: ThroughHole_d1.0_D1.7, ThroughHole:ThroughHole_d1.0_D1.7, F.Cu at (67.3, 127.6)
- added REF**203: ThroughHole_d1.0_D1.7, ThroughHole:ThroughHole_d1.0_D1.7, F.Cu at (69.8, 127.6)
- added REF**204: ThroughHole_d1.0_D1.7, ThroughHole:ThroughHole_d1.0_D1.7, F.Cu at (72.4, 127.6)
- added REF**205: ThroughHole_d1.0_D1.7, ThroughHole:ThroughHole_d1.0_D1.7, F.Cu at (74.9, 127.6)
- added REF**206: ThroughHole_d1.0_D1.7, ThroughHole:ThroughHole_d1.0_D1.7, F.Cu at (77.5, 127.6)
- added REF**207: ThroughHole_d1.0_D1.7, ThroughHole:ThroughHole_d1.0_D1.7, F.Cu at (80.0, 127.6)
- added REF**208: ThroughHole_d1.0_D1.7, ThroughHole:ThroughHole_d1.0_D1.7, F.Cu at (82.5, 127.6)
- added REF**209: ThroughHole_d1.0_D1.7, ThroughHole:ThroughHole_d1.0_D1.7, F.Cu at (85.1, 127.6)
- added REF**21: ThroughHole_d1.0_D1.7, ThroughHole:ThroughHole_d1.0_D1.7, F.Cu at (100.3, 109.9)
- added REF**21: ThroughHole_d1.0_D1.7, ThroughHole:ThroughHole_d1.0_D1.7, F.Cu at (102.9, 114.9)
- added REF**21: ThroughHole_d1.0_D1.7, ThroughHole:ThroughHole_d1.0_D1.7, F.Cu at (100.3, 112.4)
- added REF**210: ThroughHole_d1.0_D1.7, ThroughHole:ThroughHole_d1.0_D1.7, F.Cu at (87.6, 127.6)
- added REF**211: ThroughHole_d1.0_D1.7, ThroughHole:ThroughHole_d1.0_D1.7, F.Cu at (90.2, 127.6)
- added REF**212: ThroughHole_d1.0_D1.7, ThroughHole:ThroughHole_d1.0_D1.7, F.Cu at (92.7, 127.6)
- added REF**213: ThroughHole_d1.0_D1.7, ThroughHole:ThroughHole_d1.0_D1.7, F.Cu at (95.2, 127.6)
- added REF**214: ThroughHole_d1.0_D1.7, ThroughHole:ThroughHole_d1.0_D1.7, F.Cu at (97.8, 127.6)
- added REF**215: ThroughHole_d1.0_D1.7, ThroughHole:ThroughHole_d1.0_D1.7, F.Cu at (100.3, 127.6)
- added REF**216: ThroughHole_d1.0_D1.7, ThroughHole:ThroughHole_d1.0_D1.7, F.Cu at (102.9, 127.6)
- added REF**217: ThroughHole_d1.0_D1.7, ThroughHole:ThroughHole_d1.0_D1.7, F.Cu at (105.4, 127.6)
- added REF**218: ThroughHole_d1.0_D1.7, ThroughHole:ThroughHole_d1.0_D1.7, F.Cu at (108.0, 127.6)
- added REF**219: ThroughHole_d1.0_D1.7, ThroughHole:ThroughHole_d1.0_D1.7, F.Cu at (110.5, 127.6)
- added REF**22: ThroughHole_d1.0_D1.7, ThroughHole:ThroughHole_d1.0_D1.7, F.Cu at (102.9, 112.4)
- added REF**22: ThroughHole_d1.0_D1.7, ThroughHole:ThroughHole_d1.0_D1.7, F.Cu at (102.9, 109.9)
- added REF**22: ThroughHole_d1.0_D1.7, ThroughHole:ThroughHole_d1.0_D1.7, F.Cu at (105.4, 114.9)
- added REF**220: ThroughHole_d1.0_D1.7, ThroughHole:ThroughHole_d1.0_D1.7, F.Cu at (113.0, 127.6)
- added REF**221: ThroughHole_d1.0_D1.7, ThroughHole:ThroughHole_d1.0_D1.7, F.Cu at (115.6, 127.6)
- added REF**222: ThroughHole_d1.0_D1.7, ThroughHole:ThroughHole_d1.0_D1.7, F.Cu at (118.1, 127.6)
- added REF**223: ThroughHole_d1.0_D1.7, ThroughHole:ThroughHole_d1.0_D1.7, F.Cu at (120.7, 127.6)
- added REF**224: ThroughHole_d1.0_D1.7, ThroughHole:ThroughHole_d1.0_D1.7, F.Cu at (123.2, 127.6)
- added REF**225: ThroughHole_d1.0_D1.7, ThroughHole:ThroughHole_d1.0_D1.7, F.Cu at (125.7, 127.6)
- added REF**226: ThroughHole_d1.0_D1.7, ThroughHole:ThroughHole_d1.0_D1.7, F.Cu at (128.3, 127.6)
- added REF**227: ThroughHole_d1.0_D1.7, ThroughHole:ThroughHole_d1.0_D1.7, F.Cu at (130.8, 127.6)
- added REF**228: ThroughHole_d1.0_D1.7, ThroughHole:ThroughHole_d1.0_D1.7, F.Cu at (133.3, 127.6)
- added REF**229: ThroughHole_d1.0_D1.7, ThroughHole:ThroughHole_d1.0_D1.7, F.Cu at (135.9, 127.6)
- added REF**23: ThroughHole_d1.0_D1.7, ThroughHole:ThroughHole_d1.0_D1.7, F.Cu at (108.0, 114.9)
- added REF**23: ThroughHole_d1.0_D1.7, ThroughHole:ThroughHole_d1.0_D1.7, F.Cu at (105.4, 112.4)
- added REF**23: ThroughHole_d1.0_D1.7, ThroughHole:ThroughHole_d1.0_D1.7, F.Cu at (105.4, 109.9)
- added REF**230: ThroughHole_d1.0_D1.7, ThroughHole:ThroughHole_d1.0_D1.7, F.Cu at (138.4, 127.6)
- added REF**231: ThroughHole_d1.0_D1.7, ThroughHole:ThroughHole_d1.0_D1.7, F.Cu at (141.0, 127.6)
- added REF**232: ThroughHole_d1.0_D1.7, ThroughHole:ThroughHole_d1.0_D1.7, F.Cu at (143.5, 127.6)
- added REF**233: ThroughHole_d1.0_D1.7, ThroughHole:ThroughHole_d1.0_D1.7, F.Cu at (146.1, 127.6)
- added REF**234: ThroughHole_d1.0_D1.7, ThroughHole:ThroughHole_d1.0_D1.7, F.Cu at (148.6, 127.6)
- added REF**235: ThroughHole_d1.0_D1.7, ThroughHole:ThroughHole_d1.0_D1.7, F.Cu at (52.1, 130.2)
- added REF**236: ThroughHole_d1.0_D1.7, ThroughHole:ThroughHole_d1.0_D1.7, F.Cu at (54.6, 130.2)
- added REF**237: ThroughHole_d1.0_D1.7, ThroughHole:ThroughHole_d1.0_D1.7, F.Cu at (57.1, 130.2)
- added REF**238: ThroughHole_d1.0_D1.7, ThroughHole:ThroughHole_d1.0_D1.7, F.Cu at (59.7, 130.2)
- added REF**239: ThroughHole_d1.0_D1.7, ThroughHole:ThroughHole_d1.0_D1.7, F.Cu at (62.2, 130.2)
- added REF**24: ThroughHole_d1.0_D1.7, ThroughHole:ThroughHole_d1.0_D1.7, F.Cu at (108.0, 109.9)
- added REF**24: ThroughHole_d1.0_D1.7, ThroughHole:ThroughHole_d1.0_D1.7, F.Cu at (110.5, 114.9)
- added REF**24: ThroughHole_d1.0_D1.7, ThroughHole:ThroughHole_d1.0_D1.7, F.Cu at (108.0, 112.4)
- added REF**240: ThroughHole_d1.0_D1.7, ThroughHole:ThroughHole_d1.0_D1.7, F.Cu at (64.8, 130.2)
- added REF**241: ThroughHole_d1.0_D1.7, ThroughHole:ThroughHole_d1.0_D1.7, F.Cu at (67.3, 130.2)
- added REF**242: ThroughHole_d1.0_D1.7, ThroughHole:ThroughHole_d1.0_D1.7, F.Cu at (69.8, 130.2)
- added REF**243: ThroughHole_d1.0_D1.7, ThroughHole:ThroughHole_d1.0_D1.7, F.Cu at (72.4, 130.2)
- added REF**244: ThroughHole_d1.0_D1.7, ThroughHole:ThroughHole_d1.0_D1.7, F.Cu at (74.9, 130.2)
- added REF**245: ThroughHole_d1.0_D1.7, ThroughHole:ThroughHole_d1.0_D1.7, F.Cu at (77.5, 130.2)
- added REF**246: ThroughHole_d1.0_D1.7, ThroughHole:ThroughHole_d1.0_D1.7, F.Cu at (80.0, 130.2)
- added REF**247: ThroughHole_d1.0_D1.7, ThroughHole:ThroughHole_d1.0_D1.7, F.Cu at (82.5, 130.2)
- added REF**248: ThroughHole_d1.0_D1.7, ThroughHole:ThroughHole_d1.0_D1.7, F.Cu at (85.1, 130.2)
- added REF**249: ThroughHole_d1.0_D1.7, ThroughHole:ThroughHole_d1.0_D1.7, F.Cu at (87.6, 130.2)
- added REF**25: ThroughHole_d1.0_D1.7, ThroughHole:ThroughHole_d1.0_D1.7, F.Cu at (110.5, 109.9)
- added REF**25: ThroughHole_d1.0_D1.7, ThroughHole:ThroughHole_d1.0_D1.7, F.Cu at (110.5, 112.4)
- added REF**25: ThroughHole_d1.0_D1.7, ThroughHole:ThroughHole_d1.0_D1.7, F.Cu at (113.0, 114.9)
- added REF**250: ThroughHole_d1.0_D1.7, ThroughHole:ThroughHole_d1.0_D1.7, F.Cu at (90.2, 130.2)
- added REF**251: ThroughHole_d1.0_D1.7, ThroughHole:ThroughHole_d1.0_D1.7, F.Cu at (92.7, 130.2)
- added REF**252: ThroughHole_d1.0_D1.7, ThroughHole:ThroughHole_d1.0_D1.7, F.Cu at (95.2, 130.2)
- added REF**253: ThroughHole_d1.0_D1.7, ThroughHole:ThroughHole_d1.0_D1.7, F.Cu at (97.8, 130.2)
- added REF**254: ThroughHole_d1.0_D1.7, ThroughHole:ThroughHole_d1.0_D1.7, F.Cu at (100.3, 130.2)
- added REF**255: ThroughHole_d1.0_D1.7, ThroughHole:ThroughHole_d1.0_D1.7, F.Cu at (102.9, 130.2)
- added REF**256: ThroughHole_d1.0_D1.7, ThroughHole:ThroughHole_d1.0_D1.7, F.Cu at (105.4, 130.2)
- added REF**257: ThroughHole_d1.0_D1.7, ThroughHole:ThroughHole_d1.0_D1.7, F.Cu at (108.0, 130.2)
- added REF**258: ThroughHole_d1.0_D1.7, ThroughHole:ThroughHole_d1.0_D1.7, F.Cu at (110.5, 130.2)
- added REF**259: ThroughHole_d1.0_D1.7, ThroughHole:ThroughHole_d1.0_D1.7, F.Cu at (113.0, 130.2)
- added REF**26: ThroughHole_d1.0_D1.7, ThroughHole:ThroughHole_d1.0_D1.7, F.Cu at (113.0, 112.4)
- added REF**26: ThroughHole_d1.0_D1.7, ThroughHole:ThroughHole_d1.0_D1.7, F.Cu at (113.0, 109.9)
- added REF**26: ThroughHole_d1.0_D1.7, ThroughHole:ThroughHole_d1.0_D1.7, F.Cu at (115.6, 114.9)
- added REF**260: ThroughHole_d1.0_D1.7, ThroughHole:ThroughHole_d1.0_D1.7, F.Cu at (115.6, 130.2)
- added REF**261: ThroughHole_d1.0_D1.7, ThroughHole:ThroughHole_d1.0_D1.7, F.Cu at (118.1, 130.2)
- added REF**262: ThroughHole_d1.0_D1.7, ThroughHole:ThroughHole_d1.0_D1.7, F.Cu at (120.7, 130.2)
- added REF**263: ThroughHole_d1.0_D1.7, ThroughHole:ThroughHole_d1.0_D1.7, F.Cu at (123.2, 130.2)
- added REF**264: ThroughHole_d1.0_D1.7, ThroughHole:ThroughHole_d1.0_D1.7, F.Cu at (125.7, 130.2)
- added REF**265: ThroughHole_d1.0_D1.7, ThroughHole:ThroughHole_d1.0_D1.7, F.Cu at (128.3, 130.2)
- added REF**266: ThroughHole_d1.0_D1.7, ThroughHole:ThroughHole_d1.0_D1.7, F.Cu at (130.8, 130.2)
- added REF**267: ThroughHole_d1.0_D1.7, ThroughHole:ThroughHole_d1.0_D1.7, F.Cu at (133.3, 130.2)
- added REF**268: ThroughHole_d1.0_D1.7, ThroughHole:ThroughHole_d1.0_D1.7, F.Cu at (135.9, 130.2)
- added REF**269: ThroughHole_d1.0_D1.7, ThroughHole:ThroughHole_d1.0_D1.7, F.Cu at (138.4, 130.2)
- added REF**27: ThroughHole_d1.0_D1.7, ThroughHole:ThroughHole_d1.0_D1.7, F.Cu at (115.6, 109.9)
- added REF**27: ThroughHole_d1.0_D1.7, ThroughHole:ThroughHole_d1.0_D1.7, F.Cu at (115.6, 112.4)
- added REF**27: ThroughHole_d1.0_D1.7, ThroughHole:ThroughHole_d1.0_D1.7, F.Cu at (118.1, 114.9)
- added REF**270: ThroughHole_d1.0_D1.7, ThroughHole:ThroughHole_d1.0_D1.7, F.Cu at (141.0, 130.2)
- added REF**271: ThroughHole_d1.0_D1.7, ThroughHole:ThroughHole_d1.0_D1.7, F.Cu at (143.5, 130.2)
- added REF**272: ThroughHole_d1.0_D1.7, ThroughHole:ThroughHole_d1.0_D1.7, F.Cu at (146.1, 130.2)
- added REF**273: ThroughHole_d1.0_D1.7, ThroughHole:ThroughHole_d1.0_D1.7, F.Cu at (148.6, 130.2)
- added REF**274: ThroughHole_d1.0_D1.7, ThroughHole:ThroughHole_d1.0_D1.7, F.Cu at (52.1, 132.7)
- added REF**275: ThroughHole_d1.0_D1.7, ThroughHole:ThroughHole_d1.0_D1.7, F.Cu at (54.6, 132.7)
- added REF**276: ThroughHole_d1.0_D1.7, ThroughHole:ThroughHole_d1.0_D1.7, F.Cu at (57.1, 132.7)
- added REF**277: ThroughHole_d1.0_D1.7, ThroughHole:ThroughHole_d1.0_D1.7, F.Cu at (59.7, 132.7)
- added REF**278: ThroughHole_d1.0_D1.7, ThroughHole:ThroughHole_d1.0_D1.7, F.Cu at (62.2, 132.7)
- added REF**279: ThroughHole_d1.0_D1.7, ThroughHole:ThroughHole_d1.0_D1.7, F.Cu at (64.8, 132.7)
- added REF**28: ThroughHole_d1.0_D1.7, ThroughHole:ThroughHole_d1.0_D1.7, F.Cu at (118.1, 112.4)
- added REF**28: ThroughHole_d1.0_D1.7, ThroughHole:ThroughHole_d1.0_D1.7, F.Cu at (118.1, 109.9)
- added REF**28: ThroughHole_d1.0_D1.7, ThroughHole:ThroughHole_d1.0_D1.7, F.Cu at (120.7, 114.9)
- added REF**280: ThroughHole_d1.0_D1.7, ThroughHole:ThroughHole_d1.0_D1.7, F.Cu at (67.3, 132.7)
- added REF**281: ThroughHole_d1.0_D1.7, ThroughHole:ThroughHole_d1.0_D1.7, F.Cu at (69.8, 132.7)
- added REF**282: ThroughHole_d1.0_D1.7, ThroughHole:ThroughHole_d1.0_D1.7, F.Cu at (72.4, 132.7)
- added REF**283: ThroughHole_d1.0_D1.7, ThroughHole:ThroughHole_d1.0_D1.7, F.Cu at (74.9, 132.7)
- added REF**284: ThroughHole_d1.0_D1.7, ThroughHole:ThroughHole_d1.0_D1.7, F.Cu at (77.5, 132.7)
- added REF**285: ThroughHole_d1.0_D1.7, ThroughHole:ThroughHole_d1.0_D1.7, F.Cu at (80.0, 132.7)
- added REF**286: ThroughHole_d1.0_D1.7, ThroughHole:ThroughHole_d1.0_D1.7, F.Cu at (82.5, 132.7)
- added REF**287: ThroughHole_d1.0_D1.7, ThroughHole:ThroughHole_d1.0_D1.7, F.Cu at (85.1, 132.7)
- added REF**288: ThroughHole_d1.0_D1.7, ThroughHole:ThroughHole_d1.0_D1.7, F.Cu at (87.6, 132.7)
- added REF**289: ThroughHole_d1.0_D1.7, ThroughHole:ThroughHole_d1.0_D1.7, F.Cu at (90.2, 132.7)
- added REF**29: ThroughHole_d1.0_D1.7, ThroughHole:ThroughHole_d1.0_D1.7, F.Cu at (123.2, 114.9)
- added REF**29: ThroughHole_d1.0_D1.7, ThroughHole:ThroughHole_d1.0_D1.7, F.Cu at (120.7, 109.9)
- added REF**29: ThroughHole_d1.0_D1.7, ThroughHole:ThroughHole_d1.0_D1.7, F.Cu at (120.7, 112.4)
- added REF**290: ThroughHole_d1.0_D1.7, ThroughHole:ThroughHole_d1.0_D1.7, F.Cu at (92.7, 132.7)
- added REF**291: ThroughHole_d1.0_D1.7, ThroughHole:ThroughHole_d1.0_D1.7, F.Cu at (95.2, 132.7)
- added REF**292: ThroughHole_d1.0_D1.7, ThroughHole:ThroughHole_d1.0_D1.7, F.Cu at (97.8, 132.7)
- added REF**293: ThroughHole_d1.0_D1.7, ThroughHole:ThroughHole_d1.0_D1.7, F.Cu at (100.3, 132.7)
- added REF**294: ThroughHole_d1.0_D1.7, ThroughHole:ThroughHole_d1.0_D1.7, F.Cu at (102.9, 132.7)
- added REF**295: ThroughHole_d1.0_D1.7, ThroughHole:ThroughHole_d1.0_D1.7, F.Cu at (105.4, 132.7)
- added REF**296: ThroughHole_d1.0_D1.7, ThroughHole:ThroughHole_d1.0_D1.7, F.Cu at (108.0, 132.7)
- added REF**297: ThroughHole_d1.0_D1.7, ThroughHole:ThroughHole_d1.0_D1.7, F.Cu at (110.5, 132.7)
- added REF**298: ThroughHole_d1.0_D1.7, ThroughHole:ThroughHole_d1.0_D1.7, F.Cu at (113.0, 132.7)
- added REF**299: ThroughHole_d1.0_D1.7, ThroughHole:ThroughHole_d1.0_D1.7, F.Cu at (115.6, 132.7)
- added REF**3: ThroughHole_d1.0_D1.7, ThroughHole:ThroughHole_d1.0_D1.7, F.Cu at (57.1, 114.9)
- added REF**30: ThroughHole_d1.0_D1.7, ThroughHole:ThroughHole_d1.0_D1.7, F.Cu at (125.7, 114.9)
- added REF**30: ThroughHole_d1.0_D1.7, ThroughHole:ThroughHole_d1.0_D1.7, F.Cu at (123.2, 109.9)
- added REF**30: ThroughHole_d1.0_D1.7, ThroughHole:ThroughHole_d1.0_D1.7, F.Cu at (123.2, 112.4)
- added REF**300: ThroughHole_d1.0_D1.7, ThroughHole:ThroughHole_d1.0_D1.7, F.Cu at (118.1, 132.7)
- added REF**301: ThroughHole_d1.0_D1.7, ThroughHole:ThroughHole_d1.0_D1.7, F.Cu at (120.7, 132.7)
- added REF**302: ThroughHole_d1.0_D1.7, ThroughHole:ThroughHole_d1.0_D1.7, F.Cu at (123.2, 132.7)
- added REF**303: ThroughHole_d1.0_D1.7, ThroughHole:ThroughHole_d1.0_D1.7, F.Cu at (125.7, 132.7)
- added REF**304: ThroughHole_d1.0_D1.7, ThroughHole:ThroughHole_d1.0_D1.7, F.Cu at (128.3, 132.7)
- added REF**305: ThroughHole_d1.0_D1.7, ThroughHole:ThroughHole_d1.0_D1.7, F.Cu at (130.8, 132.7)
- added REF**306: ThroughHole_d1.0_D1.7, ThroughHole:ThroughHole_d1.0_D1.7, F.Cu at (133.3, 132.7)
- added REF**307: ThroughHole_d1.0_D1.7, ThroughHole:ThroughHole_d1.0_D1.7, F.Cu at (135.9, 132.7)
- added REF**308: ThroughHole_d1.0_D1.7, ThroughHole:ThroughHole_d1.0_D1.7, F.Cu at (138.4, 132.7)
- added REF**309: ThroughHole_d1.0_D1.7, ThroughHole:ThroughHole_d1.0_D1.7, F.Cu at (141.0, 132.7)
- added REF**31: ThroughHole_d1.0_D1.7, ThroughHole:ThroughHole_d1.0_D1.7, F.Cu at (128.3, 114.9)
- added REF**31: ThroughHole_d1.0_D1.7, ThroughHole:ThroughHole_d1.0_D1.7, F.Cu at (125.7, 109.9)
- added REF**31: ThroughHole_d1.0_D1.7, ThroughHole:ThroughHole_d1.0_D1.7, F.Cu at (125.7, 112.4)
- added REF**310: ThroughHole_d1.0_D1.7, ThroughHole:ThroughHole_d1.0_D1.7, F.Cu at (143.5, 132.7)
- added REF**311: ThroughHole_d1.0_D1.7, ThroughHole:ThroughHole_d1.0_D1.7, F.Cu at (146.1, 132.7)
- added REF**312: ThroughHole_d1.0_D1.7, ThroughHole:ThroughHole_d1.0_D1.7, F.Cu at (148.6, 132.7)
- added REF**313: ThroughHole_d1.0_D1.7, ThroughHole:ThroughHole_d1.0_D1.7, F.Cu at (52.1, 135.3)
- added REF**314: ThroughHole_d1.0_D1.7, ThroughHole:ThroughHole_d1.0_D1.7, F.Cu at (54.6, 135.3)
- added REF**315: ThroughHole_d1.0_D1.7, ThroughHole:ThroughHole_d1.0_D1.7, F.Cu at (57.1, 135.3)
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Connections:
- IC2 pad 1: /A15 -> /A10
- IC2 pad 2: /A14 -> /A11
- IC2 pad 3: /A13 -> /A12
- IC2 pad 4: /A12 -> /A13
- IC2 pad 5: /A11 -> /A14
- IC2 pad 6: /A10 -> /A15
- IC5 pad 11: /D7 -> /D0
- IC5 pad 12: /D6 -> /D1
- IC5 pad 13: /D5 -> /D2
- IC5 pad 14: /D4 -> /D3
- IC5 pad 15: /D3 -> /D4
- IC5 pad 16: /D2 -> /D5
- IC5 pad 17: /D1 -> /D6
- IC5 pad 18: /D0 -> /D7
- J1 pad 27: unconnected-(J1-Pin_27-Pad27) -> /R/~{W}
- J1 pad 31: unconnected-(J1-Pin_31-Pad31) -> /PA0
- J1 pad 32: unconnected-(J1-Pin_32-Pad32) -> /PA1
- J1 pad 33: unconnected-(J1-Pin_33-Pad33) -> /PA2
- J1 pad 34: unconnected-(J1-Pin_34-Pad34) -> /PA3
- J1 pad 35: unconnected-(J1-Pin_35-Pad35) -> /PA4
- J1 pad 36: unconnected-(J1-Pin_36-Pad36) -> /PA5
- J1 pad 37: unconnected-(J1-Pin_37-Pad37) -> /PA6
- J1 pad 38: unconnected-(J1-Pin_38-Pad38) -> /PA7
- J4 pad 27: unconnected-(J4-Pin_27-Pad27) -> /R/~{W}
- J4 pad 31: unconnected-(J4-Pin_31-Pad31) -> /PA0
- J4 pad 32: unconnected-(J4-Pin_32-Pad32) -> /PA1
- J4 pad 33: unconnected-(J4-Pin_33-Pad33) -> /PA2
- J4 pad 34: unconnected-(J4-Pin_34-Pad34) -> /PA3
- J4 pad 35: unconnected-(J4-Pin_35-Pad35) -> /PA4
- J4 pad 36: unconnected-(J4-Pin_36-Pad36) -> /PA5
- J4 pad 37: unconnected-(J4-Pin_37-Pad37) -> /PA6
- J4 pad 38: unconnected-(J4-Pin_38-Pad38) -> /PA7
- JP2 pad 2: /AD15 -> /A15
- SW1 pad 1: Net-(IC5-A0) -> VCC
- SW1 pad 10: VCC -> Net-(IC5-A6)
- SW1 pad 11: VCC -> Net-(IC5-A5)
- SW1 pad 12: VCC -> Net-(IC5-A4)
- SW1 pad 13: VCC -> Net-(IC5-A3)
- SW1 pad 14: VCC -> Net-(IC5-A2)
- SW1 pad 15: VCC -> Net-(IC5-A1)
- SW1 pad 16: VCC -> Net-(IC5-A0)
- SW1 pad 2: Net-(IC5-A1) -> VCC
- SW1 pad 3: Net-(IC5-A2) -> VCC
- SW1 pad 4: Net-(IC5-A3) -> VCC
- SW1 pad 5: Net-(IC5-A4) -> VCC
- SW1 pad 6: Net-(IC5-A5) -> VCC
- SW1 pad 7: Net-(IC5-A6) -> VCC
- SW1 pad 8: Net-(IC5-A7) -> VCC
- SW1 pad 9: VCC -> Net-(IC5-A7)
Routing:
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Other:
- board text added: "~{IRQ}"

Commit message: 完成
Parts:
- removed the REF**13 at (80.0, 109.9)
- removed the REF**13 at (80.0, 112.4)
- added G***: LOGO, LOGO, F.Cu at (85.1, 79.4)
- moved CP2 2.54 mm to (93.3, 84.5)
- moved IC2 2.54 mm to (111.1, 79.4)
- moved CP5 0.66 mm to (112.4, 57.2)
- moved IC5 0.63 mm to (109.9, 54.6)
Connections:
- JP1 pad 10: VCC -> GND
- JP1 pad 9: GND -> VCC
Routing:
- net /~{WR}: track 11.1 -> 163.0 mm, vias 0 -> 1
- net VCC: track 168.5 -> 300.3 mm, vias 0 -> 2
- net /~{RD}: track 11.1 -> 137.3 mm, vias 0 -> 1
- net GND: track 143.9 -> 217.6 mm, vias 0 -> 39
- net Net-(IC5-G2): track 0.00 -> 59.7 mm
- net /~{IO_S0}: track 8.03 -> 44.3 mm, vias 0 -> 1
- net /~{IO_S1}: track 8.03 -> 38.6 mm
- net /~{IRQ}: track 11.1 -> 28.6 mm
- net Net-(J2-Pin_1): track 0.00 -> 16.6 mm
- net /A15: track 107.1 -> 94.4 mm, vias 0 -> 1
- net Net-(J7-Pin_1): track 0.00 -> 7.40 mm
- net Net-(J6-Pin_1): track 0.00 -> 6.61 mm
- net /A8: track 91.4 -> 97.5 mm, vias 2 -> 1
- net /A9: track 89.6 -> 86.7 mm, vias 3 -> 2
- net Net-(IC3-~{E1}): track 9.46 -> 6.92 mm
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- added copper zone on B.Cu, net GND
- added copper zone on F.Cu, net GND
Other:
- board text added: "A0"
- board text added: "A1"
- board text added: "A10"
- board text added: "A11"
- board text added: "A12"
- board text added: "A13"
- board text added: "A14"
- board text added: "A15"
- board text added: "A2"
- board text added: "A3"
- board text added: "A4"
- board text added: "A5"
- board text added: "A6"
- board text added: "A7"
- board text added: "A8"
- board text added: "A9"
- board text added: "Default: 0x0000-7FFF: RAM 0x8000-FEFF: Reserved 0xFF00-F7FF: I/O 0xF800-FFFF: Reserved For other mappings, see the documentations for each CPU."
- board text added: "GND"
- board text added: "HCx_Memory Rev 1.0 2025 DGK"
- board text added: "VCC"

Commit message: Memboardv2.0
Parts:
- removed IC5: 74HC541, Package_DIP:DIP-20_W7.62mm
- removed JP1: Conn_02x17_Counter_Clockwise, Connector_PinHeader_2.54mm:PinHeader_2x17_P2.54mm_Vertical
- removed JP2: Jumper_2_Bridged, Connector_PinHeader_2.54mm:PinHeader_1x02_P2.54mm_Vertical
- removed REF** (x4): ThroughHole_d1.0_D1.7, ThroughHole:ThroughHole_d1.0_D1.7
- removed the REF**14 at (85.1, 114.9)
- removed the REF**14 at (82.5, 112.4)
- removed the REF**14 at (82.5, 109.9)
- removed the REF**15 at (87.6, 114.9)
- removed the REF**15 at (85.1, 112.4)
- removed the REF**15 at (85.1, 109.9)
- removed the REF**16 at (87.6, 112.4)
- removed the REF**16 at (87.6, 109.9)
- removed the REF**16 at (90.2, 114.9)
- removed the REF**17 at (92.7, 114.9)
- removed the REF**17 at (90.2, 112.4)
- removed the REF**17 at (90.2, 109.9)
- removed the REF**18 at (92.7, 112.4)
- removed the REF**18 at (95.2, 114.9)
- removed the REF**18 at (92.7, 109.9)
- removed the REF**19 at (95.2, 109.9)
- removed the REF**19 at (95.2, 112.4)
- removed the REF**19 at (97.8, 114.9)
- removed the REF**20 at (97.8, 112.4)
- removed the REF**20 at (97.8, 109.9)
- removed the REF**20 at (100.3, 114.9)
- removed the REF**21 at (100.3, 109.9)
- removed the REF**21 at (102.9, 114.9)
- removed the REF**21 at (100.3, 112.4)
- removed the REF**22 at (102.9, 112.4)
- removed the REF**22 at (102.9, 109.9)
- removed the REF**22 at (105.4, 114.9)
- removed the REF**23 at (108.0, 114.9)
- removed the REF**23 at (105.4, 112.4)
- removed the REF**23 at (105.4, 109.9)
- removed the REF**24 at (108.0, 109.9)
- removed the REF**24 at (110.5, 114.9)
- removed the REF**24 at (108.0, 112.4)
- removed the REF**25 at (110.5, 109.9)
- removed the REF**25 at (110.5, 112.4)
- removed the REF**25 at (113.0, 114.9)
- removed the REF**26 at (113.0, 112.4)
- removed the REF**26 at (113.0, 109.9)
- removed the REF**26 at (115.6, 114.9)
- removed the REF**27 at (115.6, 109.9)
- removed the REF**27 at (115.6, 112.4)
- removed the REF**27 at (118.1, 114.9)
- removed the REF**28 at (118.1, 112.4)
- removed the REF**28 at (118.1, 109.9)
- removed the REF**28 at (120.7, 114.9)
- removed the REF**29 at (123.2, 114.9)
- removed the REF**29 at (120.7, 109.9)
- removed the REF**29 at (120.7, 112.4)
- removed the REF**30 at (125.7, 114.9)
- removed the REF**30 at (123.2, 109.9)
- removed the REF**30 at (123.2, 112.4)
- removed the REF**31 at (128.3, 114.9)
- removed the REF**31 at (125.7, 109.9)
- removed the REF**31 at (125.7, 112.4)
- removed the REF**32 at (130.8, 114.9)
- removed the REF**32 at (128.3, 109.9)
- removed the REF**32 at (128.3, 112.4)
- removed the REF**33 at (130.8, 112.4)
- removed the REF**33 at (130.8, 109.9)
- removed the REF**33 at (133.3, 114.9)
- removed the REF**34 at (133.3, 109.9)
- removed the REF**34 at (135.9, 114.9)
- removed the REF**34 at (133.3, 112.4)
- removed the REF**35 at (138.4, 114.9)
- removed the REF**35 at (135.9, 109.9)
- removed the REF**35 at (135.9, 112.4)
- removed the REF**36 at (138.4, 109.9)
- removed the REF**36 at (138.4, 112.4)
- removed the REF**36 at (141.0, 114.9)
- removed the REF**37 at (141.0, 109.9)
- removed the REF**37 at (141.0, 112.4)
- removed the REF**37 at (143.5, 114.9)
- removed the REF**38 at (143.5, 112.4)
- removed the REF**38 at (146.1, 114.9)
- removed the REF**38 at (143.5, 109.9)
- removed the REF**39 at (146.1, 112.4)
- removed the REF**39 at (148.6, 114.9)
- removed the REF**39 at (146.1, 109.9)
- added CP1: 0.1u, Capacitor_THT:C_Disc_D3.0mm_W1.6mm_P2.50mm, F.Cu at (121.3, 91.4)
- added J3: Changer, Connector_PinSocket_2.54mm:PinSocket_1x20_P2.54mm_Vertical, F.Cu at (72.1, 63.5)
- added J4: Changer, Connector_PinSocket_2.54mm:PinSocket_1x20_P2.54mm_Vertical, F.Cu at (79.8, 63.5)
- added J5: Conn_01x03_Pin, Connector_PinSocket_2.54mm:PinSocket_1x03_P2.54mm_Vertical, F.Cu at (123.8, 96.5)
- added J7: Conn_01x03_Pin, Connector_PinSocket_2.54mm:PinSocket_1x03_P2.54mm_Vertical, F.Cu at (131.4, 83.8)
- added J8: Conn_01x03_Pin, Connector_PinSocket_2.54mm:PinSocket_1x03_P2.54mm_Vertical, F.Cu at (131.4, 96.5)
- added REF**14: ThroughHole_d1.0_D1.7, ThroughHole:ThroughHole_d1.0_D1.7, F.Cu at (85.1, 115.6)
- added REF**15: ThroughHole_d1.0_D1.7, ThroughHole:ThroughHole_d1.0_D1.7, F.Cu at (87.6, 115.6)
- added REF**16: ThroughHole_d1.0_D1.7, ThroughHole:ThroughHole_d1.0_D1.7, F.Cu at (90.2, 115.6)
- added REF**17: ThroughHole_d1.0_D1.7, ThroughHole:ThroughHole_d1.0_D1.7, F.Cu at (92.7, 115.6)
- added REF**18: ThroughHole_d1.0_D1.7, ThroughHole:ThroughHole_d1.0_D1.7, F.Cu at (95.2, 115.6)
- added REF**19: ThroughHole_d1.0_D1.7, ThroughHole:ThroughHole_d1.0_D1.7, F.Cu at (97.8, 115.6)
- added REF**20: ThroughHole_d1.0_D1.7, ThroughHole:ThroughHole_d1.0_D1.7, F.Cu at (100.3, 115.6)
- added REF**21: ThroughHole_d1.0_D1.7, ThroughHole:ThroughHole_d1.0_D1.7, F.Cu at (102.9, 115.6)
- added REF**22: ThroughHole_d1.0_D1.7, ThroughHole:ThroughHole_d1.0_D1.7, F.Cu at (105.4, 115.6)
- added REF**23: ThroughHole_d1.0_D1.7, ThroughHole:ThroughHole_d1.0_D1.7, F.Cu at (108.0, 115.6)
- added REF**24: ThroughHole_d1.0_D1.7, ThroughHole:ThroughHole_d1.0_D1.7, F.Cu at (110.5, 115.6)
- added REF**25: ThroughHole_d1.0_D1.7, ThroughHole:ThroughHole_d1.0_D1.7, F.Cu at (113.0, 115.6)
- added REF**26: ThroughHole_d1.0_D1.7, ThroughHole:ThroughHole_d1.0_D1.7, F.Cu at (115.6, 115.6)
- added REF**27: ThroughHole_d1.0_D1.7, ThroughHole:ThroughHole_d1.0_D1.7, F.Cu at (118.1, 115.6)
- added REF**28: ThroughHole_d1.0_D1.7, ThroughHole:ThroughHole_d1.0_D1.7, F.Cu at (120.7, 115.6)
- added REF**29: ThroughHole_d1.0_D1.7, ThroughHole:ThroughHole_d1.0_D1.7, F.Cu at (123.2, 115.6)
- added REF**30: ThroughHole_d1.0_D1.7, ThroughHole:ThroughHole_d1.0_D1.7, F.Cu at (125.7, 115.6)
- added REF**31: ThroughHole_d1.0_D1.7, ThroughHole:ThroughHole_d1.0_D1.7, F.Cu at (128.3, 115.6)
- added REF**32: ThroughHole_d1.0_D1.7, ThroughHole:ThroughHole_d1.0_D1.7, F.Cu at (130.8, 115.6)
- added REF**33: ThroughHole_d1.0_D1.7, ThroughHole:ThroughHole_d1.0_D1.7, F.Cu at (133.3, 115.6)
- added REF**34: ThroughHole_d1.0_D1.7, ThroughHole:ThroughHole_d1.0_D1.7, F.Cu at (135.9, 115.6)
- added REF**35: ThroughHole_d1.0_D1.7, ThroughHole:ThroughHole_d1.0_D1.7, F.Cu at (138.4, 115.6)
- added REF**36: ThroughHole_d1.0_D1.7, ThroughHole:ThroughHole_d1.0_D1.7, F.Cu at (141.0, 115.6)
- added REF**37: ThroughHole_d1.0_D1.7, ThroughHole:ThroughHole_d1.0_D1.7, F.Cu at (143.5, 115.6)
- added REF**38: ThroughHole_d1.0_D1.7, ThroughHole:ThroughHole_d1.0_D1.7, F.Cu at (146.1, 115.6)
- added REF**39: ThroughHole_d1.0_D1.7, ThroughHole:ThroughHole_d1.0_D1.7, F.Cu at (148.6, 115.6)
- added REF**432: ThroughHole_d1.0_D1.7, ThroughHole:ThroughHole_d1.0_D1.7, F.Cu at (57.1, 143.5)
- added REF**466: ThroughHole_d1.0_D1.7, ThroughHole:ThroughHole_d1.0_D1.7, F.Cu at (143.5, 143.5)
- added U1: 74HC573, Package_DIP:DIP-20_W7.62mm, F.Cu at (109.7, 54.1)
- added U2: 74HC00, Package_DIP:DIP-14_W7.62mm, F.Cu at (139.1, 86.4)
- moved CP2 32.7 mm to (111.8, 67.3), turned to 90 degrees
- moved IC4 24.7 mm to (147.3, 64.8), turned to -90 degrees
- moved G*** 10.6 mm to (90.8, 70.5)
- moved J6 9.10 mm to (116.8, 111.1), turned to 90 degrees
- moved J12 8.64 mm to (132.1, 111.1), turned to 90 degrees
- moved J11 8.28 mm to (124.5, 111.1), turned to 90 degrees
- moved CP3 7.65 mm to (92.7, 92.1)
- moved CP4 7.65 mm to (90.2, 104.1)
- moved CP5 7.65 mm to (121.3, 104.1)
- moved IC3 7.65 mm to (110.5, 99.1)
- moved IC1 7.65 mm to (139.1, 99.1)
- moved IC2 7.65 mm to (110.5, 87.0)
- moved J10 7.01 mm to (110.5, 109.2)
- moved J9 5.76 mm to (110.5, 111.8)
- moved REF**352 0.64 mm to (52.1, 138.4)
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- renumbered CP1 to CP2, CP2 to CP3, CP3 to CP4, CP4 to CP5, CP5 to CP6, IC4 to IC1, IC1 to IC4, J5 to J10, J6 to J11, J7 to J12, J4 to J2, J2 to J6, J3 to J9
Connections:
- net Net-(IC3-~{E1}) renamed /7430
- IC3 pad 1: /A4 -> /A5
- IC3 pad 2: /A5 -> /A6
- IC3 pad 3: /A6 -> /A7
- IC3 pad 4: /A7 -> GND
- IC4 pad 1: /A14 -> /AD14
- IC4 pad 10: /A0 -> /AD0
- IC4 pad 2: /A12 -> /AD12
- IC4 pad 20: Net-(IC1-~{CS}) -> /~{RAM_CE}
- IC4 pad 21: /A10 -> /AD10
- IC4 pad 23: /A11 -> /AD11
- IC4 pad 24: /A9 -> /AD9
- IC4 pad 25: /A8 -> /AD8
- IC4 pad 26: /A13 -> /AD13
- IC4 pad 3: /A7 -> /AD7
- IC4 pad 4: /A6 -> /AD6
- IC4 pad 5: /A5 -> /AD5
- IC4 pad 6: /A4 -> /AD4
- IC4 pad 7: /A3 -> /AD3
- IC4 pad 8: /A2 -> /AD2
- IC4 pad 9: /A1 -> /AD1
Routing:
- net GND: track 217.6 -> 40.5 mm, vias 39 -> 2
- net /AD14: track 34.0 -> 133.7 mm, vias 0 -> 2
- net /AD6: track 24.3 -> 124.0 mm, vias 0 -> 2
- net /AD7: track 21.9 -> 119.1 mm, vias 0 -> 3
- net /AD12: track 31.4 -> 127.7 mm, vias 0 -> 1
- net Net-(J3-Pin_20): track 0.00 -> 85.7 mm, vias 0 -> 1
- net /AD13: track 29.5 -> 113.9 mm, vias 0 -> 1
- net /~{RAM_CE}: track 0.00 -> 76.4 mm, vias 0 -> 1
- net /AD9: track 24.4 -> 98.5 mm
- net /A4: track 73.6 -> 0.00 mm
- net /AD5: track 20.8 -> 93.4 mm, vias 0 -> 2
- net /AD8: track 26.3 -> 98.9 mm, vias 0 -> 4
- net /A13: track 101.0 -> 29.5 mm
- net /AD3: track 18.7 -> 90.0 mm, vias 0 -> 1
- net /AD4: track 23.3 -> 93.2 mm, vias 0 -> 2
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Other:
- board text added: "HCx_Memory Rev 2.0 2025 DGK"
- board text removed: "Default: 0x0000-7FFF: RAM 0x8000-FEFF: Reserved 0xFF00-F7FF: I/O 0xF800-FFFF: Reserved For other mappings, see the documentations for each CPU."
- board text removed: "HCx_Memory Rev 1.0 2025 DGK"
