File: HC_MemoryBoard/HC_MemoryBoard.kicad_sch (KiCad schematic)
At the start: 22 parts, among them IC1 HM62256BLP, IC2 74HC30, IC3 74HC138, IC4 74HC32, IC5 74HC541, J1 Expantion_Connector, J2 Conn_01x02_Pin, J3 Conn_01x08_Pin, J4 Expantion_Connector, J5 Conn_01x08_Pin, J6 Conn_01x02_Pin, J7 Conn_01x02_Pin, SW1 SW_DIP_x08

Commit message: 基板ぬ
Parts:
- added H1, H2, H3, H4: MountingHole, MountingHole:MountingHole_3.2mm_M3, symbol Mechanical:MountingHole
- J2: footprint Connector_PinHeader_2.54mm:PinHeader_2x01_P2.54mm_Vertical -> Connector_PinHeader_2.54mm:PinHeader_1x02_P2.54mm_Vertical
- J3: footprint Connector_PinHeader_2.54mm:PinHeader_1x08_P2.54mm_Vertical_SMD_Pin1Left -> Connector_PinHeader_2.54mm:PinHeader_1x08_P2.54mm_Vertical
- J4: footprint Connector_PinHeader_2.54mm:PinHeader_1x40_P2.54mm_Vertical -> Connector_PinHeader_2.54mm:PinHeader_2x20_P2.54mm_Vertical
- JP1: symbol Connector_Generic:Conn_02x17_Counter_Clockwise -> Connector_Generic:Conn_02x17_Odd_Even
- JP2: footprint Connector_PinHeader_2.54mm:PinHeader_2x01_P2.54mm_Horizontal -> Connector_PinHeader_2.54mm:PinHeader_1x02_P2.54mm_Vertical
Connections:
- net A0: now also JP1.2 (Pin_2); no longer JP1.34 (Pin_34)
- net A1: now also JP1.4 (Pin_4); no longer JP1.33 (Pin_33)
- net A10: now also JP1.24 (Pin_24); no longer JP1.23 (Pin_23)
- net A11: now also JP1.26 (Pin_26); no longer JP1.22 (Pin_22)
- net A12: now also JP1.28 (Pin_28); no longer JP1.21 (Pin_21)
- net A13: now also JP1.30 (Pin_30); no longer JP1.20 (Pin_20)
- net A14: now also JP1.32 (Pin_32); no longer JP1.19 (Pin_19)
- net A15: now also JP1.34 (Pin_34); no longer JP1.18 (Pin_18)
- net A2: now also JP1.6 (Pin_6); no longer JP1.32 (Pin_32)
- net A3: now also JP1.8 (Pin_8); no longer JP1.31 (Pin_31)
- net A4: now also JP1.12 (Pin_12); no longer JP1.29 (Pin_29)
- net A5: now also JP1.14 (Pin_14); no longer JP1.28 (Pin_28)
- net A6: now also JP1.16 (Pin_16); no longer JP1.27 (Pin_27)
- net A7: now also JP1.18 (Pin_18); no longer JP1.26 (Pin_26)
- net A8: now also JP1.20 (Pin_20); no longer JP1.25 (Pin_25)
- net A9: now also JP1.22 (Pin_22); no longer JP1.24 (Pin_24)
- net AD1: now also JP1.3 (Pin_3); no longer JP1.2 (Pin_2)
- net AD10: now also JP1.23 (Pin_23); no longer JP1.12 (Pin_12)
- net AD11: now also JP1.25 (Pin_25); no longer JP1.13 (Pin_13)
- net AD12: now also JP1.27 (Pin_27); no longer JP1.14 (Pin_14)
- net AD13: now also JP1.29 (Pin_29); no longer JP1.15 (Pin_15)
- net AD14: now also JP1.31 (Pin_31); no longer JP1.16 (Pin_16)
- net AD15: now also JP1.33 (Pin_33); no longer JP1.17 (Pin_17)
- net AD2: now also JP1.5 (Pin_5); no longer JP1.3 (Pin_3)
- net AD3: now also JP1.7 (Pin_7); no longer JP1.4 (Pin_4)
- net AD4: now also JP1.11 (Pin_11); no longer JP1.6 (Pin_6)
- net AD5: now also JP1.13 (Pin_13); no longer JP1.7 (Pin_7)
- net AD6: now also JP1.15 (Pin_15); no longer JP1.8 (Pin_8)
- net AD7: now also JP1.17 (Pin_17); no longer JP1.9 (Pin_9)
- net AD8: now also JP1.19 (Pin_19); no longer JP1.10 (Pin_10)
- net AD9: now also JP1.21 (Pin_21); no longer JP1.11 (Pin_11)
- net GND: now also JP1.9 (Pin_9); no longer JP1.5 (Pin_5)
- net VCC: now also JP1.10 (Pin_10), SW1.10, SW1.11, SW1.12, SW1.13, SW1.14, SW1.15, SW1.16, SW1.9; no longer JP1.30 (Pin_30), SW1.1, SW1.2, SW1.3, SW1.4, SW1.5, SW1.6, SW1.7, SW1.8
- net R/~{W}: now reaches J1.27 (Pin_27)
- net R/~{W}: now also J4.27 (Pin_27)
- net PA0: now reaches J1.31 (Pin_31)
- net PA0: now also J4.31 (Pin_31)
- net PA1: now reaches J1.32 (Pin_32)
- net PA1: now also J4.32 (Pin_32)
- net PA2: now reaches J1.33 (Pin_33)
- net PA2: now also J4.33 (Pin_33)
- net PA3: now reaches J1.34 (Pin_34)
- net PA3: now also J4.34 (Pin_34)
- net PA4: now reaches J1.35 (Pin_35)
- net PA4: now also J4.35 (Pin_35)
- net PA5: now reaches J1.36 (Pin_36)
- net PA5: now also J4.36 (Pin_36)
- net PA6: now reaches J1.37 (Pin_37)
- net PA6: now also J4.37 (Pin_37)
- net PA7: now reaches J1.38 (Pin_38)
- net PA7: now also J4.38 (Pin_38)
- net at IC5.8 (A6), RN1.3 (R2): now also SW1.7; no longer SW1.10
- net at IC5.7 (A5), RN1.4 (R3): now also SW1.6; no longer SW1.11
- net at IC5.6 (A4), RN1.5 (R4): now also SW1.5; no longer SW1.12
- net at IC5.5 (A3), RN1.6 (R5): now also SW1.4; no longer SW1.13
- net at IC5.4 (A2), RN1.7 (R6): now also SW1.3; no longer SW1.14
- net at IC5.3 (A1), RN1.8 (R7): now also SW1.2; no longer SW1.15
- net at IC5.2 (A0), RN1.9 (R8): now also SW1.1; no longer SW1.16
- net at IC5.9 (A7), RN1.2 (R1): now also SW1.8; no longer SW1.9
- no-connect marks 18 -> 0

Commit message: 配線
Connections:
- net A10: now also IC2.1; no longer IC2.6
- net A11: now also IC2.2; no longer IC2.5
- net A12: now also IC2.3; no longer IC2.4
- net A13: now also IC2.4; no longer IC2.3
- net A14: now also IC2.5; no longer IC2.2
- net A15: now also IC2.6, JP2.2 (B); no longer IC2.1
- net AD15: no longer JP2.2 (B)
- net D0: now also IC5.11 (Y7); no longer IC5.18 (Y0)
- net D1: now also IC5.12 (Y6); no longer IC5.17 (Y1)
- net D2: now also IC5.13 (Y5); no longer IC5.16 (Y2)
- net D3: now also IC5.14 (Y4); no longer IC5.15 (Y3)
- net D4: now also IC5.15 (Y3); no longer IC5.14 (Y4)
- net D5: now also IC5.16 (Y2); no longer IC5.13 (Y5)
- net D6: now also IC5.17 (Y1); no longer IC5.12 (Y6)
- net D7: now also IC5.18 (Y0); no longer IC5.11 (Y7)
- net VCC: now also SW1.1, SW1.2, SW1.3, SW1.4, SW1.5, SW1.6, SW1.7, SW1.8; no longer SW1.10, SW1.11, SW1.12, SW1.13, SW1.14, SW1.15, SW1.16, SW1.9
- net at IC5.2 (A0), RN1.9 (R8): now also SW1.16; no longer SW1.1
- net at IC5.3 (A1), RN1.8 (R7): now also SW1.15; no longer SW1.2
- net at IC5.4 (A2), RN1.7 (R6): now also SW1.14; no longer SW1.3
- net at IC5.5 (A3), RN1.6 (R5): now also SW1.13; no longer SW1.4
- net at IC5.6 (A4), RN1.5 (R4): now also SW1.12; no longer SW1.5
- net at IC5.7 (A5), RN1.4 (R3): now also SW1.11; no longer SW1.6
- net at IC5.8 (A6), RN1.3 (R2): now also SW1.10; no longer SW1.7
- net at IC5.9 (A7), RN1.2 (R1): now also SW1.9; no longer SW1.8
Other:
- moved on the sheet: IC2A

Commit message: 完成
Connections:
- net GND: now also JP1.10 (Pin_10); no longer JP1.9 (Pin_9)
- net VCC: now also JP1.9 (Pin_9); no longer JP1.10 (Pin_10)
Other:
- title: (none) -> HCx series memory board
Changed lines of the file:
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@@
 	(generator_version "9.0")
 	(paper "A4")
+	(title_block
+		(title "HCx series memory board")
+		(date "2025-04-22")
+		(rev "Rev1.0")
+	)
 	(junction
 		(at 160.02 173.99)
@@
 	(wire
 		(pts
-			(xy 111.76 50.8) (xy 115.57 50.8)
+			(xy 111.76 50.8) (xy 119.38 50.8)
 		)
 		(stroke
@@
 	(symbol
 		(lib_id "power:GND")
-		(at 90.17 50.8 0)
+		(at 119.38 50.8 0)
 		(unit 1)
 		(exclude_from_sim no)
@@
 		(dnp no)
 		(property "Reference" "#PWR06"
-			(at 90.17 57.15 0)
+			(at 119.38 57.15 0)
 			(effects
 				(font
@@
 		)
 		(property "Value" "GND"
-			(at 86.36 51.562 0)
+			(at 122.936 50.546 0)
 			(effects
 				(font
@@
 		)
 		(property "Footprint" ""
-			(at 90.17 50.8 0)
+			(at 119.38 50.8 0)
 			(effects
 				(font
@@
 		)
 		(property "Datasheet" ""
-			(at 90.17 50.8 0)
+			(at 119.38 50.8 0)
 			(effects
 				(font
@@
 		)
 		(property "Description" "Power symbol creates a global label with name \"GND\" , ground"
-			(at 90.17 50.8 0)
+			(at 119.38 50.8 0)
 			(effects
 				(font
@@
 	(symbol
 		(lib_id "power:VCC")
-		(at 115.57 50.8 0)
+		(at 90.17 50.8 0)
 		(unit 1)
 		(exclude_from_sim no)
@@
 		(dnp no)
 		(property "Reference" "#PWR05"
-			(at 115.57 54.61 0)
+			(at 90.17 54.61 0)
 			(effects
 				(font
@@
 		)
 		(property "Value" "VCC"
-			(at 119.126 50.038 0)
+			(at 93.726 50.038 0)
 			(effects
 				(font
@@
 		)
 		(property "Footprint" ""
-			(at 115.57 50.8 0)
+			(at 90.17 50.8 0)
 			(effects
 				(font
@@
 		)
 		(property "Datasheet" ""
-			(at 115.57 50.8 0)
+			(at 90.17 50.8 0)
 			(effects
 				(font
@@
 		)
 		(property "Description" "Power symbol creates a global label with name \"VCC\""
-			(at 115.57 50.8 0)
+			(at 90.17 50.8 0)
 			(effects
 				(font

Commit message: Memboardv2.0
Parts:
- removed IC5: 74HC541, Package_DIP:DIP-20_W7.62mm, symbol 74xx_2:74HC541
- removed JP1: Conn_02x17_Counter_Clockwise, Connector_PinHeader_2.54mm:PinHeader_2x17_P2.54mm_Vertical, symbol Connector_Generic:Conn_02x17_Odd_Even
- removed JP2: Jumper_2_Bridged, Connector_PinHeader_2.54mm:PinHeader_1x02_P2.54mm_Vertical, symbol Jumper:Jumper_2_Bridged
- added CP1: 0.1u, Capacitor_THT:C_Disc_D3.0mm_W1.6mm_P2.50mm, symbol Device2:C_Bypass
- added J3, J4: Changer, Connector_PinSocket_2.54mm:PinSocket_1x20_P2.54mm_Vertical, symbol Connector:Conn_01x20_Pin
- added J5, J7, J8: Conn_01x03_Pin, Connector_PinSocket_2.54mm:PinSocket_1x03_P2.54mm_Vertical, symbol Connector:Conn_01x03_Pin
- added U1: 74HC573, Package_DIP:DIP-20_W7.62mm, symbol 74xx:74LS573
- added U2: 74HC00, Package_DIP:DIP-14_W7.62mm, symbol 74xx:74HC00
- renumbered CP1 to CP2, CP2 to CP3, CP3 to CP4, CP4 to CP5, CP5 to CP6, IC4 to IC1, IC1 to IC4, J5 to J10, J6 to J11, J7 to J12, J4 to J2, J2 to J6, J3 to J9
Connections:
- net A0: now also J4.2 (Pin_2); no longer IC4.10 (A0)
- net A1: now also J4.3 (Pin_3); no longer IC4.9 (A1)
- net A10: now also J4.13 (Pin_13); no longer IC4.21 (A10)
- net A11: now also J4.14 (Pin_14); no longer IC4.23 (A11)
- net A12: now also J4.15 (Pin_15); no longer IC4.2 (A12)
- net A13: now also J4.16 (Pin_16); no longer IC4.26 (A13)
- net A14: now also J4.17 (Pin_17); no longer IC4.1 (A14)
- net A15: now also J4.18 (Pin_18)
- net A2: now also J4.4 (Pin_4); no longer IC4.8 (A2)
- net A3: now also J4.5 (Pin_5); no longer IC4.7 (A3)
- net A4: now also J4.6 (Pin_6); no longer IC3.1 (A0), IC4.6 (A4)
- net A5: now also IC3.1 (A0), J4.7 (Pin_7); no longer IC3.2 (A1), IC4.5 (A5)
- net A6: now also IC3.2 (A1), J4.8 (Pin_8); no longer IC3.3 (A2), IC4.4 (A6)
- net A7: now also IC3.3 (A2), J4.9 (Pin_9); no longer IC3.4 (~{E0}), IC4.3 (A7)
- net A8: now also J4.11 (Pin_11); no longer IC4.25 (A8)
- net A9: now also J4.12 (Pin_12); no longer IC4.24 (A9)
- net AD0: now also IC4.10 (A0), J3.2 (Pin_2)
- net AD1: now also IC4.9 (A1), J3.3 (Pin_3)
- net AD10: now also IC4.21 (A10), J3.13 (Pin_13)
- net AD11: now also IC4.23 (A11), J3.14 (Pin_14)
- net AD12: now also IC4.2 (A12), J3.15 (Pin_15)
- net AD13: now also IC4.26 (A13), J3.16 (Pin_16)
- net AD14: now also IC4.1 (A14), J3.17 (Pin_17)
- net AD15: now also J3.18 (Pin_18)
- net AD2: now also IC4.8 (A2), J3.4 (Pin_4)
- net AD3: now also IC4.7 (A3), J3.5 (Pin_5)
- net AD4: now also IC4.6 (A4), J3.6 (Pin_6)
- net AD5: now also IC4.5 (A5), J3.7 (Pin_7)
- net AD6: now also IC4.4 (A6), J3.8 (Pin_8)
- net AD7: now also IC4.3 (A7), J3.9 (Pin_9)
- net AD8: now also IC4.25 (A8), J3.11 (Pin_11)
- net AD9: now also IC4.24 (A9), J3.12 (Pin_12)
- net D0: now also U1.12 (Q7)
- net D1: now also U1.13 (Q6)
- net D2: now also U1.14 (Q5)
- net D3: now also U1.15 (Q4)
- net D4: now also U1.16 (Q3)
- net D5: now also U1.17 (Q2)
- net D6: now also U1.18 (Q1)
- net D7: now also U1.19 (Q0)
- net GND: now also IC3.4 (~{E0}), CP1.2, J4.1 (Pin_1), J4.10 (Pin_10), J4.19 (Pin_19), U1.10 (GND), U2.7 (GND)
- net VCC: now also CP1.1, J3.1 (Pin_1), J3.10 (Pin_10), J3.19 (Pin_19), U1.20 (VCC), U2.1, U2.14 (VCC)
- net 7430: now reaches IC2.8, IC3.5 (~{E1})
- net 7430: now also U2.2
- net ~{RAM_CE}: now reaches IC4.20 (~{CS})
- net ~{RAM_CE}: now also J4.20 (Pin_20)
- net at IC1.3: now also U1.1 (OE), U1.11 (Load)
- net at RN1.3 (R2), SW1.10: now also U1.8 (D6)
- net at RN1.4 (R3), SW1.11: now also U1.7 (D5)
- net at RN1.5 (R4), SW1.12: now also U1.6 (D4)
- net at RN1.6 (R5), SW1.13: now also U1.5 (D3)
- net at RN1.7 (R6), SW1.14: now also U1.4 (D2)
- net at RN1.8 (R7), SW1.15: now also U1.3 (D1)
- net at RN1.9 (R8), SW1.16: now also U1.2 (D0)
- net at RN1.2 (R1), SW1.9: now also U1.9 (D7)
- new net: J8.1 (Pin_1), U2.11
- new net: J8.2 (Pin_2), U2.12
- new net: J8.3 (Pin_3), U2.13
- new net: J5.1 (Pin_1), U2.8
- new net: J5.2 (Pin_2), U2.9
- new net: J5.3 (Pin_3), U2.10
- new net: J7.1 (Pin_1), U2.4
- new net: J7.2 (Pin_2), U2.5
- new net: J7.3 (Pin_3), U2.6
- new net: J3.20 (Pin_20), U2.3
Other:
- moved on the sheet: CP2, CP3, CP4, CP5, CP6, IC1E, IC2B, IC3, J10, J9
